File: breakouts/splitter_breakout/splitter_breakout.sch (KiCad schematic (older format))
At the start: 4 parts, among them U101 CONN_SMA_2GND, U102 CONN_SMA_2GND, U103 CONN_SMA_2GND, U3 PWR_SPLITTER

Commit message: modified splitter breakout to use coplanar waveguide.
Parts:
- U101, U102, U103: footprint vna_footprints:142-0721-882_sma_cutout -> vna_footprints:SMA_CPW_1MM_.2MM
Changed lines of the file:
@@
 LIBS:tcm-63ax+
 LIBS:mounting_box
-LIBS:conn_sma_2gnd
 LIBS:splitter_breakout-cache
 EELAYER 25 0
@@
 F 0 "U101" H 6000 4000 60  0000 C CNN
 F 1 "CONN_SMA_2GND" H 6350 4100 60  0000 C CNN
-F 2 "vna_footprints:142-0721-882_sma_cutout" H 6300 3800 60  0001 C CNN
+F 2 "vna_footprints:SMA_CPW_1MM_.2MM" H 6300 3800 60  0001 C CNN
 F 3 "" H 6300 3800 60  0000 C CNN
 	1    6300 3800
@@
 F 0 "U103" H 9300 4400 60  0000 C CNN
 F 1 "CONN_SMA_2GND" H 9650 4500 60  0000 C CNN
-F 2 "vna_footprints:142-0721-882_sma_cutout" H 9600 4200 60  0001 C CNN
+F 2 "vna_footprints:SMA_CPW_1MM_.2MM" H 9600 4200 60  0001 C CNN
 F 3 "" H 9600 4200 60  0000 C CNN
 	1    9600 4200
@@
 F 0 "U102" H 9300 3550 60  0000 C CNN
 F 1 "CONN_SMA_2GND" H 9650 3650 60  0000 C CNN
-F 2 "vna_footprints:142-0721-882_sma_cutout" H 9600 3350 60  0001 C CNN
+F 2 "vna_footprints:SMA_CPW_1MM_.2MM" H 9600 3350 60  0001 C CNN
 F 3 "" H 9600 3350 60  0000 C CNN
 	1    9600 3350
