File: breakouts/switch_breakout/switch_breakout.sch (KiCad schematic (older format))
At the start: 10 parts, among them P1 CONN_01X03, U101 CONN_SMA_2GND, U102 CONN_SMA_2GND, U103 CONN_SMA_2GND, U3 PE42521

Commit message: switched switch board to be coplanar waveguide fed
Parts:
- U101, U102, U103: footprint vna_footprints:142-0721-882_sma_cutout -> vna_footprints:SMA_CPW_1MM_.2MM
Changed lines of the file:
@@
 	6300 5750 6300 5350
 $Comp
-L GND #PWR111
+L GND #PWR01
 U 1 1 56AEF357
 P 6400 5450
-F 0 "#PWR111" H 6400 5200 50  0001 C CNN
+F 0 "#PWR01" H 6400 5200 50  0001 C CNN
 F 1 "GND" H 6400 5300 50  0000 C CNN
 F 2 "" H 6400 5450 50  0000 C CNN
@@
 $EndComp
 $Comp
-L GND #PWR113
+L GND #PWR02
 U 1 1 56AEF39E
 P 6500 5450
-F 0 "#PWR113" H 6500 5200 50  0001 C CNN
+F 0 "#PWR02" H 6500 5200 50  0001 C CNN
 F 1 "GND" H 6500 5300 50  0000 C CNN
 F 2 "" H 6500 5450 50  0000 C CNN
@@
 $EndComp
 $Comp
-L GND #PWR109
+L GND #PWR03
 U 1 1 56AEF4BB
 P 6200 5450
-F 0 "#PWR109" H 6200 5200 50  0001 C CNN
+F 0 "#PWR03" H 6200 5200 50  0001 C CNN
 F 1 "GND" H 6200 5300 50  0000 C CNN
 F 2 "" H 6200 5450 50  0000 C CNN
@@
 	6500 5450 6500 5350
 $Comp
-L GND #PWR112
+L GND #PWR04
 U 1 1 56AEF535
 P 6500 3900
-F 0 "#PWR112" H 6500 3650 50  0001 C CNN
+F 0 "#PWR04" H 6500 3650 50  0001 C CNN
 F 1 "GND" H 6500 3750 50  0000 C CNN
 F 2 "" H 6500 3900 50  0000 C CNN
@@
 	6500 3900 6500 4050
 $Comp
-L GND #PWR110
+L GND #PWR05
 U 1 1 56AEF5AD
 P 6400 3900
-F 0 "#PWR110" H 6400 3650 50  0001 C CNN
+F 0 "#PWR05" H 6400 3650 50  0001 C CNN
 F 1 "GND" H 6400 3750 50  0000 C CNN
 F 2 "" H 6400 3900 50  0000 C CNN
@@
 	6400 3900 6400 4050
 $Comp
-L GND #PWR108
+L GND #PWR06
 U 1 1 56AEF5EA
 P 6200 3900
-F 0 "#PWR108" H 6200 3650 50  0001 C CNN
+F 0 "#PWR06" H 6200 3650 50  0001 C CNN
 F 1 "GND" H 6200 3750 50  0000 C CNN
 F 2 "" H 6200 3900 50  0000 C CNN
@@
 	6200 3900 6200 4050
 $Comp
-L GND #PWR115
+L GND #PWR07
 U 1 1 56AEF628
 P 7100 4550
-F 0 "#PWR115" H 7100 4300 50  0001 C CNN
+F 0 "#PWR07" H 7100 4300 50  0001 C CNN
 F 1 "GND" H 7100 4400 50  0000 C CNN
 F 2 "" H 7100 4550 50  0000 C CNN
@@
 	7000 4550 7100 4550
 $Comp
-L GND #PWR116
+L GND #PWR08
 U 1 1 56AEF667
 P 7100 4750
-F 0 "#PWR116" H 7100 4500 50  0001 C CNN
+F 0 "#PWR08" H 7100 4500 50  0001 C CNN
 F 1 "GND" H 7100 4600 50  0000 C CNN
 F 2 "" H 7100 4750 50  0000 C CNN
@@
 	7100 4750 7000 4750
 $Comp
-L GND #PWR117
+L GND #PWR09
 U 1 1 56AEF6A7
 P 7100 4850
-F 0 "#PWR117" H 7100 4600 50  0001 C CNN
+F 0 "#PWR09" H 7100 4600 50  0001 C CNN
 F 1 "GND" H 7100 4700 50  0000 C CNN
 F 2 "" H 7100 4850 50  0000 C CNN
@@
 	7100 4850 7000 4850
 $Comp
-L GND #PWR106
+L GND #PWR010
 U 1 1 56AEF70C
 P 5600 4550
-F 0 "#PWR106" H 5600 4300 50  0001 C CNN
+F 0 "#PWR010" H 5600 4300 50  0001 C CNN
 F 1 "GND" H 5600 4400 50  0000 C CNN
 F 2 "" H 5600 4550 50  0000 C CNN
@@
 	5600 4550 5700 4550
 $Comp
-L GND #PWR107
+L GND #PWR011
 U 1 1 56AEF771
 P 5600 4750
-F 0 "#PWR107" H 5600 4500 50  0001 C CNN
+F 0 "#PWR011" H 5600 4500 50  0001 C CNN
 F 1 "GND" H 5600 4600 50  0000 C CNN
 F 2 "" H 5600 4750 50  0000 C CNN
@@
 	5700 4850 4400 4850
 $Comp
-L GND #PWR103
+L GND #PWR012
 U 1 1 56AF1A38
 P 4550 4750
-F 0 "#PWR103" H 4550 4500 50  0001 C CNN
+F 0 "#PWR012" H 4550 4500 50  0001 C CNN
 F 1 "GND" H 4550 4600 50  0000 C CNN
 F 2 "" H 4550 4750 50  0000 C CNN
@@
 $EndComp
 $Comp
-L GND #PWR104
+L GND #PWR013
 U 1 1 56AF1B84
 P 4650 5300
-F 0 "#PWR104" H 4650 5050 50  0001 C CNN
+F 0 "#PWR013" H 4650 5050 50  0001 C CNN
 F 1 "GND" H 4650 5150 50  0000 C CNN
 F 2 "" H 4650 5300 50  0000 C CNN
@@
 Connection ~ 4650 4850
 $Comp
-L GND #PWR105
+L GND #PWR014
 U 1 1 56AF1C5F
 P 5000 5300
-F 0 "#PWR105" H 5000 5050 50  0001 C CNN
+F 0 "#PWR014" H 5000 5050 50  0001 C CNN
 F 1 "GND" H 5000 5150 50  0000 C CNN
 F 2 "" H 5000 5300 50  0000 C CNN
@@
 Connection ~ 5000 4850
 $Comp
-L GND #PWR114
+L GND #PWR015
 U 1 1 56CE6531
 P 7100 4450
-F 0 "#PWR114" H 7100 4200 50  0001 C CNN
+F 0 "#PWR015" H 7100 4200 50  0001 C CNN
 F 1 "GND" H 7100 4300 50  0000 C CNN
 F 2 "" H 7100 4450 50  0000 C CNN
@@
 F 0 "U101" H 2450 3550 60  0000 C CNN
 F 1 "CONN_SMA_2GND" H 2800 3650 60  0000 C CNN
-F 2 "vna_footprints:142-0721-882_sma_cutout" H 2750 3350 60  0001 C CNN
+F 2 "vna_footprints:SMA_CPW_1MM_.2MM" H 2750 3350 60  0001 C CNN
 F 3 "" H 2750 3350 60  0000 C CNN
 	1    2750 3350
@@
 $EndComp
 $Comp
-L GND #PWR101
+L GND #PWR016
 U 1 1 576CF63E
 P 2750 3900
-F 0 "#PWR101" H 2750 3650 50  0001 C CNN
+F 0 "#PWR016" H 2750 3650 50  0001 C CNN
 F 1 "GND" H 2750 3750 50  0000 C CNN
 F 2 "" H 2750 3900 50  0000 C CNN
@@
 F 0 "U102" H 2450 5950 60  0000 C CNN
 F 1 "CONN_SMA_2GND" H 2800 6050 60  0000 C CNN
-F 2 "vna_footprints:142-0721-882_sma_cutout" H 2750 5750 60  0001 C CNN
+F 2 "vna_footprints:SMA_CPW_1MM_.2MM" H 2750 5750 60  0001 C CNN
 F 3 "" H 2750 5750 60  0000 C CNN
 	1    2750 5750
@@
 $EndComp
 $Comp
-L GND #PWR102
+L GND #PWR017
 U 1 1 576CF7CE
 P 2750 6300
-F 0 "#PWR102" H 2750 6050 50  0001 C CNN
+F 0 "#PWR017" H 2750 6050 50  0001 C CNN
 F 1 "GND" H 2750 6150 50  0000 C CNN
 F 2 "" H 2750 6300 50  0000 C CNN
@@
 F 0 "U103" H 8850 4850 60  0000 C CNN
 F 1 "CONN_SMA_2GND" H 9200 4950 60  0000 C CNN
-F 2 "vna_footprints:142-0721-882_sma_cutout" H 9150 4650 60  0001 C CNN
+F 2 "vna_footprints:SMA_CPW_1MM_.2MM" H 9150 4650 60  0001 C CNN
 F 3 "" H 9150 4650 60  0000 C CNN
 	1    9150 4650
@@
 $EndComp
 $Comp
-L GND #PWR118
+L GND #PWR018
 U 1 1 576CF931
 P 9150 5200
-F 0 "#PWR118" H 9150 4950 50  0001 C CNN
+F 0 "#PWR018" H 9150 4950 50  0001 C CNN
 F 1 "GND" H 9150 5050 50  0000 C CNN
 F 2 "" H 9150 5200 50  0000 C CNN
