File: hardware/frequency_synth/attenuator.sch (KiCad schematic (older format))
At the start: 31 parts, among them U401 LTC1983, U402 HMC424, U403 74HC04_FULL

Commit message: modified mixer breakout to work with ltc5548, moved to soldermask defined pads
Parts:
- D401, D402, D403, D404, D405, D406: value 3.3V -> 5.1V
Changed lines of the file:
@@
 P 9800 1900
 F 0 "D404" H 9800 2000 50  0000 C CNN
-F 1 "3.3V" H 9800 1800 50  0000 C CNN
+F 1 "5.1V" H 9800 1800 50  0000 C CNN
 F 2 "Diodes_SMD:SOD-123" H 9800 1900 50  0001 C CNN
 F 3 "" H 9800 1900 50  0000 C CNN
@@
 P 9800 2100
 F 0 "D405" H 9800 2200 50  0000 C CNN
-F 1 "3.3V" H 9800 2000 50  0000 C CNN
+F 1 "5.1V" H 9800 2000 50  0000 C CNN
 F 2 "Diodes_SMD:SOD-123" H 9800 2100 50  0001 C CNN
 F 3 "" H 9800 2100 50  0000 C CNN
@@
 P 9800 2300
 F 0 "D406" H 9800 2400 50  0000 C CNN
-F 1 "3.3V" H 9800 2200 50  0000 C CNN
+F 1 "5.1V" H 9800 2200 50  0000 C CNN
 F 2 "Diodes_SMD:SOD-123" H 9800 2300 50  0001 C CNN
 F 3 "" H 9800 2300 50  0000 C CNN
@@
 P 6250 2000
 F 0 "D402" H 6250 2100 50  0000 C CNN
-F 1 "3.3V" H 6250 1900 50  0000 C CNN
+F 1 "5.1V" H 6250 1900 50  0000 C CNN
 F 2 "Diodes_SMD:SOD-123" H 6250 2000 50  0001 C CNN
 F 3 "" H 6250 2000 50  0000 C CNN
@@
 P 6250 2200
 F 0 "D403" H 6250 2300 50  0000 C CNN
-F 1 "3.3V" H 6250 2100 50  0000 C CNN
+F 1 "5.1V" H 6250 2100 50  0000 C CNN
 F 2 "Diodes_SMD:SOD-123" H 6250 2200 50  0001 C CNN
 F 3 "" H 6250 2200 50  0000 C CNN
@@
 P 6250 1800
 F 0 "D401" H 6250 1900 50  0000 C CNN
-F 1 "3.3V" H 6250 1700 50  0000 C CNN
+F 1 "5.1V" H 6250 1700 50  0000 C CNN
 F 2 "Diodes_SMD:SOD-123" H 6250 1800 50  0001 C CNN
 F 3 "" H 6250 1800 50  0000 C CNN

Commit message: fixed footprints for filters on synth board
Parts:
- U403: symbol 74HC04_FULL -> 74HC04_FULL-RESCUE-frequency_synth
Changed lines of the file:
@@
 EESchema Schematic File Version 2
+LIBS:frequency_synth-rescue
 LIBS:power
 LIBS:device
@@
 $EndComp
 $Comp
-L GND #PWR0107
+L GND #PWR0105
 U 1 1 572AE6C7
 P 8800 1800
-F 0 "#PWR0107" H 8800 1550 50  0001 C CNN
+F 0 "#PWR0105" H 8800 1550 50  0001 C CNN
 F 1 "GND" H 8800 1650 50  0000 C CNN
 F 2 "" H 8800 1800 50  0000 C CNN
@@
 	8800 1800 8550 1800
 $Comp
-L VEE #PWR0108
+L VEE #PWR0106
 U 1 1 572AE6C8
 P 7000 2400
-F 0 "#PWR0108" H 7000 2250 50  0001 C CNN
+F 0 "#PWR0106" H 7000 2250 50  0001 C CNN
 F 1 "VEE" H 7000 2550 50  0000 C CNN
 F 2 "" H 7000 2400 50  0000 C CNN
@@
 $EndComp
 $Comp
-L GND #PWR0109
+L GND #PWR0107
 U 1 1 572AE6CA
 P 7350 2800
-F 0 "#PWR0109" H 7350 2550 50  0001 C CNN
+F 0 "#PWR0107" H 7350 2550 50  0001 C CNN
 F 1 "GND" H 7350 2650 50  0000 C CNN
 F 2 "" H 7350 2800 50  0000 C CNN
@@
 	9450 1300 9450 1150
 $Comp
-L VEE #PWR0110
+L VEE #PWR0108
 U 1 1 572AE6D7
 P 6550 1150
-F 0 "#PWR0110" H 6550 1000 50  0001 C CNN
+F 0 "#PWR0108" H 6550 1000 50  0001 C CNN
 F 1 "VEE" H 6550 1300 50  0000 C CNN
 F 2 "" H 6550 1150 50  0000 C CNN
@@
 $EndComp
 $Comp
-L VEE #PWR0111
+L VEE #PWR0109
 U 1 1 572AE6D8
 P 6650 1150
-F 0 "#PWR0111" H 6650 1000 50  0001 C CNN
+F 0 "#PWR0109" H 6650 1000 50  0001 C CNN
 F 1 "VEE" H 6650 1300 50  0000 C CNN
 F 2 "" H 6650 1150 50  0000 C CNN
@@
 $EndComp
 $Comp
-L VEE #PWR0112
+L VEE #PWR0110
 U 1 1 572AE6D9
 P 6750 1150
-F 0 "#PWR0112" H 6750 1000 50  0001 C CNN
+F 0 "#PWR0110" H 6750 1000 50  0001 C CNN
 F 1 "VEE" H 6750 1300 50  0000 C CNN
 F 2 "" H 6750 1150 50  0000 C CNN
@@
 $EndComp
 $Comp
-L VEE #PWR0113
+L VEE #PWR0111
 U 1 1 572AE6DA
 P 9250 1150
-F 0 "#PWR0113" H 9250 1000 50  0001 C CNN
+F 0 "#PWR0111" H 9250 1000 50  0001 C CNN
 F 1 "VEE" H 9250 1300 50  0000 C CNN
 F 2 "" H 9250 1150 50  0000 C CNN
@@
 $EndComp
 $Comp
-L VEE #PWR0114
+L VEE #PWR0112
 U 1 1 572AE6DB
 P 9350 1150
-F 0 "#PWR0114" H 9350 1000 50  0001 C CNN
+F 0 "#PWR0112" H 9350 1000 50  0001 C CNN
 F 1 "VEE" H 9350 1300 50  0000 C CNN
 F 2 "" H 9350 1150 50  0000 C CNN
@@
 $EndComp
 $Comp
-L VEE #PWR0115
+L VEE #PWR0113
 U 1 1 572AE6DC
 P 9450 1150
-F 0 "#PWR0115" H 9450 1000 50  0001 C CNN
+F 0 "#PWR0113" H 9450 1000 50  0001 C CNN
 F 1 "VEE" H 9450 1300 50  0000 C CNN
 F 2 "" H 9450 1150 50  0000 C CNN
@@
 	5800 5250 6450 5250
 $Comp
-L GND #PWR0116
+L GND #PWR0114
 U 1 1 572AE6DF
 P 5950 5150
-F 0 "#PWR0116" H 5950 4900 50  0001 C CNN
+F 0 "#PWR0114" H 5950 4900 50  0001 C CNN
 F 1 "GND" H 5950 5000 50  0000 C CNN
 F 2 "" H 5950 5150 50  0000 C CNN
@@
 	5950 5150 5800 5150
 $Comp
-L GND #PWR0117
+L GND #PWR0115
 U 1 1 572AE6E0
 P 5950 5350
-F 0 "#PWR0117" H 5950 5100 50  0001 C CNN
+F 0 "#PWR0115" H 5950 5100 50  0001 C CNN
 F 1 "GND" H 5950 5200 50  0000 C CNN
 F 2 "" H 5950 5350 50  0000 C CNN
@@
 	5950 5350 5800 5350
 $Comp
-L GND #PWR0118
+L GND #PWR0116
 U 1 1 572AE6E1
 P 5450 6050
-F 0 "#PWR0118" H 5450 5800 50  0001 C CNN
+F 0 "#PWR0116" H 5450 5800 50  0001 C CNN
 F 1 "GND" H 5450 5900 50  0000 C CNN
 F 2 "" H 5450 6050 50  0000 C CNN
@@
 	5450 6050 5450 5900
 $Comp
-L GND #PWR0119
+L GND #PWR0117
 U 1 1 572AE6E2
 P 4450 5350
-F 0 "#PWR0119" H 4450 5100 50  0001 C CNN
+F 0 "#PWR0117" H 4450 5100 50  0001 C CNN
 F 1 "GND" H 4450 5200 50  0000 C CNN
 F 2 "" H 4450 5350 50  0000 C CNN
@@
 $EndComp
 $Comp
-L GND #PWR0120
+L GND #PWR0118
 U 1 1 572AE6E3
 P 4450 5150
-F 0 "#PWR0120" H 4450 4900 50  0001 C CNN
+F 0 "#PWR0118" H 4450 4900 50  0001 C CNN
 F 1 "GND" H 4450 5000 50  0000 C CNN
 F 2 "" H 4450 5150 50  0000 C CNN
@@
 	4450 5350 4600 5350
 $Comp
-L VEE #PWR0121
+L VEE #PWR0119
 U 1 1 572AE6E4
 P 5150 3800
-F 0 "#PWR0121" H 5150 3650 50  0001 C CNN
+F 0 "#PWR0119" H 5150 3650 50  0001 C CNN
 F 1 "VEE" H 5150 3950 50  0000 C CNN
 F 2 "" H 5150 3800 50  0000 C CNN
@@
 $EndComp
 $Comp
-L GND #PWR0122
+L GND #PWR0120
 U 1 1 572AE6E6
 P 5350 4300
-F 0 "#PWR0122" H 5350 4050 50  0001 C CNN
+F 0 "#PWR0120" H 5350 4050 50  0001 C CNN
 F 1 "GND" H 5350 4150 50  0000 C CNN
 F 2 "" H 5350 4300 50  0000 C CNN
@@
 	5050 5900 5050 6350
 $Comp
-L GND #PWR0123
+L GND #PWR0121
 U 1 1 572AE6E8
 P 1200 4050
-F 0 "#PWR0123" H 1200 3800 50  0001 C CNN
+F 0 "#PWR0121" H 1200 3800 50  0001 C CNN
 F 1 "GND" H 1200 3900 50  0000 C CNN
 F 2 "" H 1200 4050 50  0000 C CNN
@@
 $EndComp
 $Comp
-L +5V #PWR0124
+L +5V #PWR0122
 U 1 1 572AE6EA
 P 1450 3850
-F 0 "#PWR0124" H 1450 3700 50  0001 C CNN
+F 0 "#PWR0122" H 1450 3700 50  0001 C CNN
 F 1 "+5V" H 1450 3990 50  0000 C CNN
 F 2 "" H 1450 3850 50  0000 C CNN
@@
 	1450 3850 1100 3850
 $Comp
-L VEE #PWR0125
+L VEE #PWR0123
 U 1 1 572AE6EB
 P 1250 2450
-F 0 "#PWR0125" H 1250 2300 50  0001 C CNN
+F 0 "#PWR0123" H 1250 2300 50  0001 C CNN
 F 1 "VEE" H 1250 2600 50  0000 C CNN
 F 2 "" H 1250 2450 50  0000 C CNN
@@
 $EndComp
 $Comp
-L +5V #PWR0126
+L +5V #PWR0124
 U 1 1 572AE6EC
 P 2150 1600
-F 0 "#PWR0126" H 2150 1450 50  0001 C CNN
+F 0 "#PWR0124" H 2150 1450 50  0001 C CNN
 F 1 "+5V" H 2150 1740 50  0000 C CNN
 F 2 "" H 2150 1600 50  0000 C CNN
@@
 	3550 2550 3450 2550
 $Comp
-L GND #PWR0127
+L GND #PWR0125
 U 1 1 572AE6EE
 P 3600 2450
-F 0 "#PWR0127" H 3600 2200 50  0001 C CNN
+F 0 "#PWR0125" H 3600 2200 50  0001 C CNN
 F 1 "GND" H 3600 2300 50  0000 C CNN
 F 2 "" H 3600 2450 50  0000 C CNN
@@
 $EndComp
 $Comp
-L GND #PWR0128
+L GND #PWR0126
 U 1 1 572AE6F0
 P 1900 2900
-F 0 "#PWR0128" H 1900 2650 50  0001 C CNN
+F 0 "#PWR0126" H 1900 2650 50  0001 C CNN
 F 1 "GND" H 1900 2750 50  0000 C CNN
 F 2 "" H 1900 2900 50  0000 C CNN
@@
 Connection ~ 1900 2450
 $Comp
-L GND #PWR0129
+L GND #PWR0127
 U 1 1 572AE6F1
 P 1900 2200
-F 0 "#PWR0129" H 1900 1950 50  0001 C CNN
+F 0 "#PWR0127" H 1900 1950 50  0001 C CNN
 F 1 "GND" H 1900 2050 50  0000 C CNN
 F 2 "" H 1900 2200 50  0000 C CNN
@@
 $EndComp
 $Comp
-L GND #PWR0130
+L GND #PWR0128
 U 1 1 572AE6F4
 P 1650 2200
-F 0 "#PWR0130" H 1650 1950 50  0001 C CNN
+F 0 "#PWR0128" H 1650 1950 50  0001 C CNN
 F 1 "GND" H 1650 2050 50  0000 C CNN
 F 2 "" H 1650 2200 50  0000 C CNN
@@
 $EndComp
 $Comp
-L GND #PWR0131
+L GND #PWR0129
 U 1 1 572AE6F6
 P 5650 4300
-F 0 "#PWR0131" H 5650 4050 50  0001 C CNN
+F 0 "#PWR0129" H 5650 4050 50  0001 C CNN
 F 1 "GND" H 5650 4150 50  0000 C CNN
 F 2 "" H 5650 4300 50  0000 C CNN
@@
 $EndComp
 $Comp
-L GND #PWR0132
+L GND #PWR0130
 U 1 1 572AE6F8
 P 1350 2200
-F 0 "#PWR0132" H 1350 1950 50  0001 C CNN
+F 0 "#PWR0130" H 1350 1950 50  0001 C CNN
 F 1 "GND" H 1350 2050 50  0000 C CNN
 F 2 "" H 1350 2200 50  0000 C CNN
@@
 ATT_RFOUT
 $Comp
-L 74HC04_FULL U403
+L 74HC04_FULL-RESCUE-frequency_synth U403
 U 1 1 572BDAD2
 P 8100 2100
+AR Path="/572BDAD2" Ref="U403"  Part="1"
+AR Path="/572AE3BA/572BDAD2" Ref="U403"  Part="1"
 F 0 "U403" H 7800 2700 60  0000 C CNN
 F 1 "74HC04_FULL" H 7900 2600 60  0000 C CNN
