File: hardware/frequency_synth/connectors_mcu.sch (KiCad schematic (older format))
At the start: 22 parts, among them P1001 CONN_01X02, Q1001 DMG2305UX, U1001 boosterpack_ti, U1002 CONN_SMA_2GND, U1003 ADM7150, U1004 picture

Commit message: finished vna port switch/multiplier board
Parts:
- D1001, D1002: symbol LED -> LED-RESCUE-frequency_synth
Changed lines of the file:
@@
 FILTC_0
 $Comp
-L LED D1002
+L LED-RESCUE-frequency_synth D1002
 U 1 1 572E0F0F
 P 5300 1100
@@
 $EndComp
 $Comp
-L LED D1001
+L LED-RESCUE-frequency_synth D1001
 U 1 1 572C5E57
 P 4850 1100
