File: hardware/frequency_synth_lowcost/filter_bank.sch (KiCad schematic (older format))
At the start: 18 parts, among them U301 PE42540, U302 PE42540, U303 PE42540

Commit message: work on next revision synth
Parts:
- FI301, FI302, FI303, FI304, FI305, FI306: footprint vna_footprints:FV1206 -> vna_footprints:FV1206-narrow
Changed lines of the file:
@@
 F 0 "FI301" H 6550 8650 50  0000 C CNN
 F 1 "LFCN-6000D+" H 6800 8352 50  0000 C CNN
-F 2 "vna_footprints:FV1206" H 6400 8500 50  0001 C CNN
+F 2 "vna_footprints:FV1206-narrow" H 6400 8500 50  0001 C CNN
 F 3 "" H 6400 8500 50  0000 C CNN
 	1    6400 8500
@@
 F 0 "FI302" H 6500 7900 50  0000 C CNN
 F 1 "LFCN-4400+" H 6750 7602 50  0000 C CNN
-F 2 "vna_footprints:FV1206" H 6350 7750 50  0001 C CNN
+F 2 "vna_footprints:FV1206-narrow" H 6350 7750 50  0001 C CNN
 F 3 "" H 6350 7750 50  0000 C CNN
 	1    6350 7750
@@
 F 0 "FI303" H 6700 5500 50  0000 C CNN
 F 1 "LFCN-3400+" H 6950 5202 50  0000 C CNN
-F 2 "vna_footprints:FV1206" H 6550 5350 50  0001 C CNN
+F 2 "vna_footprints:FV1206-narrow" H 6550 5350 50  0001 C CNN
 F 3 "" H 6550 5350 50  0000 C CNN
 	1    6550 5350
@@
 F 0 "FI304" H 6650 4700 50  0000 C CNN
 F 1 "LFCN-2250+" H 6900 4402 50  0000 C CNN
-F 2 "vna_footprints:FV1206" H 6500 4550 50  0001 C CNN
+F 2 "vna_footprints:FV1206-narrow" H 6500 4550 50  0001 C CNN
 F 3 "" H 6500 4550 50  0000 C CNN
 	1    6500 4550
@@
 F 0 "FI305" H 6650 3750 50  0000 C CNN
 F 1 "LFCN-1450+" H 6900 3452 50  0000 C CNN
-F 2 "vna_footprints:FV1206" H 6500 3600 50  0001 C CNN
+F 2 "vna_footprints:FV1206-narrow" H 6500 3600 50  0001 C CNN
 F 3 "" H 6500 3600 50  0000 C CNN
 	1    6500 3600
@@
 F 0 "FI306" H 6650 2700 50  0000 C CNN
 F 1 "LFCN-1000+" H 6900 2402 50  0000 C CNN
-F 2 "vna_footprints:FV1206" H 6500 2550 50  0001 C CNN
+F 2 "vna_footprints:FV1206-narrow" H 6500 2550 50  0001 C CNN
 F 3 "" H 6500 2550 50  0000 C CNN
 	1    6500 2550
