File: hardware/frequency_synth_lowcost/frequency_synth.kicad_pcb (KiCad board)
At the start: 4 copper layers, 97.1 x 32.8 mm, 137 parts, among them P601 CONN_02X10, Q1001 DMG2305UX, U1002 CONN_SMA_2GND, U1003 ADM7150, U1004 picture, U201 CONN_SMA_2GND, U202 LMX2592, U301 PE42540, U302 PE42540, U303 PE42540, U501 PE43705, U901 LMK61E2

Commit message: work on next revision synth
Parts:
- removed R220, R221, R226, R227, R506, R507, R508, R509, R510, R511, R512: 0, Resistors_SMD:R_0402
- removed R505: 10k, Resistors_SMD:R_0402
- FI301, FI302, FI303, FI304, FI305, FI306: footprint vna_footprints:FV1206 -> vna_footprints:FV1206-narrow
- moved R603 100.2 mm to (170.0, 93.0), turned to 180 degrees
- moved R602 90.8 mm to (170.0, 105.8)
- moved R601 88.9 mm to (170.2, 101.0), turned to 180 degrees
- moved Q1001 80.2 mm to (176.0, 81.5), turned to 180 degrees
- moved R1003 78.8 mm to (179.2, 81.0), turned to 90 degrees
- moved C205 68.8 mm to (200.5, 93.8), turned to 90 degrees
- moved R304 68.4 mm to (170.2, 109.0), turned to 180 degrees
- moved R303 67.0 mm to (170.3, 107.5), turned to 180 degrees
- moved L201 65.2 mm to (195.2, 96.3), turned to 90 degrees
- moved C201 62.7 mm to (199.2, 101.2)
- moved L204 61.1 mm to (197.2, 101.5), turned to 270 degrees
- moved C203 55.9 mm to (204.8, 104.8), turned to 90 degrees
- moved R502 49.4 mm to (236.0, 93.0), turned to 90 degrees
- moved R504 48.4 mm to (228.0, 96.2), turned to 270 degrees
- moved R501 41.2 mm to (234.5, 93.0), turned to 90 degrees
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Connections:
- C228 pad 1: Net-(C228-Pad1) -> /filter bank/RFINB
- C229 pad 1: Net-(C229-Pad1) -> /filter bank/RFINA
- C230 pad 1: Net-(C230-Pad1) -> /filter bank/RFIND
- C231 pad 1: Net-(C231-Pad1) -> /filter bank/RFINC
- R222 pad 1: Net-(C228-Pad1) -> /filter bank/RFINB
- R223 pad 1: Net-(C230-Pad1) -> /filter bank/RFIND
- R224 pad 2: Net-(C229-Pad1) -> /filter bank/RFINA
- R225 pad 2: Net-(C231-Pad1) -> /filter bank/RFINC
- R501 pad 1: /ATT_SI -> /attenuator/SI
- R502 pad 1: /ATT_CLK -> /attenuator/CLK
- R503 pad 1: /ATT_LE -> /attenuator/LE
- U501 pad 23: /ATT_LE -> /attenuator/LE
- U501 pad 24: /ATT_CLK -> /attenuator/CLK
- U501 pad 25: /ATT_SI -> /attenuator/SI
- U501 pad 26: Net-(R512-Pad2) -> GND
- U501 pad 27: Net-(R511-Pad2) -> GND
- U501 pad 28: Net-(R510-Pad2) -> GND
- U501 pad 29: Net-(R509-Pad2) -> GND
- U501 pad 30: Net-(R508-Pad2) -> GND
- U501 pad 31: Net-(R507-Pad2) -> GND
- U501 pad 32: Net-(R506-Pad2) -> GND
