File: hardware/frequency_synth_lowcost/synth.sch (KiCad schematic (older format))
At the start: 70 parts, among them U201 CONN_SMA_2GND, U202 LMX2592

Commit message: work on next revision synth
Parts:
- removed R220, R221, R226, R227: 0, Resistors_SMD:R_0402, symbol R_Small
Connections:
- net RFOUTAM: now also C231.1, R225.2
- net RFOUTAP: now also C230.1, R223.1
- net RFOUTBM: now also C228.1, R222.1
- net RFOUTBP: now also C229.1, R224.2
Changed lines of the file:
@@
-$EndComp
-$Comp
-L R_Small R221
-U 1 1 572AD541
-P 14150 7900
-F 0 "R221" H 14180 7920 50  0000 L CNN
-F 1 "0" H 14180 7860 50  0000 L CNN
-F 2 "Resistors_SMD:R_0402" H 14150 7900 50  0001 C CNN
-F 3 "" H 14150 7900 50  0000 C CNN
-	1    14150 7900
-	0    -1   -1   0
-$EndComp
-$Comp
-L R_Small R220
-U 1 1 572AD542
-P 14150 6000
-F 0 "R220" H 14180 6020 50  0000 L CNN
-F 1 "0" H 14180 5960 50  0000 L CNN
-F 2 "Resistors_SMD:R_0402" H 14150 6000 50  0001 C CNN
-F 3 "" H 14150 6000 50  0000 C CNN
-	1    14150 6000
-	0    -1   -1   0
 $EndComp
 $Comp
@@
 Connection ~ 7800 10000
 Wire Wire Line
-	13700 7900 14050 7900
+	13700 7900 14750 7900
 Wire Wire Line
 	12500 7900 13500 7900
 Wire Wire Line
-	13700 6000 14050 6000
+	13700 6000 14600 6000
 Wire Wire Line
 	12500 6000 13500 6000
@@
 	13750 4850 13750 4950
 Connection ~ 13050 7900
-Wire Wire Line
-	14250 7900 14750 7900
 Wire Wire Line
 	7900 10250 7900 10600
@@
 Text HLabel 14600 6000 2    60   Input ~ 0
 RFOUTBM
-Wire Wire Line
-	14600 6000 14250 6000
 $Comp
 L R_Small R222
@@
 $EndComp
 $Comp
-L R_Small R227
-U 1 1 5820389B
-P 14200 3800
-F 0 "R227" H 14230 3820 50  0000 L CNN
-F 1 "0" H 14230 3760 50  0000 L CNN
-F 2 "Resistors_SMD:R_0402" H 14200 3800 50  0001 C CNN
-F 3 "" H 14200 3800 50  0000 C CNN
-	1    14200 3800
-	0    -1   -1   0
-$EndComp
-$Comp
-L R_Small R226
-U 1 1 582038A1
-P 14200 1900
-F 0 "R226" H 14230 1920 50  0000 L CNN
-F 1 "0" H 14230 1860 50  0000 L CNN
-F 2 "Resistors_SMD:R_0402" H 14200 1900 50  0001 C CNN
-F 3 "" H 14200 1900 50  0000 C CNN
-	1    14200 1900
-	0    -1   -1   0
-$EndComp
-$Comp
 L L_Small L201
 U 1 1 582038A7
@@
 $EndComp
 Wire Wire Line
-	13750 3800 14100 3800
+	13750 3800 14800 3800
 Wire Wire Line
 	12550 3800 13550 3800
 Wire Wire Line
-	13750 1900 14100 1900
+	13750 1900 14650 1900
 Wire Wire Line
 	12550 1900 13550 1900
@@
 	13800 750  13800 850
 Connection ~ 13100 3800
-Wire Wire Line
-	14300 3800 14800 3800
 $Comp
 L R_Small R219
@@
 Text HLabel 14650 1900 2    60   Input ~ 0
 RFOUTAP
-Wire Wire Line
-	14650 1900 14300 1900
 $Comp
 L R_Small R223
