File: breakouts/cpw_test/cpw_test.sch (KiCad schematic (older format))
At the start: 3 parts, among them P101 CONN_01X01, U101 CONN_SMA_2GND, U102 CONN_SMA_2GND

Commit message: finished vna port switch/multiplier board
Parts:
- removed P101: CONN_01X01, symbol CONN_01X01
- U101, U102: footprint vna_footprints:SMA_CPW_1MM_.2MM -> vna_footprints:SMA_901-10512_30MIL_RT6002_CPW_LAUNCH
Connections:
- wire segments 10 -> 9
Changed lines of the file:
@@
 LIBS:valves
 LIBS:conn_sma_2gnd
+LIBS:cpw_test-cache
 EELAYER 25 0
 EELAYER END
@@
 F 0 "U101" H 3050 2850 60  0000 C CNN
 F 1 "CONN_SMA_2GND" H 3400 2950 60  0000 C CNN
-F 2 "vna_footprints:SMA_CPW_1MM_.2MM" H 3350 2650 60  0001 C CNN
+F 2 "vna_footprints:SMA_901-10512_30MIL_RT6002_CPW_LAUNCH" H 3350 2650 60  0001 C CNN
 F 3 "" H 3350 2650 60  0000 C CNN
 	1    3350 2650
@@
 F 0 "U102" H 4250 2850 60  0000 C CNN
 F 1 "CONN_SMA_2GND" H 4600 2950 60  0000 C CNN
-F 2 "vna_footprints:SMA_CPW_1MM_.2MM" H 4550 2650 60  0001 C CNN
+F 2 "vna_footprints:SMA_901-10512_30MIL_RT6002_CPW_LAUNCH" H 4550 2650 60  0001 C CNN
 F 3 "" H 4550 2650 60  0000 C CNN
 	1    4550 2650
@@
 Wire Wire Line
 	3750 2650 4150 2650
-$Comp
-L CONN_01X01 P101
-U 1 1 577AFB68
-P 3250 3950
-F 0 "P101" H 3250 4050 50  0000 C CNN
-F 1 "CONN_01X01" V 3350 3950 50  0000 C CNN
-F 2 "" H 3250 3950 50  0000 C CNN
-F 3 "" H 3250 3950 50  0000 C CNN
-	1    3250 3950
-	1    0    0    -1
-$EndComp
-$Comp
-L GND #PWR03
-U 1 1 577AFBC3
-P 3000 3950
-F 0 "#PWR03" H 3000 3700 50  0001 C CNN
-F 1 "GND" H 3000 3800 50  0000 C CNN
-F 2 "" H 3000 3950 50  0000 C CNN
-F 3 "" H 3000 3950 50  0000 C CNN
-	1    3000 3950
-	0    1    1    0
-$EndComp
-Wire Wire Line
-	3000 3950 3050 3950
 $EndSCHEMATC
