File: hardware/vna_r0/vna_rf/conn_power.sch (KiCad schematic (older format))
At the start: 0 parts

Commit message: finished vna r0 demod schematic
Parts:
- added D? (x2): LED_Small, symbol LED_Small
- added R? (x2): R_Small, symbol R_Small
- added U? (x2): CONN_SMA_2GND, symbol CONN_SMA_2GND
- added U?: CONN_SMA, symbol CONN_SMA
Connections:
- new net: D?.2 (A), R?.2 (x2)
- new net +3V3: R?.1
- new net -5V: D?.1 (K)
- new net GND: D?.1 (K), R?.1, U?.2 (GND), U?.2 (GND), U?.2 (GND), U?.3 (GND), U?.3 (GND), U?.3 (GND), U?.4 (GND), U?.5 (GND)
- new net PORT1: U?.1 (RF)
- new net PORT2: U?.1 (RF)
- new net SYNTH_REF: U?.1 (RF)
Changed lines of the file:
@@
 LIBS:ltc2630
 LIBS:ltc2054cs5
+LIBS:conn_sma_2gnd
+LIBS:conn_sma
 LIBS:vna_rf-cache
 EELAYER 25 0
@@
 Comment4 ""
 $EndDescr
+$Comp
+L +3V3 #PWR?
+U 1 1 593F1269
+P 3400 2400
+F 0 "#PWR?" H 3400 2250 50  0001 C CNN
+F 1 "+3V3" H 3400 2540 50  0000 C CNN
+F 2 "" H 3400 2400 50  0001 C CNN
+F 3 "" H 3400 2400 50  0001 C CNN
+	1    3400 2400
+	1    0    0    -1
+$EndComp
+$Comp
+L -5V #PWR?
+U 1 1 593F127D
+P 3800 3250
+F 0 "#PWR?" H 3800 3350 50  0001 C CNN
+F 1 "-5V" H 3800 3400 50  0000 C CNN
+F 2 "" H 3800 3250 50  0001 C CNN
+F 3 "" H 3800 3250 50  0001 C CNN
+	1    3800 3250
+	-1   0    0    1
+$EndComp
+$Comp
+L R_Small R?
+U 1 1 593F1291
+P 3400 2650
+F 0 "R?" H 3430 2670 50  0000 L CNN
+F 1 "R_Small" H 3430 2610 50  0000 L CNN
+F 2 "" H 3400 2650 50  0001 C CNN
+F 3 "" H 3400 2650 50  0001 C CNN
+	1    3400 2650
+	1    0    0    -1
+$EndComp
+$Comp
+L LED_Small D?
+U 1 1 593F12E5
+P 3400 3000
+F 0 "D?" H 3350 3125 50  0000 L CNN
+F 1 "LED_Small" H 3225 2900 50  0000 L CNN
+F 2 "" V 3400 3000 50  0001 C CNN
+F 3 "" V 3400 3000 50  0001 C CNN
+	1    3400 3000
+	0    -1   -1   0
+$EndComp
+$Comp
+L GND #PWR?
+U 1 1 593F1346
+P 3400 3250
+F 0 "#PWR?" H 3400 3000 50  0001 C CNN
+F 1 "GND" H 3400 3100 50  0000 C CNN
+F 2 "" H 3400 3250 50  0001 C CNN
+F 3 "" H 3400 3250 50  0001 C CNN
+	1    3400 3250
+	1    0    0    -1
+$EndComp
+Wire Wire Line
+	3400 3100 3400 3250
+Wire Wire Line
+	3400 2750 3400 2900
+Wire Wire Line
+	3400 2400 3400 2550
+$Comp
+L LED_Small D?
+U 1 1 593F150A
+P 3800 3000
+F 0 "D?" H 3750 3125 50  0000 L CNN
+F 1 "LED_Small" H 3625 2900 50  0000 L CNN
+F 2 "" V 3800 3000 50  0001 C CNN
+F 3 "" V 3800 3000 50  0001 C CNN
+	1    3800 3000
+	0    -1   -1   0
+$EndComp
+$Comp
+L R_Small R?
+U 1 1 593F1587
+P 3800 2650
+F 0 "R?" H 3830 2670 50  0000 L CNN
+F 1 "R_Small" H 3830 2610 50  0000 L CNN
+F 2 "" H 3800 2650 50  0001 C CNN
+F 3 "" H 3800 2650 50  0001 C CNN
+	1    3800 2650
+	1    0    0    -1
+$EndComp
+$Comp
+L GND #PWR?
+U 1 1 593F15AF
+P 3800 2400
+F 0 "#PWR?" H 3800 2150 50  0001 C CNN
+F 1 "GND" H 3800 2250 50  0000 C CNN
+F 2 "" H 3800 2400 50  0001 C CNN
+F 3 "" H 3800 2400 50  0001 C CNN
+	1    3800 2400
+	-1   0    0    1
+$EndComp
+Wire Wire Line
+	3800 3250 3800 3100
+Wire Wire Line
+	3800 2900 3800 2750
+Wire Wire Line
+	3800 2550 3800 2400
+$Comp
+L CONN_SMA_2GND U?
+U 1 1 593F48FB
+P 10200 2400
+F 0 "U?" H 9900 2600 60  0000 C CNN
+F 1 "CONN_SMA_2GND" H 10250 2700 60  0000 C CNN
+F 2 "" H 10200 2400 60  0000 C CNN
+F 3 "" H 10200 2400 60  0000 C CNN
+	1    10200 2400
+	-1   0    0    -1
+$EndComp
+$Comp
+L CONN_SMA U?
+U 1 1 593F491A
+P 10250 4800
+F 0 "U?" H 9900 5000 60  0000 C CNN
+F 1 "CONN_SMA" H 10100 5150 60  0000 C CNN
+F 2 "" H 10250 4800 60  0000 C CNN
+F 3 "" H 10250 4800 60  0000 C CNN
+	1    10250 4800
+	1    0    0    -1
+$EndComp
+$Comp
+L GND #PWR?
+U 1 1 593F49C3
+P 10250 5400
+F 0 "#PWR?" H 10250 5150 50  0001 C CNN
+F 1 "GND" H 10250 5250 50  0000 C CNN
+F 2 "" H 10250 5400 50  0001 C CNN
+F 3 "" H 10250 5400 50  0001 C CNN
+	1    10250 5400
+	1    0    0    -1
+$EndComp
+$Comp
+L GND #PWR?
+U 1 1 593F4A3C
+P 10200 2950
+F 0 "#PWR?" H 10200 2700 50  0001 C CNN
+F 1 "GND" H 10200 2800 50  0000 C CNN
+F 2 "" H 10200 2950 50  0001 C CNN
+F 3 "" H 10200 2950 50  0001 C CNN
+	1    10200 2950
+	1    0    0    -1
+$EndComp
+Wire Wire Line
+	10150 2850 10150 2900
+Wire Wire Line
+	10150 2900 10250 2900
+Wire Wire Line
+	10250 2900 10250 2850
+Wire Wire Line
+	10200 2900 10200 2950
+Connection ~ 10200 2900
+Wire Wire Line
+	9800 2400 9550 2400
+Text HLabel 9550 2400 0    60   Input ~ 0
+PORT1
+$Comp
+L CONN_SMA_2GND U?
+U 1 1 593F4C2B
+P 10200 3500
+F 0 "U?" H 9900 3700 60  0000 C CNN
+F 1 "CONN_SMA_2GND" H 10250 3800 60  0000 C CNN
+F 2 "" H 10200 3500 60  0000 C CNN
+F 3 "" H 10200 3500 60  0000 C CNN
+	1    10200 3500
+	-1   0    0    -1
+$EndComp
+$Comp
+L GND #PWR?
+U 1 1 593F4C31
+P 10200 4050
+F 0 "#PWR?" H 10200 3800 50  0001 C CNN
+F 1 "GND" H 10200 3900 50  0000 C CNN
+F 2 "" H 10200 4050 50  0001 C CNN
+F 3 "" H 10200 4050 50  0001 C CNN
+	1    10200 4050
+	1    0    0    -1
+$EndComp
+Wire Wire Line
+	10150 3950 10150 4000
+Wire Wire Line
+	10150 4000 10250 4000
+Wire Wire Line
+	10250 4000 10250 3950
+Wire Wire Line
+	10200 4000 10200 4050
+Connection ~ 10200 4000
+Wire Wire Line
+	9800 3500 9550 3500
+Text HLabel 9550 3500 0    60   Input ~ 0
+PORT2
+Wire Wire Line
+	10100 5250 10100 5300
+Wire Wire Line
+	10100 5300 10400 5300
+Wire Wire Line
+	10400 5300 10400 5250
+Wire Wire Line
+	10200 5250 10200 5300
+Connection ~ 10200 5300
+Wire Wire Line
+	10300 5250 10300 5300
+Connection ~ 10300 5300
+Wire Wire Line
+	10250 5300 10250 5400
+Connection ~ 10250 5300
+Wire Wire Line
+	9700 4800 9450 4800
+Text HLabel 9450 4800 0    60   Input ~ 0
+SYNTH_REF
+Text HLabel 8450 5800 2    60   Input ~ 0
+AMP_5V
+Text HLabel 8450 5650 2    60   Input ~ 0
+PORT_SEL
+Text HLabel 8450 5450 2    60   Input ~ 0
+RFSW_1
+Text HLabel 8450 5350 2    60   Input ~ 0
+RFSW_2
+Text HLabel 7450 5750 2    60   Input ~ 0
+LMX_CE
+Text HLabel 7450 6000 2    60   Input ~ 0
+DAC_CS
+Text HLabel 7450 5400 2    60   Input ~ 0
+SCK
+Text HLabel 7450 5300 2    60   Input ~ 0
+MOSI
+Text HLabel 7450 5650 2    60   Input ~ 0
+LMX_MUXOUT
+Text HLabel 7450 5900 2    60   Input ~ 0
+LMX_CS
+Text HLabel 7450 5200 2    60   Input ~ 0
+MISO
 $EndSCHEMATC

Commit message: finiished schematic for vna r0 rf board
Parts:
- added C? (x3): CP_Small, symbol CP_Small
- added D?: LED_Small, symbol LED_Small
- added J?: CONN_02X10, symbol CONN_02X10
- added R?: R_Small, symbol R_Small
Connections:
- net +3V3: now also C?.1, J?.11 (P11), J?.12 (P12), J?.13 (P13)
- net -5V: now also C?.2
- net AMP_5V: now also C?.1, J?.1 (P1), J?.2 (P2), R?.1
- net DAC_CS: now also J?.18 (P18)
- net GND: now also C?.1, C?.2, C?.2, D?.1 (K), J?.14 (P14), J?.3 (P3), J?.5 (P5), J?.7 (P7)
- net LMX_CE: now also J?.10 (P10)
- net LMX_CS: now also J?.9 (P9)
- net LMX_MUXOUT: now also J?.8 (P8)
- net PORT_SEL: now also J?.16 (P16)
- net RFSW_1: now also J?.19 (P19)
- net RFSW_2: now also J?.20 (P20)
- new net: D?.2 (A), R?.2
- new net DAC_SCK: J?.15 (P15)
- new net DAC_SDI: J?.17 (P17)
- new net LMX_SCK: J?.6 (P6)
- new net LMX_SDI: J?.4 (P4)

Commit message: footprint assignment on vna r0
Parts:
- removed C?: CP_Small, symbol CP_Small
- added C403: 10 uF, Capacitors_SMD:C_0603, symbol C_Small
- C401, C402: renamed from C?; value CP_Small -> 100 uF; footprint (none) -> Capacitors_SMD:c_elec_10x10
- D401, D402, D403: renamed from D?; footprint (none) -> LEDs:LED_0603
- J401: renamed from J?; footprint (none) -> Connect:IDC_Header_Straight_20pins
- R401, R402, R403: renamed from R?; footprint (none) -> Resistors_SMD:R_0402
- U401, U402: renamed from U?; footprint (none) -> vna_footprints:SMA_901-10512_30MIL_OSHFR408_CPW_LAUNCH
- U403: renamed from U?; footprint (none) -> vna_footprints:732511150_sma_thin
Connections:
- net -5V: now also C403.2
- net GND: now also C403.1
Changed lines of the file:
@@
 $EndDescr
 $Comp
-L +3V3 #PWR?
+L +3V3 #PWR0108
 U 1 1 593F1269
 P 3400 2400
-F 0 "#PWR?" H 3400 2250 50  0001 C CNN
+F 0 "#PWR0108" H 3400 2250 50  0001 C CNN
 F 1 "+3V3" H 3400 2540 50  0000 C CNN
 F 2 "" H 3400 2400 50  0001 C CNN
@@
 $EndComp
 $Comp
-L -5V #PWR?
+L -5V #PWR404
 U 1 1 593F127D
 P 3800 3250
-F 0 "#PWR?" H 3800 3350 50  0001 C CNN
+F 0 "#PWR404" H 3800 3350 50  0001 C CNN
 F 1 "-5V" H 3800 3400 50  0000 C CNN
 F 2 "" H 3800 3250 50  0001 C CNN
@@
 $EndComp
 $Comp
-L R_Small R?
+L R_Small R401
 U 1 1 593F1291
 P 3400 2650
-F 0 "R?" H 3430 2670 50  0000 L CNN
+F 0 "R401" H 3430 2670 50  0000 L CNN
 F 1 "R_Small" H 3430 2610 50  0000 L CNN
-F 2 "" H 3400 2650 50  0001 C CNN
+F 2 "Resistors_SMD:R_0402" H 3400 2650 50  0001 C CNN
 F 3 "" H 3400 2650 50  0001 C CNN
 	1    3400 2650
@@
 $EndComp
 $Comp
-L LED_Small D?
+L LED_Small D401
 U 1 1 593F12E5
 P 3400 3000
-F 0 "D?" H 3350 3125 50  0000 L CNN
+F 0 "D401" H 3350 3125 50  0000 L CNN
 F 1 "LED_Small" H 3225 2900 50  0000 L CNN
-F 2 "" V 3400 3000 50  0001 C CNN
+F 2 "LEDs:LED_0603" V 3400 3000 50  0001 C CNN
 F 3 "" V 3400 3000 50  0001 C CNN
 	1    3400 3000
@@
 $EndComp
 $Comp
-L GND #PWR?
+L GND #PWR0109
 U 1 1 593F1346
 P 3400 3250
-F 0 "#PWR?" H 3400 3000 50  0001 C CNN
+F 0 "#PWR0109" H 3400 3000 50  0001 C CNN
 F 1 "GND" H 3400 3100 50  0000 C CNN
 F 2 "" H 3400 3250 50  0001 C CNN
@@
 $EndComp
 $Comp
-L LED_Small D?
+L LED_Small D402
 U 1 1 593F150A
 P 3800 3000
-F 0 "D?" H 3750 3125 50  0000 L CNN
+F 0 "D402" H 3750 3125 50  0000 L CNN
 F 1 "LED_Small" H 3625 2900 50  0000 L CNN
-F 2 "" V 3800 3000 50  0001 C CNN
+F 2 "LEDs:LED_0603" V 3800 3000 50  0001 C CNN
 F 3 "" V 3800 3000 50  0001 C CNN
 	1    3800 3000
@@
 $EndComp
 $Comp
-L R_Small R?
+L R_Small R402
 U 1 1 593F1587
 P 3800 2650
-F 0 "R?" H 3830 2670 50  0000 L CNN
+F 0 "R402" H 3830 2670 50  0000 L CNN
 F 1 "R_Small" H 3830 2610 50  0000 L CNN
-F 2 "" H 3800 2650 50  0001 C CNN
+F 2 "Resistors_SMD:R_0402" H 3800 2650 50  0001 C CNN
 F 3 "" H 3800 2650 50  0001 C CNN
 	1    3800 2650
@@
 $EndComp
 $Comp
-L GND #PWR?
+L GND #PWR0110
 U 1 1 593F15AF
 P 3800 2400
-F 0 "#PWR?" H 3800 2150 50  0001 C CNN
+F 0 "#PWR0110" H 3800 2150 50  0001 C CNN
 F 1 "GND" H 3800 2250 50  0000 C CNN
 F 2 "" H 3800 2400 50  0001 C CNN
@@
 $EndComp
 $Comp
-L CONN_SMA_2GND U?
+L CONN_SMA_2GND U401
 U 1 1 593F48FB
 P 10200 2400
-F 0 "U?" H 9900 2600 60  0000 C CNN
+F 0 "U401" H 9900 2600 60  0000 C CNN
 F 1 "CONN_SMA_2GND" H 10250 2700 60  0000 C CNN
-F 2 "" H 10200 2400 60  0000 C CNN
+F 2 "vna_footprints:SMA_901-10512_30MIL_OSHFR408_CPW_LAUNCH" H 10200 2400 60  0001 C CNN
 F 3 "" H 10200 2400 60  0000 C CNN
 	1    10200 2400
@@
 $EndComp
 $Comp
-L CONN_SMA U?
+L CONN_SMA U403
 U 1 1 593F491A
 P 10250 4800
-F 0 "U?" H 9900 5000 60  0000 C CNN
+F 0 "U403" H 9900 5000 60  0000 C CNN
 F 1 "CONN_SMA" H 10100 5150 60  0000 C CNN
-F 2 "" H 10250 4800 60  0000 C CNN
+F 2 "vna_footprints:732511150_sma_thin" H 10250 4800 60  0001 C CNN
 F 3 "" H 10250 4800 60  0000 C CNN
 	1    10250 4800
@@
 $EndComp
 $Comp
-L GND #PWR?
+L GND #PWR0111
 U 1 1 593F49C3
 P 10250 5400
-F 0 "#PWR?" H 10250 5150 50  0001 C CNN
+F 0 "#PWR0111" H 10250 5150 50  0001 C CNN
 F 1 "GND" H 10250 5250 50  0000 C CNN
 F 2 "" H 10250 5400 50  0001 C CNN
@@
 $EndComp
 $Comp
-L GND #PWR?
+L GND #PWR0112
 U 1 1 593F4A3C
 P 10200 2950
-F 0 "#PWR?" H 10200 2700 50  0001 C CNN
+F 0 "#PWR0112" H 10200 2700 50  0001 C CNN
 F 1 "GND" H 10200 2800 50  0000 C CNN
 F 2 "" H 10200 2950 50  0001 C CNN
@@
 PORT1
 $Comp
-L CONN_SMA_2GND U?
+L CONN_SMA_2GND U402
 U 1 1 593F4C2B
 P 10200 3500
-F 0 "U?" H 9900 3700 60  0000 C CNN
+F 0 "U402" H 9900 3700 60  0000 C CNN
 F 1 "CONN_SMA_2GND" H 10250 3800 60  0000 C CNN
-F 2 "" H 10200 3500 60  0000 C CNN
+F 2 "vna_footprints:SMA_901-10512_30MIL_OSHFR408_CPW_LAUNCH" H 10200 3500 60  0001 C CNN
 F 3 "" H 10200 3500 60  0000 C CNN
 	1    10200 3500
@@
 $EndComp
 $Comp
-L GND #PWR?
+L GND #PWR0113
 U 1 1 593F4C31
 P 10200 4050
-F 0 "#PWR?" H 10200 3800 50  0001 C CNN
+F 0 "#PWR0113" H 10200 3800 50  0001 C CNN
 F 1 "GND" H 10200 3900 50  0000 C CNN
 F 2 "" H 10200 4050 50  0001 C CNN
@@
 LMX_CS
 $Comp
-L CONN_02X10 J?
+L CONN_02X10 J401
 U 1 1 593F9D53
 P 5850 5500
-F 0 "J?" H 5850 6050 50  0000 C CNN
+F 0 "J401" H 5850 6050 50  0000 C CNN
 F 1 "CONN_02X10" V 5850 5500 50  0000 C CNN
-F 2 "" H 5850 4300 50  0001 C CNN
+F 2 "Connect:IDC_Header_Straight_20pins" H 5850 4300 50  0001 C CNN
 F 3 "" H 5850 4300 50  0001 C CNN
 	1    5850 5500
@@
 LMX_SDI
 $Comp
-L CP_Small C?
-U 1 1 59402B31
-P 5850 3850
-F 0 "C?" H 5860 3920 50  0000 L CNN
-F 1 "CP_Small" H 5860 3770 50  0000 L CNN
-F 2 "" H 5850 3850 50  0001 C CNN
-F 3 "" H 5850 3850 50  0001 C CNN
-	1    5850 3850
-	1    0    0    -1
-$EndComp
-$Comp
-L CP_Small C?
+L CP_Small C401
 U 1 1 59402B85
 P 5200 3850
-F 0 "C?" H 5210 3920 50  0000 L CNN
-F 1 "CP_Small" H 5210 3770 50  0000 L CNN
-F 2 "" H 5200 3850 50  0001 C CNN
+F 0 "C401" H 5210 3920 50  0000 L CNN
+F 1 "100 uF" H 5210 3770 50  0000 L CNN
+F 2 "Capacitors_SMD:c_elec_10x10" H 5200 3850 50  0001 C CNN
 F 3 "" H 5200 3850 50  0001 C CNN
 	1    5200 3850
@@
 Connection ~ 5500 5050
 $Comp
-L GND #PWR?
+L GND #PWR0114
 U 1 1 59402D3D
 P 5850 4050
-F 0 "#PWR?" H 5850 3800 50  0001 C CNN
+F 0 "#PWR0114" H 5850 3800 50  0001 C CNN
 F 1 "GND" H 5850 3900 50  0000 C CNN
 F 2 "" H 5850 4050 50  0001 C CNN
@@
 	5850 3950 5850 4050
 $Comp
-L +3V3 #PWR?
+L +3V3 #PWR0115
 U 1 1 59402E68
 P 5850 3600
-F 0 "#PWR?" H 5850 3450 50  0001 C CNN
+F 0 "#PWR0115" H 5850 3450 50  0001 C CNN
 F 1 "+3V3" H 5850 3740 50  0000 C CNN
 F 2 "" H 5850 3600 50  0001 C CNN
@@
 Connection ~ 5200 3550
 $Comp
-L GND #PWR?
+L GND #PWR0116
 U 1 1 59403225
 P 5200 4050
-F 0 "#PWR?" H 5200 3800 50  0001 C CNN
+F 0 "#PWR0116" H 5200 3800 50  0001 C CNN
 F 1 "GND" H 5200 3900 50  0000 C CNN
 F 2 "" H 5200 4050 50  0001 C CNN
@@
 	5200 4050 5200 3950
 $Comp
-L -5V #PWR?
+L -5V #PWR416
 U 1 1 59403473
 P 6300 4050
-F 0 "#PWR?" H 6300 4150 50  0001 C CNN
+F 0 "#PWR416" H 6300 4150 50  0001 C CNN
 F 1 "-5V" H 6300 4200 50  0000 C CNN
 F 2 "" H 6300 4050 50  0001 C CNN
@@
 $EndComp
 $Comp
-L GND #PWR?
+L GND #PWR0117
 U 1 1 594034F6
 P 6300 3600
-F 0 "#PWR?" H 6300 3350 50  0001 C CNN
+F 0 "#PWR0117" H 6300 3350 50  0001 C CNN
 F 1 "GND" H 6300 3450 50  0000 C CNN
 F 2 "" H 6300 3600 50  0001 C CNN
@@
 	-1   0    0    1
 $EndComp
-$Comp
-L CP_Small C?
-U 1 1 59403529
-P 6300 3850
-F 0 "C?" H 6310 3920 50  0000 L CNN
-F 1 "CP_Small" H 6310 3770 50  0000 L CNN
-F 2 "" H 6300 3850 50  0001 C CNN
-F 3 "" H 6300 3850 50  0001 C CNN
-	1    6300 3850
-	1    0    0    -1
-$EndComp
 Wire Wire Line
 	6300 3950 6300 4050
@@
 	6300 3600 6300 3750
 $Comp
-L GND #PWR?
+L GND #PWR0118
 U 1 1 59404F0C
 P 5450 5150
-F 0 "#PWR?" H 5450 4900 50  0001 C CNN
+F 0 "#PWR0118" H 5450 4900 50  0001 C CNN
 F 1 "GND" H 5450 5000 50  0000 C CNN
 F 2 "" H 5450 5150 50  0001 C CNN
@@
 	6250 5150 6100 5150
 $Comp
-L GND #PWR?
+L GND #PWR0119
 U 1 1 59404FB3
 P 5450 5250
-F 0 "#PWR?" H 5450 5000 50  0001 C CNN
+F 0 "#PWR0119" H 5450 5000 50  0001 C CNN
 F 1 "GND" H 5450 5100 50  0000 C CNN
 F 2 "" H 5450 5250 50  0001 C CNN
@@
 	6100 5250 6250 5250
 $Comp
-L GND #PWR?
+L GND #PWR0120
 U 1 1 5940505E
 P 5450 5350
-F 0 "#PWR?" H 5450 5100 50  0001 C CNN
+F 0 "#PWR0120" H 5450 5100 50  0001 C CNN
 F 1 "GND" H 5450 5200 50  0000 C CNN
 F 2 "" H 5450 5350 50  0001 C CNN
@@
 	5500 5450 5600 5450
 $Comp
-L +3V3 #PWR?
+L +3V3 #PWR0121
 U 1 1 594052AB
 P 5500 5600
-F 0 "#PWR?" H 5500 5450 50  0001 C CNN
+F 0 "#PWR0121" H 5500 5450 50  0001 C CNN
 F 1 "+3V3" H 5500 5740 50  0000 C CNN
 F 2 "" H 5500 5600 50  0001 C CNN
@@
 Connection ~ 5550 5600
 $Comp
-L +3V3 #PWR?
+L +3V3 #PWR0122
 U 1 1 5940537D
 P 6250 5550
-F 0 "#PWR?" H 6250 5400 50  0001 C CNN
+F 0 "#PWR0122" H 6250 5400 50  0001 C CNN
 F 1 "+3V3" H 6250 5690 50  0000 C CNN
 F 2 "" H 6250 5550 50  0001 C CNN
@@
 	6250 5550 6100 5550
 $Comp
-L GND #PWR?
+L GND #PWR0123
 U 1 1 594053F3
 P 6200 5650
-F 0 "#PWR?" H 6200 5400 50  0001 C CNN
+F 0 "#PWR0123" H 6200 5400 50  0001 C CNN
 F 1 "GND" H 6200 5500 50  0000 C CNN
 F 2 "" H 6200 5650 50  0001 C CNN
@@
 AMP_5V
 $Comp
-L R_Small R?
+L R_Small R403
 U 1 1 59405912
 P 4300 2650
-F 0 "R?" H 4330 2670 50  0000 L CNN
+F 0 "R403" H 4330 2670 50  0000 L CNN
 F 1 "R_Small" H 4330 2610 50  0000 L CNN
-F 2 "" H 4300 2650 50  0001 C CNN
+F 2 "Resistors_SMD:R_0402" H 4300 2650 50  0001 C CNN
 F 3 "" H 4300 2650 50  0001 C CNN
 	1    4300 2650
@@
 $EndComp
 $Comp
-L LED_Small D?
+L LED_Small D403
 U 1 1 59405918
 P 4300 3000
-F 0 "D?" H 4250 3125 50  0000 L CNN
+F 0 "D403" H 4250 3125 50  0000 L CNN
 F 1 "LED_Small" H 4125 2900 50  0000 L CNN
-F 2 "" V 4300 3000 50  0001 C CNN
+F 2 "LEDs:LED_0603" V 4300 3000 50  0001 C CNN
 F 3 "" V 4300 3000 50  0001 C CNN
 	1    4300 3000
@@
 $EndComp
 $Comp
-L GND #PWR?
+L GND #PWR0124
 U 1 1 5940591E
 P 4300 3250
-F 0 "#PWR?" H 4300 3000 50  0001 C CNN
+F 0 "#PWR0124" H 4300 3000 50  0001 C CNN
 F 1 "GND" H 4300 3100 50  0000 C CNN
 F 2 "" H 4300 3250 50  0001 C CNN
@@
 Wire Wire Line
 	4300 2350 4300 2550
+$Comp
+L C_Small C403
+U 1 1 59405744
+P 6300 3850
+F 0 "C403" H 6310 3920 50  0000 L CNN
+F 1 "10 uF" H 6310 3770 50  0000 L CNN
+F 2 "Capacitors_SMD:C_0603" H 6300 3850 50  0001 C CNN
+F 3 "" H 6300 3850 50  0001 C CNN
+	1    6300 3850
+	1    0    0    -1
+$EndComp
+$Comp
+L CP_Small C402
+U 1 1 59402B31
+P 5850 3850
+F 0 "C402" H 5860 3920 50  0000 L CNN
+F 1 "100 uF" H 5860 3770 50  0000 L CNN
+F 2 "Capacitors_SMD:c_elec_10x10" H 5850 3850 50  0001 C CNN
+F 3 "" H 5850 3850 50  0001 C CNN
+	1    5850 3850
+	1    0    0    -1
+$EndComp
 $EndSCHEMATC

Commit message: started layout of vna r0
Parts:
- removed C401: 100 uF, Capacitors_SMD:c_elec_10x10, symbol CP_Small
- added C401: 10 uF, Capacitors_SMD:C_0603, symbol C_Small
Connections:
- net AMP_5V: now also C401.1
- net GND: now also C401.2
Changed lines of the file:
@@
 $EndDescr
 $Comp
-L +3V3 #PWR0108
+L +3V3 #PWR401
 U 1 1 593F1269
 P 3400 2400
-F 0 "#PWR0108" H 3400 2250 50  0001 C CNN
+F 0 "#PWR401" H 3400 2250 50  0001 C CNN
 F 1 "+3V3" H 3400 2540 50  0000 C CNN
 F 2 "" H 3400 2400 50  0001 C CNN
@@
 $EndComp
 $Comp
-L GND #PWR0109
+L GND #PWR402
 U 1 1 593F1346
 P 3400 3250
-F 0 "#PWR0109" H 3400 3000 50  0001 C CNN
+F 0 "#PWR402" H 3400 3000 50  0001 C CNN
 F 1 "GND" H 3400 3100 50  0000 C CNN
 F 2 "" H 3400 3250 50  0001 C CNN
@@
 $EndComp
 $Comp
-L GND #PWR0110
+L GND #PWR403
 U 1 1 593F15AF
 P 3800 2400
-F 0 "#PWR0110" H 3800 2150 50  0001 C CNN
+F 0 "#PWR403" H 3800 2150 50  0001 C CNN
 F 1 "GND" H 3800 2250 50  0000 C CNN
 F 2 "" H 3800 2400 50  0001 C CNN
@@
 $EndComp
 $Comp
-L GND #PWR0111
+L GND #PWR419
 U 1 1 593F49C3
 P 10250 5400
-F 0 "#PWR0111" H 10250 5150 50  0001 C CNN
+F 0 "#PWR419" H 10250 5150 50  0001 C CNN
 F 1 "GND" H 10250 5250 50  0000 C CNN
 F 2 "" H 10250 5400 50  0001 C CNN
@@
 $EndComp
 $Comp
-L GND #PWR0112
+L GND #PWR417
 U 1 1 593F4A3C
 P 10200 2950
-F 0 "#PWR0112" H 10200 2700 50  0001 C CNN
+F 0 "#PWR417" H 10200 2700 50  0001 C CNN
 F 1 "GND" H 10200 2800 50  0000 C CNN
 F 2 "" H 10200 2950 50  0001 C CNN
@@
 $EndComp
 $Comp
-L GND #PWR0113
+L GND #PWR418
 U 1 1 593F4C31
 P 10200 4050
-F 0 "#PWR0113" H 10200 3800 50  0001 C CNN
+F 0 "#PWR418" H 10200 3800 50  0001 C CNN
 F 1 "GND" H 10200 3900 50  0000 C CNN
 F 2 "" H 10200 4050 50  0001 C CNN
@@
 Text HLabel 6250 5150 2    60   Input ~ 0
 LMX_SDI
-$Comp
-L CP_Small C401
-U 1 1 59402B85
-P 5200 3850
-F 0 "C401" H 5210 3920 50  0000 L CNN
-F 1 "100 uF" H 5210 3770 50  0000 L CNN
-F 2 "Capacitors_SMD:c_elec_10x10" H 5200 3850 50  0001 C CNN
-F 3 "" H 5200 3850 50  0001 C CNN
-	1    5200 3850
-	1    0    0    -1
-$EndComp
 Wire Wire Line
 	3400 3100 3400 3250
@@
 Connection ~ 5500 5050
 $Comp
-L GND #PWR0114
+L GND #PWR412
 U 1 1 59402D3D
 P 5850 4050
-F 0 "#PWR0114" H 5850 3800 50  0001 C CNN
+F 0 "#PWR412" H 5850 3800 50  0001 C CNN
 F 1 "GND" H 5850 3900 50  0000 C CNN
 F 2 "" H 5850 4050 50  0001 C CNN
@@
 	5850 3950 5850 4050
 $Comp
-L +3V3 #PWR0115
+L +3V3 #PWR411
 U 1 1 59402E68
 P 5850 3600
-F 0 "#PWR0115" H 5850 3450 50  0001 C CNN
+F 0 "#PWR411" H 5850 3450 50  0001 C CNN
 F 1 "+3V3" H 5850 3740 50  0000 C CNN
 F 2 "" H 5850 3600 50  0001 C CNN
@@
 Connection ~ 5200 3550
 $Comp
-L GND #PWR0116
+L GND #PWR406
 U 1 1 59403225
 P 5200 4050
-F 0 "#PWR0116" H 5200 3800 50  0001 C CNN
+F 0 "#PWR406" H 5200 3800 50  0001 C CNN
 F 1 "GND" H 5200 3900 50  0000 C CNN
 F 2 "" H 5200 4050 50  0001 C CNN
@@
 $EndComp
 $Comp
-L GND #PWR0117
+L GND #PWR415
 U 1 1 594034F6
 P 6300 3600
-F 0 "#PWR0117" H 6300 3350 50  0001 C CNN
+F 0 "#PWR415" H 6300 3350 50  0001 C CNN
 F 1 "GND" H 6300 3450 50  0000 C CNN
 F 2 "" H 6300 3600 50  0001 C CNN
@@
 	6300 3600 6300 3750
 $Comp
-L GND #PWR0118
+L GND #PWR407
 U 1 1 59404F0C
 P 5450 5150
-F 0 "#PWR0118" H 5450 4900 50  0001 C CNN
+F 0 "#PWR407" H 5450 4900 50  0001 C CNN
 F 1 "GND" H 5450 5000 50  0000 C CNN
 F 2 "" H 5450 5150 50  0001 C CNN
@@
 	6250 5150 6100 5150
 $Comp
-L GND #PWR0119
+L GND #PWR408
 U 1 1 59404FB3
 P 5450 5250
-F 0 "#PWR0119" H 5450 5000 50  0001 C CNN
+F 0 "#PWR408" H 5450 5000 50  0001 C CNN
 F 1 "GND" H 5450 5100 50  0000 C CNN
 F 2 "" H 5450 5250 50  0001 C CNN
@@
 	6100 5250 6250 5250
 $Comp
-L GND #PWR0120
+L GND #PWR409
 U 1 1 5940505E
 P 5450 5350
-F 0 "#PWR0120" H 5450 5100 50  0001 C CNN
+F 0 "#PWR409" H 5450 5100 50  0001 C CNN
 F 1 "GND" H 5450 5200 50  0000 C CNN
 F 2 "" H 5450 5350 50  0001 C CNN
@@
 	5500 5450 5600 5450
 $Comp
-L +3V3 #PWR0121
+L +3V3 #PWR410
 U 1 1 594052AB
 P 5500 5600
-F 0 "#PWR0121" H 5500 5450 50  0001 C CNN
+F 0 "#PWR410" H 5500 5450 50  0001 C CNN
 F 1 "+3V3" H 5500 5740 50  0000 C CNN
 F 2 "" H 5500 5600 50  0001 C CNN
@@
 Connection ~ 5550 5600
 $Comp
-L +3V3 #PWR0122
+L +3V3 #PWR414
 U 1 1 5940537D
 P 6250 5550
-F 0 "#PWR0122" H 6250 5400 50  0001 C CNN
+F 0 "#PWR414" H 6250 5400 50  0001 C CNN
 F 1 "+3V3" H 6250 5690 50  0000 C CNN
 F 2 "" H 6250 5550 50  0001 C CNN
@@
 	6250 5550 6100 5550
 $Comp
-L GND #PWR0123
+L GND #PWR413
 U 1 1 594053F3
 P 6200 5650
-F 0 "#PWR0123" H 6200 5400 50  0001 C CNN
+F 0 "#PWR413" H 6200 5400 50  0001 C CNN
 F 1 "GND" H 6200 5500 50  0000 C CNN
 F 2 "" H 6200 5650 50  0001 C CNN
@@
 $EndComp
 $Comp
-L GND #PWR0124
+L GND #PWR405
 U 1 1 5940591E
 P 4300 3250
-F 0 "#PWR0124" H 4300 3000 50  0001 C CNN
+F 0 "#PWR405" H 4300 3000 50  0001 C CNN
 F 1 "GND" H 4300 3100 50  0000 C CNN
 F 2 "" H 4300 3250 50  0001 C CNN
@@
 	1    0    0    -1
 $EndComp
+$Comp
+L C_Small C401
+U 1 1 5945C695
+P 5200 3850
+F 0 "C401" H 5210 3920 50  0000 L CNN
+F 1 "10 uF" H 5210 3770 50  0000 L CNN
+F 2 "Capacitors_SMD:C_0603" H 5200 3850 50  0001 C CNN
+F 3 "" H 5200 3850 50  0001 C CNN
+	1    5200 3850
+	1    0    0    -1
+$EndComp
