File: hardware/vna_r0/vna_rf/conn_power.sch (KiCad schematic (older format))
At the start: 13 parts, among them J401 CONN_02X10, U401 CONN_SMA_2GND, U402 CONN_SMA_2GND, U403 CONN_SMA

Commit message: work on vna r0 component placement
Parts:
- added U404, U405: CONN_SMA, vna_footprints:732511150_sma_thin, symbol CONN_SMA
Connections:
- net GND: now also U404.2 (GND), U404.3 (GND), U404.4 (GND), U404.5 (GND), U405.2 (GND), U405.3 (GND), U405.4 (GND), U405.5 (GND)
- new net PORT1_BIAS: U404.1 (RF)
- new net PORT2_BIAS: U405.1 (RF)
Changed lines of the file:
@@
 $EndComp
 $Comp
-L -5V #PWR404
+L -5V #PWR406
 U 1 1 593F127D
 P 3800 3250
-F 0 "#PWR404" H 3800 3350 50  0001 C CNN
+F 0 "#PWR406" H 3800 3350 50  0001 C CNN
 F 1 "-5V" H 3800 3400 50  0000 C CNN
 F 2 "" H 3800 3250 50  0001 C CNN
@@
 $EndComp
 $Comp
-L GND #PWR403
+L GND #PWR405
 U 1 1 593F15AF
 P 3800 2400
-F 0 "#PWR403" H 3800 2150 50  0001 C CNN
+F 0 "#PWR405" H 3800 2150 50  0001 C CNN
 F 1 "GND" H 3800 2250 50  0000 C CNN
 F 2 "" H 3800 2400 50  0001 C CNN
@@
 $EndComp
 $Comp
-L GND #PWR419
+L GND #PWR421
 U 1 1 593F49C3
 P 10250 5400
-F 0 "#PWR419" H 10250 5150 50  0001 C CNN
+F 0 "#PWR421" H 10250 5150 50  0001 C CNN
 F 1 "GND" H 10250 5250 50  0000 C CNN
 F 2 "" H 10250 5400 50  0001 C CNN
@@
 $EndComp
 $Comp
-L GND #PWR417
+L GND #PWR419
 U 1 1 593F4A3C
 P 10200 2950
-F 0 "#PWR417" H 10200 2700 50  0001 C CNN
+F 0 "#PWR419" H 10200 2700 50  0001 C CNN
 F 1 "GND" H 10200 2800 50  0000 C CNN
 F 2 "" H 10200 2950 50  0001 C CNN
@@
 $EndComp
 $Comp
-L GND #PWR418
+L GND #PWR420
 U 1 1 593F4C31
 P 10200 4050
-F 0 "#PWR418" H 10200 3800 50  0001 C CNN
+F 0 "#PWR420" H 10200 3800 50  0001 C CNN
 F 1 "GND" H 10200 3900 50  0000 C CNN
 F 2 "" H 10200 4050 50  0001 C CNN
@@
 Connection ~ 5500 5050
 $Comp
-L GND #PWR412
+L GND #PWR414
 U 1 1 59402D3D
 P 5850 4050
-F 0 "#PWR412" H 5850 3800 50  0001 C CNN
+F 0 "#PWR414" H 5850 3800 50  0001 C CNN
 F 1 "GND" H 5850 3900 50  0000 C CNN
 F 2 "" H 5850 4050 50  0001 C CNN
@@
 	5850 3950 5850 4050
 $Comp
-L +3V3 #PWR411
+L +3V3 #PWR413
 U 1 1 59402E68
 P 5850 3600
-F 0 "#PWR411" H 5850 3450 50  0001 C CNN
+F 0 "#PWR413" H 5850 3450 50  0001 C CNN
 F 1 "+3V3" H 5850 3740 50  0000 C CNN
 F 2 "" H 5850 3600 50  0001 C CNN
@@
 Connection ~ 5200 3550
 $Comp
-L GND #PWR406
+L GND #PWR408
 U 1 1 59403225
 P 5200 4050
-F 0 "#PWR406" H 5200 3800 50  0001 C CNN
+F 0 "#PWR408" H 5200 3800 50  0001 C CNN
 F 1 "GND" H 5200 3900 50  0000 C CNN
 F 2 "" H 5200 4050 50  0001 C CNN
@@
 	5200 4050 5200 3950
 $Comp
-L -5V #PWR416
+L -5V #PWR418
 U 1 1 59403473
 P 6300 4050
-F 0 "#PWR416" H 6300 4150 50  0001 C CNN
+F 0 "#PWR418" H 6300 4150 50  0001 C CNN
 F 1 "-5V" H 6300 4200 50  0000 C CNN
 F 2 "" H 6300 4050 50  0001 C CNN
@@
 $EndComp
 $Comp
-L GND #PWR415
+L GND #PWR417
 U 1 1 594034F6
 P 6300 3600
-F 0 "#PWR415" H 6300 3350 50  0001 C CNN
+F 0 "#PWR417" H 6300 3350 50  0001 C CNN
 F 1 "GND" H 6300 3450 50  0000 C CNN
 F 2 "" H 6300 3600 50  0001 C CNN
@@
 	6300 3600 6300 3750
 $Comp
-L GND #PWR407
+L GND #PWR409
 U 1 1 59404F0C
 P 5450 5150
-F 0 "#PWR407" H 5450 4900 50  0001 C CNN
+F 0 "#PWR409" H 5450 4900 50  0001 C CNN
 F 1 "GND" H 5450 5000 50  0000 C CNN
 F 2 "" H 5450 5150 50  0001 C CNN
@@
 	6250 5150 6100 5150
 $Comp
-L GND #PWR408
+L GND #PWR410
 U 1 1 59404FB3
 P 5450 5250
-F 0 "#PWR408" H 5450 5000 50  0001 C CNN
+F 0 "#PWR410" H 5450 5000 50  0001 C CNN
 F 1 "GND" H 5450 5100 50  0000 C CNN
 F 2 "" H 5450 5250 50  0001 C CNN
@@
 	6100 5250 6250 5250
 $Comp
-L GND #PWR409
+L GND #PWR411
 U 1 1 5940505E
 P 5450 5350
-F 0 "#PWR409" H 5450 5100 50  0001 C CNN
+F 0 "#PWR411" H 5450 5100 50  0001 C CNN
 F 1 "GND" H 5450 5200 50  0000 C CNN
 F 2 "" H 5450 5350 50  0001 C CNN
@@
 	5500 5450 5600 5450
 $Comp
-L +3V3 #PWR410
+L +3V3 #PWR412
 U 1 1 594052AB
 P 5500 5600
-F 0 "#PWR410" H 5500 5450 50  0001 C CNN
+F 0 "#PWR412" H 5500 5450 50  0001 C CNN
 F 1 "+3V3" H 5500 5740 50  0000 C CNN
 F 2 "" H 5500 5600 50  0001 C CNN
@@
 Connection ~ 5550 5600
 $Comp
-L +3V3 #PWR414
+L +3V3 #PWR416
 U 1 1 5940537D
 P 6250 5550
-F 0 "#PWR414" H 6250 5400 50  0001 C CNN
+F 0 "#PWR416" H 6250 5400 50  0001 C CNN
 F 1 "+3V3" H 6250 5690 50  0000 C CNN
 F 2 "" H 6250 5550 50  0001 C CNN
@@
 	6250 5550 6100 5550
 $Comp
-L GND #PWR413
+L GND #PWR415
 U 1 1 594053F3
 P 6200 5650
-F 0 "#PWR413" H 6200 5400 50  0001 C CNN
+F 0 "#PWR415" H 6200 5400 50  0001 C CNN
 F 1 "GND" H 6200 5500 50  0000 C CNN
 F 2 "" H 6200 5650 50  0001 C CNN
@@
 $EndComp
 $Comp
-L GND #PWR405
+L GND #PWR407
 U 1 1 5940591E
 P 4300 3250
-F 0 "#PWR405" H 4300 3000 50  0001 C CNN
+F 0 "#PWR407" H 4300 3000 50  0001 C CNN
 F 1 "GND" H 4300 3100 50  0000 C CNN
 F 2 "" H 4300 3250 50  0001 C CNN
@@
 	1    0    0    -1
 $EndComp
+Text HLabel 2850 5400 0    60   Input ~ 0
+PORT1_BIAS
+Text HLabel 2850 6600 0    60   Input ~ 0
+PORT2_BIAS
+$Comp
+L CONN_SMA U405
+U 1 1 594792B9
+P 3750 6600
+F 0 "U405" H 3400 6800 60  0000 C CNN
+F 1 "CONN_SMA" H 3600 6950 60  0000 C CNN
+F 2 "vna_footprints:732511150_sma_thin" H 3750 6600 60  0001 C CNN
+F 3 "" H 3750 6600 60  0000 C CNN
+	1    3750 6600
+	1    0    0    -1
+$EndComp
+$Comp
+L GND #PWR404
+U 1 1 594792BF
+P 3750 7200
+F 0 "#PWR404" H 3750 6950 50  0001 C CNN
+F 1 "GND" H 3750 7050 50  0000 C CNN
+F 2 "" H 3750 7200 50  0001 C CNN
+F 3 "" H 3750 7200 50  0001 C CNN
+	1    3750 7200
+	1    0    0    -1
+$EndComp
+Wire Wire Line
+	3600 7050 3600 7100
+Wire Wire Line
+	3600 7100 3900 7100
+Wire Wire Line
+	3900 7100 3900 7050
+Wire Wire Line
+	3700 7050 3700 7100
+Connection ~ 3700 7100
+Wire Wire Line
+	3800 7050 3800 7100
+Connection ~ 3800 7100
+Wire Wire Line
+	3750 7100 3750 7200
+Connection ~ 3750 7100
+Wire Wire Line
+	3200 6600 2850 6600
+$Comp
+L CONN_SMA U404
+U 1 1 59479521
+P 3750 5400
+F 0 "U404" H 3400 5600 60  0000 C CNN
+F 1 "CONN_SMA" H 3600 5750 60  0000 C CNN
+F 2 "vna_footprints:732511150_sma_thin" H 3750 5400 60  0001 C CNN
+F 3 "" H 3750 5400 60  0000 C CNN
+	1    3750 5400
+	1    0    0    -1
+$EndComp
+$Comp
+L GND #PWR403
+U 1 1 59479527
+P 3750 6000
+F 0 "#PWR403" H 3750 5750 50  0001 C CNN
+F 1 "GND" H 3750 5850 50  0000 C CNN
+F 2 "" H 3750 6000 50  0001 C CNN
+F 3 "" H 3750 6000 50  0001 C CNN
+	1    3750 6000
+	1    0    0    -1
+$EndComp
+Wire Wire Line
+	3600 5850 3600 5900
+Wire Wire Line
+	3600 5900 3900 5900
+Wire Wire Line
+	3900 5900 3900 5850
+Wire Wire Line
+	3700 5850 3700 5900
+Connection ~ 3700 5900
+Wire Wire Line
+	3800 5850 3800 5900
+Connection ~ 3800 5900
+Wire Wire Line
+	3750 5900 3750 6000
+Connection ~ 3750 5900
+Wire Wire Line
+	3200 5400 2850 5400
 $EndSCHEMATC

Commit message: work on vna r0 layout..
Parts:
- added H401, H402, H403, H404: MOUNTING_HOLE, Mounting_Holes:MountingHole_2-7mm, symbol MOUNTING_HOLE
- added J402: RF_Shield_Two_Pieces, Shielding_Cabinets:Laird_Technologies_BMI-S-205-F_38.10x25.40mm, symbol RF_Shield_Two_Pieces
Connections:
- net -5V: now also J401.14 (P14)
- net GND: now also J402.1 (Shield); no longer J401.14 (P14)
Changed lines of the file:
@@
 LIBS:conn_sma_2gnd
 LIBS:conn_sma
+LIBS:mounting_hole
 LIBS:vna_rf-cache
 EELAYER 25 0
@@
 $EndDescr
 $Comp
-L +3V3 #PWR401
+L +3V3 #PWR0113
 U 1 1 593F1269
 P 3400 2400
-F 0 "#PWR401" H 3400 2250 50  0001 C CNN
+F 0 "#PWR0113" H 3400 2250 50  0001 C CNN
 F 1 "+3V3" H 3400 2540 50  0000 C CNN
 F 2 "" H 3400 2400 50  0001 C CNN
@@
 $EndComp
 $Comp
-L GND #PWR402
+L GND #PWR0114
 U 1 1 593F1346
 P 3400 3250
-F 0 "#PWR402" H 3400 3000 50  0001 C CNN
+F 0 "#PWR0114" H 3400 3000 50  0001 C CNN
 F 1 "GND" H 3400 3100 50  0000 C CNN
 F 2 "" H 3400 3250 50  0001 C CNN
@@
 $EndComp
 $Comp
-L GND #PWR405
+L GND #PWR0115
 U 1 1 593F15AF
 P 3800 2400
-F 0 "#PWR405" H 3800 2150 50  0001 C CNN
+F 0 "#PWR0115" H 3800 2150 50  0001 C CNN
 F 1 "GND" H 3800 2250 50  0000 C CNN
 F 2 "" H 3800 2400 50  0001 C CNN
@@
 $EndComp
 $Comp
-L GND #PWR421
+L GND #PWR0116
 U 1 1 593F49C3
 P 10250 5400
-F 0 "#PWR421" H 10250 5150 50  0001 C CNN
+F 0 "#PWR0116" H 10250 5150 50  0001 C CNN
 F 1 "GND" H 10250 5250 50  0000 C CNN
 F 2 "" H 10250 5400 50  0001 C CNN
@@
 $EndComp
 $Comp
-L GND #PWR419
+L GND #PWR0117
 U 1 1 593F4A3C
 P 10200 2950
-F 0 "#PWR419" H 10200 2700 50  0001 C CNN
+F 0 "#PWR0117" H 10200 2700 50  0001 C CNN
 F 1 "GND" H 10200 2800 50  0000 C CNN
 F 2 "" H 10200 2950 50  0001 C CNN
@@
 $EndComp
 $Comp
-L GND #PWR420
+L GND #PWR0118
 U 1 1 593F4C31
 P 10200 4050
-F 0 "#PWR420" H 10200 3800 50  0001 C CNN
+F 0 "#PWR0118" H 10200 3800 50  0001 C CNN
 F 1 "GND" H 10200 3900 50  0000 C CNN
 F 2 "" H 10200 4050 50  0001 C CNN
@@
 Connection ~ 5500 5050
 $Comp
-L GND #PWR414
+L GND #PWR0119
 U 1 1 59402D3D
 P 5850 4050
-F 0 "#PWR414" H 5850 3800 50  0001 C CNN
+F 0 "#PWR0119" H 5850 3800 50  0001 C CNN
 F 1 "GND" H 5850 3900 50  0000 C CNN
 F 2 "" H 5850 4050 50  0001 C CNN
@@
 	5850 3950 5850 4050
 $Comp
-L +3V3 #PWR413
+L +3V3 #PWR0120
 U 1 1 59402E68
 P 5850 3600
-F 0 "#PWR413" H 5850 3450 50  0001 C CNN
+F 0 "#PWR0120" H 5850 3450 50  0001 C CNN
 F 1 "+3V3" H 5850 3740 50  0000 C CNN
 F 2 "" H 5850 3600 50  0001 C CNN
@@
 Connection ~ 5200 3550
 $Comp
-L GND #PWR408
+L GND #PWR0121
 U 1 1 59403225
 P 5200 4050
-F 0 "#PWR408" H 5200 3800 50  0001 C CNN
+F 0 "#PWR0121" H 5200 3800 50  0001 C CNN
 F 1 "GND" H 5200 3900 50  0000 C CNN
 F 2 "" H 5200 4050 50  0001 C CNN
@@
 $EndComp
 $Comp
-L GND #PWR417
+L GND #PWR0122
 U 1 1 594034F6
 P 6300 3600
-F 0 "#PWR417" H 6300 3350 50  0001 C CNN
+F 0 "#PWR0122" H 6300 3350 50  0001 C CNN
 F 1 "GND" H 6300 3450 50  0000 C CNN
 F 2 "" H 6300 3600 50  0001 C CNN
@@
 	6300 3600 6300 3750
 $Comp
-L GND #PWR409
+L GND #PWR0123
 U 1 1 59404F0C
 P 5450 5150
-F 0 "#PWR409" H 5450 4900 50  0001 C CNN
+F 0 "#PWR0123" H 5450 4900 50  0001 C CNN
 F 1 "GND" H 5450 5000 50  0000 C CNN
 F 2 "" H 5450 5150 50  0001 C CNN
@@
 	6250 5150 6100 5150
 $Comp
-L GND #PWR410
+L GND #PWR0124
 U 1 1 59404FB3
 P 5450 5250
-F 0 "#PWR410" H 5450 5000 50  0001 C CNN
+F 0 "#PWR0124" H 5450 5000 50  0001 C CNN
 F 1 "GND" H 5450 5100 50  0000 C CNN
 F 2 "" H 5450 5250 50  0001 C CNN
@@
 	6100 5250 6250 5250
 $Comp
-L GND #PWR411
+L GND #PWR0125
 U 1 1 5940505E
 P 5450 5350
-F 0 "#PWR411" H 5450 5100 50  0001 C CNN
+F 0 "#PWR0125" H 5450 5100 50  0001 C CNN
 F 1 "GND" H 5450 5200 50  0000 C CNN
 F 2 "" H 5450 5350 50  0001 C CNN
@@
 	5500 5450 5600 5450
 $Comp
-L +3V3 #PWR412
+L +3V3 #PWR0126
 U 1 1 594052AB
 P 5500 5600
-F 0 "#PWR412" H 5500 5450 50  0001 C CNN
+F 0 "#PWR0126" H 5500 5450 50  0001 C CNN
 F 1 "+3V3" H 5500 5740 50  0000 C CNN
 F 2 "" H 5500 5600 50  0001 C CNN
@@
 Connection ~ 5550 5600
 $Comp
-L +3V3 #PWR416
+L +3V3 #PWR0127
 U 1 1 5940537D
 P 6250 5550
-F 0 "#PWR416" H 6250 5400 50  0001 C CNN
+F 0 "#PWR0127" H 6250 5400 50  0001 C CNN
 F 1 "+3V3" H 6250 5690 50  0000 C CNN
 F 2 "" H 6250 5550 50  0001 C CNN
@@
 Wire Wire Line
 	6250 5550 6100 5550
-$Comp
-L GND #PWR415
-U 1 1 594053F3
-P 6200 5650
-F 0 "#PWR415" H 6200 5400 50  0001 C CNN
-F 1 "GND" H 6200 5500 50  0000 C CNN
-F 2 "" H 6200 5650 50  0001 C CNN
-F 3 "" H 6200 5650 50  0001 C CNN
-	1    6200 5650
-	0    -1   -1   0
-$EndComp
 Wire Wire Line
 	6200 5650 6100 5650
@@
 $EndComp
 $Comp
-L GND #PWR407
+L GND #PWR0128
 U 1 1 5940591E
 P 4300 3250
-F 0 "#PWR407" H 4300 3000 50  0001 C CNN
+F 0 "#PWR0128" H 4300 3000 50  0001 C CNN
 F 1 "GND" H 4300 3100 50  0000 C CNN
 F 2 "" H 4300 3250 50  0001 C CNN
@@
 $EndComp
 $Comp
-L GND #PWR404
+L GND #PWR0129
 U 1 1 594792BF
 P 3750 7200
-F 0 "#PWR404" H 3750 6950 50  0001 C CNN
+F 0 "#PWR0129" H 3750 6950 50  0001 C CNN
 F 1 "GND" H 3750 7050 50  0000 C CNN
 F 2 "" H 3750 7200 50  0001 C CNN
@@
 $EndComp
 $Comp
-L GND #PWR403
+L GND #PWR0130
 U 1 1 59479527
 P 3750 6000
-F 0 "#PWR403" H 3750 5750 50  0001 C CNN
+F 0 "#PWR0130" H 3750 5750 50  0001 C CNN
 F 1 "GND" H 3750 5850 50  0000 C CNN
 F 2 "" H 3750 6000 50  0001 C CNN
@@
 Wire Wire Line
 	3200 5400 2850 5400
+$Comp
+L -5V #PWR415
+U 1 1 59479398
+P 6200 5650
+F 0 "#PWR415" H 6200 5750 50  0001 C CNN
+F 1 "-5V" H 6200 5800 50  0000 C CNN
+F 2 "" H 6200 5650 50  0001 C CNN
+F 3 "" H 6200 5650 50  0001 C CNN
+	1    6200 5650
+	0    1    1    0
+$EndComp
+$Comp
+L RF_Shield_Two_Pieces J402
+U 1 1 594A1BB1
+P 6900 2000
+F 0 "J402" H 6900 2200 50  0000 C CNN
+F 1 "RF_Shield_Two_Pieces" H 6900 2100 50  0000 C CNN
+F 2 "Shielding_Cabinets:Laird_Technologies_BMI-S-205-F_38.10x25.40mm" H 6900 1900 50  0001 C CNN
+F 3 "" H 6900 1900 50  0001 C CNN
+	1    6900 2000
+	1    0    0    -1
+$EndComp
+$Comp
+L MOUNTING_HOLE H401
+U 1 1 594A1CEE
+P 8350 2150
+F 0 "H401" H 8050 2200 60  0000 C CNN
+F 1 "MOUNTING_HOLE" H 8350 2300 60  0000 C CNN
+F 2 "Mounting_Holes:MountingHole_2-7mm" H 8350 2150 60  0001 C CNN
+F 3 "" H 8350 2150 60  0000 C CNN
+	1    8350 2150
+	1    0    0    -1
+$EndComp
+$Comp
+L MOUNTING_HOLE H402
+U 1 1 594A1D86
+P 8350 2450
+F 0 "H402" H 8050 2500 60  0000 C CNN
+F 1 "MOUNTING_HOLE" H 8350 2600 60  0000 C CNN
+F 2 "Mounting_Holes:MountingHole_2-7mm" H 8350 2450 60  0001 C CNN
+F 3 "" H 8350 2450 60  0000 C CNN
+	1    8350 2450
+	1    0    0    -1
+$EndComp
+$Comp
+L MOUNTING_HOLE H403
+U 1 1 594A1DD8
+P 8350 2750
+F 0 "H403" H 8050 2800 60  0000 C CNN
+F 1 "MOUNTING_HOLE" H 8350 2900 60  0000 C CNN
+F 2 "Mounting_Holes:MountingHole_2-7mm" H 8350 2750 60  0001 C CNN
+F 3 "" H 8350 2750 60  0000 C CNN
+	1    8350 2750
+	1    0    0    -1
+$EndComp
+$Comp
+L MOUNTING_HOLE H404
+U 1 1 594A1E29
+P 8350 3050
+F 0 "H404" H 8050 3100 60  0000 C CNN
+F 1 "MOUNTING_HOLE" H 8350 3200 60  0000 C CNN
+F 2 "Mounting_Holes:MountingHole_2-7mm" H 8350 3050 60  0001 C CNN
+F 3 "" H 8350 3050 60  0000 C CNN
+	1    8350 3050
+	1    0    0    -1
+$EndComp
+$Comp
+L GND #PWR?
+U 1 1 594A25A4
+P 6900 2450
+F 0 "#PWR?" H 6900 2200 50  0001 C CNN
+F 1 "GND" H 6900 2300 50  0000 C CNN
+F 2 "" H 6900 2450 50  0001 C CNN
+F 3 "" H 6900 2450 50  0001 C CNN
+	1    6900 2450
+	1    0    0    -1
+$EndComp
+Wire Wire Line
+	6900 2450 6900 2400
 $EndSCHEMATC

Commit message: work on vna r0 layout
Parts:
- added U406: CONN_SMA_2GND, vna_footprints:734120110_ufl_umc, symbol CONN_SMA_2GND
Connections:
- net GND: now also U406.2 (GND), U406.3 (GND)
- net SYNTH_REF: now also U406.1 (RF)
Changed lines of the file:
@@
 $EndDescr
 $Comp
-L +3V3 #PWR0113
+L +3V3 #PWR0112
 U 1 1 593F1269
 P 3400 2400
-F 0 "#PWR0113" H 3400 2250 50  0001 C CNN
+F 0 "#PWR0112" H 3400 2250 50  0001 C CNN
 F 1 "+3V3" H 3400 2540 50  0000 C CNN
 F 2 "" H 3400 2400 50  0001 C CNN
@@
 $EndComp
 $Comp
-L GND #PWR0114
+L GND #PWR0113
 U 1 1 593F1346
 P 3400 3250
-F 0 "#PWR0114" H 3400 3000 50  0001 C CNN
+F 0 "#PWR0113" H 3400 3000 50  0001 C CNN
 F 1 "GND" H 3400 3100 50  0000 C CNN
 F 2 "" H 3400 3250 50  0001 C CNN
@@
 $EndComp
 $Comp
-L GND #PWR0115
+L GND #PWR0114
 U 1 1 593F15AF
 P 3800 2400
-F 0 "#PWR0115" H 3800 2150 50  0001 C CNN
+F 0 "#PWR0114" H 3800 2150 50  0001 C CNN
 F 1 "GND" H 3800 2250 50  0000 C CNN
 F 2 "" H 3800 2400 50  0001 C CNN
@@
 $EndComp
 $Comp
-L GND #PWR0116
+L GND #PWR0115
 U 1 1 593F49C3
 P 10250 5400
-F 0 "#PWR0116" H 10250 5150 50  0001 C CNN
+F 0 "#PWR0115" H 10250 5150 50  0001 C CNN
 F 1 "GND" H 10250 5250 50  0000 C CNN
 F 2 "" H 10250 5400 50  0001 C CNN
@@
 $EndComp
 $Comp
-L GND #PWR0117
+L GND #PWR0116
 U 1 1 593F4A3C
 P 10200 2950
-F 0 "#PWR0117" H 10200 2700 50  0001 C CNN
+F 0 "#PWR0116" H 10200 2700 50  0001 C CNN
 F 1 "GND" H 10200 2800 50  0000 C CNN
 F 2 "" H 10200 2950 50  0001 C CNN
@@
 $EndComp
 $Comp
-L GND #PWR0118
+L GND #PWR0117
 U 1 1 593F4C31
 P 10200 4050
-F 0 "#PWR0118" H 10200 3800 50  0001 C CNN
+F 0 "#PWR0117" H 10200 3800 50  0001 C CNN
 F 1 "GND" H 10200 3900 50  0000 C CNN
 F 2 "" H 10200 4050 50  0001 C CNN
@@
 Connection ~ 5500 5050
 $Comp
-L GND #PWR0119
+L GND #PWR0118
 U 1 1 59402D3D
 P 5850 4050
-F 0 "#PWR0119" H 5850 3800 50  0001 C CNN
+F 0 "#PWR0118" H 5850 3800 50  0001 C CNN
 F 1 "GND" H 5850 3900 50  0000 C CNN
 F 2 "" H 5850 4050 50  0001 C CNN
@@
 	5850 3950 5850 4050
 $Comp
-L +3V3 #PWR0120
+L +3V3 #PWR0119
 U 1 1 59402E68
 P 5850 3600
-F 0 "#PWR0120" H 5850 3450 50  0001 C CNN
+F 0 "#PWR0119" H 5850 3450 50  0001 C CNN
 F 1 "+3V3" H 5850 3740 50  0000 C CNN
 F 2 "" H 5850 3600 50  0001 C CNN
@@
 Connection ~ 5200 3550
 $Comp
-L GND #PWR0121
+L GND #PWR0120
 U 1 1 59403225
 P 5200 4050
-F 0 "#PWR0121" H 5200 3800 50  0001 C CNN
+F 0 "#PWR0120" H 5200 3800 50  0001 C CNN
 F 1 "GND" H 5200 3900 50  0000 C CNN
 F 2 "" H 5200 4050 50  0001 C CNN
@@
 $EndComp
 $Comp
-L GND #PWR0122
+L GND #PWR0121
 U 1 1 594034F6
 P 6300 3600
-F 0 "#PWR0122" H 6300 3350 50  0001 C CNN
+F 0 "#PWR0121" H 6300 3350 50  0001 C CNN
 F 1 "GND" H 6300 3450 50  0000 C CNN
 F 2 "" H 6300 3600 50  0001 C CNN
@@
 	6300 3600 6300 3750
 $Comp
-L GND #PWR0123
+L GND #PWR0122
 U 1 1 59404F0C
 P 5450 5150
-F 0 "#PWR0123" H 5450 4900 50  0001 C CNN
+F 0 "#PWR0122" H 5450 4900 50  0001 C CNN
 F 1 "GND" H 5450 5000 50  0000 C CNN
 F 2 "" H 5450 5150 50  0001 C CNN
@@
 	6250 5150 6100 5150
 $Comp
-L GND #PWR0124
+L GND #PWR0123
 U 1 1 59404FB3
 P 5450 5250
-F 0 "#PWR0124" H 5450 5000 50  0001 C CNN
+F 0 "#PWR0123" H 5450 5000 50  0001 C CNN
 F 1 "GND" H 5450 5100 50  0000 C CNN
 F 2 "" H 5450 5250 50  0001 C CNN
@@
 	6100 5250 6250 5250
 $Comp
-L GND #PWR0125
+L GND #PWR0124
 U 1 1 5940505E
 P 5450 5350
-F 0 "#PWR0125" H 5450 5100 50  0001 C CNN
+F 0 "#PWR0124" H 5450 5100 50  0001 C CNN
 F 1 "GND" H 5450 5200 50  0000 C CNN
 F 2 "" H 5450 5350 50  0001 C CNN
@@
 	5500 5450 5600 5450
 $Comp
-L +3V3 #PWR0126
+L +3V3 #PWR0125
 U 1 1 594052AB
 P 5500 5600
-F 0 "#PWR0126" H 5500 5450 50  0001 C CNN
+F 0 "#PWR0125" H 5500 5450 50  0001 C CNN
 F 1 "+3V3" H 5500 5740 50  0000 C CNN
 F 2 "" H 5500 5600 50  0001 C CNN
@@
 Connection ~ 5550 5600
 $Comp
-L +3V3 #PWR0127
+L +3V3 #PWR0126
 U 1 1 5940537D
 P 6250 5550
-F 0 "#PWR0127" H 6250 5400 50  0001 C CNN
+F 0 "#PWR0126" H 6250 5400 50  0001 C CNN
 F 1 "+3V3" H 6250 5690 50  0000 C CNN
 F 2 "" H 6250 5550 50  0001 C CNN
@@
 $EndComp
 $Comp
-L GND #PWR0128
+L GND #PWR0127
 U 1 1 5940591E
 P 4300 3250
-F 0 "#PWR0128" H 4300 3000 50  0001 C CNN
+F 0 "#PWR0127" H 4300 3000 50  0001 C CNN
 F 1 "GND" H 4300 3100 50  0000 C CNN
 F 2 "" H 4300 3250 50  0001 C CNN
@@
 $EndComp
 $Comp
-L GND #PWR0129
+L GND #PWR0128
 U 1 1 594792BF
 P 3750 7200
-F 0 "#PWR0129" H 3750 6950 50  0001 C CNN
+F 0 "#PWR0128" H 3750 6950 50  0001 C CNN
 F 1 "GND" H 3750 7050 50  0000 C CNN
 F 2 "" H 3750 7200 50  0001 C CNN
@@
 $EndComp
 $Comp
-L GND #PWR0130
+L GND #PWR0129
 U 1 1 59479527
 P 3750 6000
-F 0 "#PWR0130" H 3750 5750 50  0001 C CNN
+F 0 "#PWR0129" H 3750 5750 50  0001 C CNN
 F 1 "GND" H 3750 5850 50  0000 C CNN
 F 2 "" H 3750 6000 50  0001 C CNN
@@
 $EndComp
 $Comp
-L GND #PWR?
+L GND #PWR0130
 U 1 1 594A25A4
 P 6900 2450
-F 0 "#PWR?" H 6900 2200 50  0001 C CNN
+F 0 "#PWR0130" H 6900 2200 50  0001 C CNN
 F 1 "GND" H 6900 2300 50  0000 C CNN
 F 2 "" H 6900 2450 50  0001 C CNN
@@
 Wire Wire Line
 	6900 2450 6900 2400
+$Comp
+L CONN_SMA_2GND U406
+U 1 1 594E46C5
+P 10200 5800
+F 0 "U406" H 9900 6000 60  0000 C CNN
+F 1 "CONN_SMA_2GND" H 10250 6100 60  0000 C CNN
+F 2 "vna_footprints:734120110_ufl_umc" H 10200 5800 60  0001 C CNN
+F 3 "" H 10200 5800 60  0000 C CNN
+	1    10200 5800
+	-1   0    0    -1
+$EndComp
+$Comp
+L GND #PWR0131
+U 1 1 594E478D
+P 10200 6400
+F 0 "#PWR0131" H 10200 6150 50  0001 C CNN
+F 1 "GND" H 10200 6250 50  0000 C CNN
+F 2 "" H 10200 6400 50  0001 C CNN
+F 3 "" H 10200 6400 50  0001 C CNN
+	1    10200 6400
+	-1   0    0    -1
+$EndComp
+Wire Wire Line
+	10250 6250 10250 6300
+Wire Wire Line
+	10250 6300 10150 6300
+Wire Wire Line
+	10200 6300 10200 6400
+Wire Wire Line
+	10150 6300 10150 6250
+Connection ~ 10200 6300
+Wire Wire Line
+	9800 5800 9600 5800
+Wire Wire Line
+	9600 5800 9600 4800
+Connection ~ 9600 4800
 $EndSCHEMATC
