File: hardware/vna_r0/vna_demod/demod.sch (KiCad schematic (older format))
At the start: 52 parts, among them U301 ad9864, U302 LTC5549

Commit message: work on vna r0 schematics
Parts:
- added C?: 10 nF, symbol C_Small
Connections:
- net IFIN: now also C?.2; no longer R?.1, R?.2
- new net: C?.1, R?.1, R?.2
Other:
- note added: "IF in is 370 ohms || 1.4 pF"
Changed lines of the file:
@@
 LIBS:conn_sma_2gnd
 LIBS:conn_sma
+LIBS:txco
+LIBS:nb3n551
+LIBS:hmc475
+LIBS:trf37b73
 LIBS:vna_demod-cache
 EELAYER 25 0
@@
 $Descr A3 16535 11693
 encoding utf-8
-Sheet 5 8
+Sheet 3 8
 Title ""
 Date ""
@@
 	1    0    0    -1
 $EndComp
-Text Label 5200 5700 0    60   ~ 0
+Text Label 5650 5700 0    60   ~ 0
 IFIN
 $Comp
@@
 	10800 5650 10800 5750
 Connection ~ 10800 5300
+Text Notes 4850 5450 0    60   ~ 0
+IF in is 370 ohms || 1.4 pF
+$Comp
+L C_Small C?
+U 1 1 593FD95B
+P 5300 5700
+F 0 "C?" H 5310 5770 50  0000 L CNN
+F 1 "10 nF" V 5350 5400 50  0000 L CNN
+F 2 "" H 5300 5700 50  0001 C CNN
+F 3 "" H 5300 5700 50  0001 C CNN
+	1    5300 5700
+	0    -1   -1   0
+$EndComp
+Wire Wire Line
+	5650 5700 5400 5700
 $EndSCHEMATC

Commit message: footprint assignment on vna r0
Parts:
- C301, C302, C303, C304, C305, C306, C307, C308, C309, C310, C311, C312, C313, C314, C315, C316, C317, C318, C319, C320, C321, C322, C323, C324, C325, C326, C327, C329: renamed from C?; footprint (none) -> Capacitors_SMD:C_0402
- C328: renamed from C?; footprint (none) -> Capacitors_SMD:C_0603
- L301, L304: renamed from L?; footprint (none) -> Resistors_SMD:R_0402
- L302, L303: renamed from L?; footprint (none) -> Resistors_SMD:R_0805
- R301, R302, R303, R304, R305, R306, R307, R308, R309, R310, R311, R312, R313, R314, R315, R316, R317: renamed from R?; footprint (none) -> Resistors_SMD:R_0402
- T301: renamed from T?; footprint (none) -> vna_footprints:5LEAD_BALUN_4p83mm_3p3mm
- U301: renamed from U302; footprint (none) -> vna_footprints:QFN_12_3mm2mm
- U302: renamed from U301; footprint (none) -> Housings_DFN_QFN:QFN-48-1EP_7x7mm_Pitch0.5mm

Commit message: started layout of vna r0
Parts:
- added J301: RF_Shield_Two_Pieces, Shielding_Cabinets:Laird_Technologies_BMI-S-209-F_29.36x18.50mm, symbol RF_Shield_Two_Pieces
Connections:
- net GND: now also J301.1 (Shield)

Commit message: started component placement on demod
Parts:
- L302, L303: value 6.8 uH -> 6.8 uH BRL1608T6R8M; footprint Resistors_SMD:R_0805 -> Resistors_SMD:R_0603

Commit message: work on demod layout
Connections:
- net +3V3: no longer C324.2
- net GND: now also C324.2
