File: hardware/vna_r0/vna_demod/clock_distro.sch (KiCad schematic (older format))
At the start: 0 parts

Commit message: work on vna r0 schematics
Parts:
- added C? (x2): C_Small, symbol C_Small
- added C? (x3): 10 nF, symbol C_Small
- added C? (x2): 100 nF, symbol C_Small
- added L?: L_Small, symbol L_Small
- added R? (x4): 30, symbol R_Small
- added R? (x12): DNP, symbol R_Small
- added R? (x3): 10k, symbol R_Small
- added R? (x2): JMP, symbol R_Small
- added R?: 1k, symbol R_Small
- added U?: TXCO, symbol TXCO
- added U?: NB3N551, symbol NB3N551
- added U?: TRF37B73, symbol TRF37B73
Connections:
- new net: R?.1, U?.1 (EN)
- new net: R?.2, U?.3 (OSC)
- new net: R?.1, R?.1, R?.2, U?.1 (ICLK)
- new net: C?.1, R?.1, R?.2
- new net: R?.1, R?.1, R?.1, R?.1, R?.2
- new net: C?.2, L?.2, U?.7 (RFOUT)
- new net: C?.1, U?.2 (RFIN)
- new net: C?.2, R?.1, R?.2
- new net: R?.1, R?.2, R?.2
- new net: R?.2, R?.2, U?.5 (PWDN)
- new net +3V3: C?.1, C?.1, C?.1, C?.1, C?.1, L?.1, R?.2, R?.2, U?.1 (VCC), U?.4 (VCC), U?.7 (Vdd)
- new net ADC_CLK_EN: R?.1, U?.8 (OE)
- new net ADC_CLK_IN: R?.2
- new net CLK_A: R?.1
- new net CLK_B: R?.1
- new net CLK_C: R?.1
- new net CLK_D: R?.1
- new net GND: C?.2, C?.2, C?.2, C?.2, C?.2, R?.1, R?.1, R?.1, R?.1, R?.1, R?.1, U?.2 (GND), U?.3 (NC), U?.4 (NC), U?.6 (GND), U?.6 (NC), U?.8 (NC), U?.9 (EP)
- new net IF_LO_A: R?.2
- new net IF_LO_B: R?.2
- new net IF_LO_C: R?.2
- new net IF_LO_D: R?.2
- new net IF_LO_EN: R?.1
- new net IF_LO_IN: R?.2, R?.2
- new net Q1: R?.2, U?.2 (Q1)
- new net Q2: R?.2, U?.3 (Q2)
- new net Q3: R?.2, U?.4 (Q3)
- new net Q4: R?.2, U?.5 (Q4)
Other:
- note added: "-6 dBm"
- note added: "3v3 square output"

Commit message: footprint assignment on vna r0
Parts:
- C801, C802, C804, C805, C806: renamed from C?; footprint (none) -> Capacitors_SMD:C_0402
- C803, C807: renamed from C?; value C_Small -> 100 nF; footprint (none) -> Capacitors_SMD:C_0402
- L801: renamed from L?; footprint (none) -> Resistors_SMD:R_0805
- R801, R802, R803, R804, R805, R806, R807, R808, R809, R810, R811, R812, R813, R814, R815, R816, R817, R818, R819, R820, R821, R822: renamed from R?; footprint (none) -> Resistors_SMD:R_0402
- U801: renamed from U?; footprint (none) -> vna_footprints:crystal_FA238-TSX3225
- U802: renamed from U?; footprint (none) -> Housings_DFN_QFN:DFN-8-1EP_2x2mm_Pitch0.5mm
- U803: renamed from U?; footprint (none) -> Housings_SOIC:SOIC-8_3.9x4.9mm_Pitch1.27mm

Commit message: started component placement on demod
Parts:
- L801: value L_Small -> 6.8 uH; footprint Resistors_SMD:R_0805 -> Resistors_SMD:R_0603
Changed lines of the file:
@@
 LIBS:hmc475
 LIBS:trf37b73
+LIBS:mounting_hole
+LIBS:mounting_box
 LIBS:vna_demod-cache
 EELAYER 25 0
@@
 P 4900 5100
 F 0 "L801" H 4930 5140 50  0000 L CNN
-F 1 "L_Small" H 4930 5060 50  0000 L CNN
-F 2 "Resistors_SMD:R_0805" H 4900 5100 50  0001 C CNN
+F 1 "6.8 uH" H 4930 5060 50  0000 L CNN
+F 2 "Resistors_SMD:R_0603" H 4900 5100 50  0001 C CNN
 F 3 "" H 4900 5100 50  0001 C CNN
 	1    4900 5100

Commit message: routing on demod, almost done..
Connections:
- net Q1: now also R821.2; no longer R819.2
- net Q3: now also R819.2; no longer R821.2
Changed lines of the file:
@@
 Text Label 3900 2900 2    60   ~ 0
 Q3
-Text Label 6950 2500 2    60   ~ 0
+Text Label 6950 2800 2    60   ~ 0
 Q1
 Text Label 6950 2650 2    60   ~ 0
 Q2
-Text Label 6950 2800 2    60   ~ 0
+Text Label 6950 2500 2    60   ~ 0
 Q3
 Text Label 6950 2950 2    60   ~ 0
