File: hardware/vna_r0/vna_control/vna_control.kicad_pcb (KiCad board)
At the start: 4 copper layers, 73.7 x 72.4 mm, 175 parts, among them J301 CONN_02X10, J302 CONN_02X10, J303 CONN_02X10, J304 CONN_02X23, J305 CONN_01X02, J306 CONN_02X23, J307 BARREL_JACK, J401 CONN_01X02, Q301 DMG2305UX, U201 AD9577, U202 CONN_SMA_2GND, U301 CONN_SMA, U302 CONN_SMA, U303 CONN_SMA, U304 CONN_SMA, U305 CONN_SMA, U401 ADP7158, U402 ADP7158, U403 ADP7158, U404 OKR-T/3-W12-C, U405 TPS2041B, U406 LTC1983, Y201 26 MHz 7M-26.000MEEQ-T

Commit message: vna r0 schematic cleanup
Other:
- outline, holes or cut-outs redrawn
Changed lines of the file:
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@@
     (area 22.784999 65.964999 96.595001 138.505001)
     (thickness 1.6)
-    (drawings 31)
+    (drawings 50)
     (tracks 1248)
     (zones 0)
@@
       (xy -1.425188 2.619559) (xy -1.444203 2.690827) (xy -1.390436 2.733073) (xy -1.292968 2.723896)) (layer B.SilkS) (width 0.01))
   )
+  (gr_line (start 53.086 129.667) (end 53.086 131.445) (layer Edge.Cuts) (width 0.15))
+  (gr_line (start 54.102 129.667) (end 53.086 129.667) (layer Edge.Cuts) (width 0.15))
+  (gr_line (start 54.102 132.715) (end 54.102 129.667) (layer Edge.Cuts) (width 0.15))
+  (gr_line (start 53.086 132.715) (end 54.102 132.715) (layer Edge.Cuts) (width 0.15))
+  (gr_line (start 53.086 132.588) (end 53.086 132.715) (layer Edge.Cuts) (width 0.15))
+  (gr_line (start 53.086 131.445) (end 53.086 132.588) (layer Edge.Cuts) (width 0.15))
+  (gr_line (start 47.371 133.604) (end 47.625 133.604) (layer Edge.Cuts) (width 0.15))
+  (gr_line (start 47.371 134.62) (end 47.371 133.604) (layer Edge.Cuts) (width 0.15))
+  (gr_line (start 47.498 134.62) (end 47.371 134.62) (layer Edge.Cuts) (width 0.15))
+  (gr_line (start 50.419 134.62) (end 47.498 134.62) (layer Edge.Cuts) (width 0.15))
+  (gr_line (start 50.419 133.604) (end 50.419 134.62) (layer Edge.Cuts) (width 0.15))
+  (gr_line (start 47.625 133.604) (end 50.419 133.604) (layer Edge.Cuts) (width 0.15))
+  (gr_line (start 47.371 127.635) (end 47.625 127.635) (layer Edge.Cuts) (width 0.15))
+  (gr_line (start 47.371 128.651) (end 47.371 127.635) (layer Edge.Cuts) (width 0.15))
+  (gr_line (start 47.498 128.651) (end 47.371 128.651) (layer Edge.Cuts) (width 0.15))
+  (gr_line (start 50.419 128.651) (end 47.498 128.651) (layer Edge.Cuts) (width 0.15))
+  (gr_line (start 50.419 127.635) (end 50.419 128.651) (layer Edge.Cuts) (width 0.15))
+  (gr_line (start 50.165 127.635) (end 50.419 127.635) (layer Edge.Cuts) (width 0.15))
+  (gr_line (start 47.625 127.635) (end 50.165 127.635) (layer Edge.Cuts) (width 0.15))
   (gr_text GND (at 75.565 130.81) (layer F.SilkS)
     (effects (font (size 1.5 1.5) (thickness 0.3)))
