File: hardware/vna_r0/vna_control/connectors.sch (KiCad schematic (older format))
At the start: 17 parts

Commit message: started layout of vna r0 control cape
Parts:
- added J307: BARREL_JACK, Connect:BARREL_JACK, symbol BARREL_JACK
- added R301, R302: DNP, Resistors_SMD:R_0402, symbol R_Small
- added R303: R_Small, Resistors_SMD:R_0402, symbol R_Small
- D301, D302: renamed from D?; footprint (none) -> LEDs:LED_0603
- F301: renamed from F?; footprint (none) -> Resistors_SMD:R_1206
- J301, J302, J303: renamed from J?; footprint (none) -> Pin_Headers:Pin_Header_Straight_2x10
- J304, J306: renamed from J?; footprint (none) -> Pin_Headers:Pin_Header_Straight_2x23
- J305: renamed from J?; footprint (none) -> Terminal_Blocks:TerminalBlock_Pheonix_PT-3.5mm_2pol
- Q301: renamed from Q?; footprint (none) -> TO_SOT_Packages_SMD:SOT-23
- R304, R305: renamed from R?; footprint (none) -> Resistors_SMD:R_0402
- U301, U302, U303, U304, U305: renamed from U?; footprint (none) -> vna_footprints:732511150_sma_thin
Connections:
- net labels added: DEMOD_LMX_CS, DEMOD_LMX_MUXOUT, SPI_SCK, SPI_SDI
- net labels removed: DEMOD_LMX_CSB, DEMOD_LMX_MUXout
- wire segments 195 -> 220
- no-connect marks 16 -> 24
Other:
- note added: "p68 file:///home/kleinjt/Downloads/BBB_SRM.pdf check pullups against,\nhttp://beagleboard.org/support/bone101"
- note removed: "TODO: add sense jumper"
- moved on the sheet: J304, J306

Commit message: component placement on vna cape..
Parts:
- J301, J302, J303: footprint Pin_Headers:Pin_Header_Straight_2x10 -> Connect:IDC_Header_Straight_20pins
Connections:
- net labels added: +3V3
- wire segments 220 -> 222
Changed lines of the file:
@@
 F 0 "J301" H 2350 3650 50  0000 C CNN
 F 1 "CONN_02X10" V 2350 3100 50  0000 C CNN
-F 2 "Pin_Headers:Pin_Header_Straight_2x10" H 2350 1900 50  0001 C CNN
+F 2 "Connect:IDC_Header_Straight_20pins" H 2350 1900 50  0001 C CNN
 F 3 "" H 2350 1900 50  0001 C CNN
 	1    2350 3100
@@
 F 0 "J302" H 2350 4950 50  0000 C CNN
 F 1 "CONN_02X10" V 2350 4400 50  0000 C CNN
-F 2 "Pin_Headers:Pin_Header_Straight_2x10" H 2350 3200 50  0001 C CNN
+F 2 "Connect:IDC_Header_Straight_20pins" H 2350 3200 50  0001 C CNN
 F 3 "" H 2350 3200 50  0001 C CNN
 	1    2350 4400
@@
 F 0 "J303" H 2350 6600 50  0000 C CNN
 F 1 "CONN_02X10" V 2350 6050 50  0000 C CNN
-F 2 "Pin_Headers:Pin_Header_Straight_2x10" H 2350 4850 50  0001 C CNN
+F 2 "Connect:IDC_Header_Straight_20pins" H 2350 4850 50  0001 C CNN
 F 3 "" H 2350 4850 50  0001 C CNN
 	1    2350 6050
@@
 Text HLabel 3750 6100 2    60   Input ~ 0
 3V3_RF_SENSE
-Text Label 9750 5400 1    60   ~ 0
-3V3_RF
 Text HLabel 1300 6150 0    60   Input ~ 0
 3V3_RF
@@
 Text Notes 7550 4050 0    60   ~ 0
 p68 file:///home/kleinjt/Downloads/BBB_SRM.pdf check pullups against,\nhttp://beagleboard.org/support/bone101
+$Comp
+L +3V3 #PWR081
+U 1 1 595C92A3
+P 9750 5400
+F 0 "#PWR081" H 9750 5250 50  0001 C CNN
+F 1 "+3V3" H 9750 5540 50  0000 C CNN
+F 2 "" H 9750 5400 50  0001 C CNN
+F 3 "" H 9750 5400 50  0001 C CNN
+	1    9750 5400
+	1    0    0    -1
+$EndComp
+Wire Wire Line
+	9750 6100 9750 6150
+Wire Wire Line
+	10100 6100 10100 6150
 $EndSCHEMATC

Commit message: layout of control cape..
Connections:
- no-connect marks 24 -> 25
Changed lines of the file:
@@
 $EndComp
 $Comp
-L -5V #PWR321
+L -5V #PWR322
 U 1 1 595B7B2D
 P 10100 5400
-F 0 "#PWR321" H 10100 5500 50  0001 C CNN
+F 0 "#PWR322" H 10100 5500 50  0001 C CNN
 F 1 "-5V" V 10100 5600 50  0000 C CNN
 F 2 "" H 10100 5400 50  0001 C CNN
@@
 Wire Wire Line
 	10100 6100 10100 6150
+NoConn ~ 7400 3000
 $EndSCHEMATC

Commit message: vna control cape layout - all nets connected
Changed lines of the file:
@@
 	1    0    0    -1
 $EndComp
-Text HLabel 5200 4200 0    60   Input ~ 0
+Text HLabel 5200 2950 0    60   Input ~ 0
 SYNTH_REF_A
 $Comp
@@
 	1    0    0    -1
 $EndComp
-Text HLabel 5200 2950 0    60   Input ~ 0
+Text HLabel 5200 4200 0    60   Input ~ 0
 SYNTH_REF_B
 $Comp
@@
 Text Notes 7950 4650 0    60   ~ 0
 5V input
+Text HLabel 10200 1450 2    60   Input ~ 0
+3V3_RF_EN
 Text HLabel 10200 1550 2    60   Input ~ 0
-3V3_RF_EN
-Text HLabel 10200 1650 2    60   Input ~ 0
 3V3_DEMOD_EN
 Text HLabel 10200 1750 2    60   Input ~ 0
@@
 Text HLabel 10200 1350 2    60   Input ~ 0
 PLL_REF_SEL
-Text HLabel 10200 1450 2    60   Input ~ 0
+Text HLabel 10200 1650 2    60   Input ~ 0
 3V3_PLL_EN
 $Comp
@@
 Text Label 8100 1600 0    60   ~ 0
 AD_PD
-Text Label 10200 2250 0    60   ~ 0
+Text Label 7400 2400 2    60   ~ 0
 AD_DOUTB
+Text Label 8100 1800 0    60   ~ 0
+AD_PE_A
+Text Label 8100 2300 0    60   ~ 0
+AD_PE_B
 Text Label 8100 1900 0    60   ~ 0
-AD_PE_A
-Text Label 8100 1800 0    60   ~ 0
-AD_PE_B
-Text Label 8100 2300 0    60   ~ 0
 AD_PE_C
 Text Label 8100 2200 0    60   ~ 0
 AD_PE_D
-Text Label 9500 1750 2    60   ~ 0
+Text Label 10200 2350 0    60   ~ 0
 MIX_EN
-Text Label 9500 1850 2    60   ~ 0
+Text Label 9500 2350 2    60   ~ 0
 MIX_X2
 Wire Wire Line
@@
 Wire Wire Line
 	9600 1350 9500 1350
-Text Label 9500 1350 2    60   ~ 0
+Text Label 9500 2450 2    60   ~ 0
 IF_REF_EN
-Text Label 9500 1450 2    60   ~ 0
+Text Label 10200 2450 0    60   ~ 0
 ADC_CLK_EN
 $Comp
@@
 Text Label 7400 1600 2    60   ~ 0
 RF_LMX_MUXOUT
-Text Label 9500 1550 2    60   ~ 0
+Text Label 7400 1700 2    60   ~ 0
 RF_LMX_CE
-Text Label 7400 2400 2    60   ~ 0
+Text Label 7400 1800 2    60   ~ 0
 RF_PORT_SEL
 Text Label 7400 1900 2    60   ~ 0
 RF_DAC_CS
-Text Label 7400 2300 2    60   ~ 0
+Text Label 7400 2200 2    60   ~ 0
 RF_SW_2
 Text Label 8100 2100 0    60   ~ 0
@@
 Text Label 7400 2100 2    60   ~ 0
 RF_DAC_SDI
-Text Label 7400 2200 2    60   ~ 0
+Text Label 7400 2300 2    60   ~ 0
 RF_SW_1
 Text Label 8100 2400 0    60   ~ 0
@@
 Text Label 8100 3100 0    60   ~ 0
 DEMOD_LMX_CS
-Text Label 9500 1650 2    60   ~ 0
+Text Label 7400 3100 2    60   ~ 0
 DEMOD_LMX_CE
-Text Label 7400 1700 2    60   ~ 0
+Text Label 8100 2500 0    60   ~ 0
 DEMOD_LMX_MUXOUT
 NoConn ~ 10200 1950

Commit message: finished vna control cape
Connections:
- wire segments 222 -> 226
- no-connect marks 25 -> 21
Changed lines of the file:
@@
 $EndComp
 $Comp
-L GND #PWR060
+L GND #PWR062
 U 1 1 595A012F
 P 8100 1100
-F 0 "#PWR060" H 8100 850 50  0001 C CNN
+F 0 "#PWR062" H 8100 850 50  0001 C CNN
 F 1 "GND" H 8100 950 50  0000 C CNN
 F 2 "" H 8100 1100 50  0001 C CNN
@@
 BeagleBone P8
 $Comp
-L GND #PWR061
+L GND #PWR063
 U 1 1 595A027F
 P 7400 1100
-F 0 "#PWR061" H 7400 850 50  0001 C CNN
+F 0 "#PWR063" H 7400 850 50  0001 C CNN
 F 1 "GND" H 7400 950 50  0000 C CNN
 F 2 "" H 7400 1100 50  0001 C CNN
@@
 $EndComp
 $Comp
-L GND #PWR062
+L GND #PWR064
 U 1 1 595B1ED9
 P 5950 4800
-F 0 "#PWR062" H 5950 4550 50  0001 C CNN
+F 0 "#PWR064" H 5950 4550 50  0001 C CNN
 F 1 "GND" H 5950 4650 50  0000 C CNN
 F 2 "" H 5950 4800 50  0001 C CNN
@@
 $EndComp
 $Comp
-L GND #PWR063
+L GND #PWR065
 U 1 1 595B21C7
 P 5950 3550
-F 0 "#PWR063" H 5950 3300 50  0001 C CNN
+F 0 "#PWR065" H 5950 3300 50  0001 C CNN
 F 1 "GND" H 5950 3400 50  0000 C CNN
 F 2 "" H 5950 3550 50  0001 C CNN
@@
 $EndComp
 $Comp
-L GND #PWR064
+L GND #PWR066
 U 1 1 595B225E
 P 5950 5850
-F 0 "#PWR064" H 5950 5600 50  0001 C CNN
+F 0 "#PWR066" H 5950 5600 50  0001 C CNN
 F 1 "GND" H 5950 5700 50  0000 C CNN
 F 2 "" H 5950 5850 50  0001 C CNN
@@
 $EndComp
 $Comp
-L GND #PWR065
+L GND #PWR067
 U 1 1 595B2825
 P 10200 1050
-F 0 "#PWR065" H 10200 800 50  0001 C CNN
+F 0 "#PWR067" H 10200 800 50  0001 C CNN
 F 1 "GND" H 10200 900 50  0000 C CNN
 F 2 "" H 10200 1050 50  0001 C CNN
@@
 	0    -1   -1   0
 $EndComp
-NoConn ~ 9600 1150
-NoConn ~ 9600 1250
-NoConn ~ 10100 1250
-NoConn ~ 10100 1150
-$Comp
-L GND #PWR066
+$Comp
+L GND #PWR068
 U 1 1 595B2834
 P 9500 1050
-F 0 "#PWR066" H 9500 800 50  0001 C CNN
+F 0 "#PWR068" H 9500 800 50  0001 C CNN
 F 1 "GND" H 9500 900 50  0000 C CNN
 F 2 "" H 9500 1050 50  0001 C CNN
@@
 $EndComp
 $Comp
-L GND #PWR067
+L GND #PWR069
 U 1 1 595B29C7
 P 2750 2900
-F 0 "#PWR067" H 2750 2650 50  0001 C CNN
+F 0 "#PWR069" H 2750 2650 50  0001 C CNN
 F 1 "GND" H 2750 2750 50  0000 C CNN
 F 2 "" H 2750 2900 50  0001 C CNN
@@
 DEMOD_LMX_MUXOUT
 $Comp
-L GND #PWR068
+L GND #PWR070
 U 1 1 595B3C95
 P 2750 4400
-F 0 "#PWR068" H 2750 4150 50  0001 C CNN
+F 0 "#PWR070" H 2750 4150 50  0001 C CNN
 F 1 "GND" H 2750 4250 50  0000 C CNN
 F 2 "" H 2750 4400 50  0001 C CNN
@@
 DEMOD_LMX_CE
 $Comp
-L GND #PWR069
+L GND #PWR071
 U 1 1 595B4764
 P 1950 4550
-F 0 "#PWR069" H 1950 4300 50  0001 C CNN
+F 0 "#PWR071" H 1950 4300 50  0001 C CNN
 F 1 "GND" H 1950 4400 50  0000 C CNN
 F 2 "" H 1950 4550 50  0001 C CNN
@@
 RF_SW_2
 $Comp
-L GND #PWR070
+L GND #PWR072
 U 1 1 595B58A3
 P 1950 5800
-F 0 "#PWR070" H 1950 5550 50  0001 C CNN
+F 0 "#PWR072" H 1950 5550 50  0001 C CNN
 F 1 "GND" H 1950 5650 50  0000 C CNN
 F 2 "" H 1950 5800 50  0001 C CNN
@@
 $EndComp
 $Comp
-L GND #PWR071
+L GND #PWR073
 U 1 1 595B7B5C
 P 10100 6150
-F 0 "#PWR071" H 10100 5900 50  0001 C CNN
+F 0 "#PWR073" H 10100 5900 50  0001 C CNN
 F 1 "GND" H 10100 6000 50  0000 C CNN
 F 2 "" H 10100 6150 50  0001 C CNN
@@
 $EndComp
 $Comp
-L GND #PWR072
+L GND #PWR074
 U 1 1 595B7B8B
 P 9750 6150
-F 0 "#PWR072" H 9750 5900 50  0001 C CNN
+F 0 "#PWR074" H 9750 5900 50  0001 C CNN
 F 1 "GND" H 9750 6000 50  0000 C CNN
 F 2 "" H 9750 6150 50  0001 C CNN
@@
 $EndComp
 $Comp
-L GND #PWR073
+L GND #PWR075
 U 1 1 595B252F
 P 6000 7100
-F 0 "#PWR073" H 6000 6850 50  0001 C CNN
+F 0 "#PWR075" H 6000 6850 50  0001 C CNN
 F 1 "GND" H 6000 6950 50  0000 C CNN
 F 2 "" H 6000 7100 50  0001 C CNN
@@
 $EndComp
 $Comp
-L +5V #PWR074
+L +5V #PWR076
 U 1 1 595CF1E4
 P 8550 6150
-F 0 "#PWR074" H 8550 6000 50  0001 C CNN
+F 0 "#PWR076" H 8550 6000 50  0001 C CNN
 F 1 "+5V" H 8550 6290 50  0000 C CNN
 F 2 "" H 8550 6150 50  0001 C CNN
@@
 	7850 5300 8200 5300
 $Comp
-L GND #PWR075
+L GND #PWR077
 U 1 1 595CF412
 P 8050 6150
-F 0 "#PWR075" H 8050 5900 50  0001 C CNN
+F 0 "#PWR077" H 8050 5900 50  0001 C CNN
 F 1 "GND" H 8050 6000 50  0000 C CNN
 F 2 "" H 8050 6150 50  0001 C CNN
@@
 $EndComp
 $Comp
-L GND #PWR076
+L GND #PWR078
 U 1 1 595D5C6E
 P 5950 2250
-F 0 "#PWR076" H 5950 2000 50  0001 C CNN
+F 0 "#PWR078" H 5950 2000 50  0001 C CNN
 F 1 "GND" H 5950 2100 50  0000 C CNN
 F 2 "" H 5950 2250 50  0001 C CNN
@@
 NoConn ~ 7400 2700
 $Comp
-L GND #PWR077
+L GND #PWR079
 U 1 1 595FA985
 P 8100 2700
-F 0 "#PWR077" H 8100 2450 50  0001 C CNN
+F 0 "#PWR079" H 8100 2450 50  0001 C CNN
 F 1 "GND" H 8100 2550 50  0000 C CNN
 F 2 "" H 8100 2700 50  0001 C CNN
@@
 $EndComp
 $Comp
-L GND #PWR078
+L GND #PWR080
 U 1 1 595FAC0E
 P 8100 3350
-F 0 "#PWR078" H 8100 3100 50  0001 C CNN
+F 0 "#PWR080" H 8100 3100 50  0001 C CNN
 F 1 "GND" H 8100 3200 50  0000 C CNN
 F 2 "" H 8100 3350 50  0001 C CNN
@@
 Connection ~ 8100 3300
 $Comp
-L GND #PWR079
+L GND #PWR081
 U 1 1 595FAEBC
 P 7400 3350
-F 0 "#PWR079" H 7400 3100 50  0001 C CNN
+F 0 "#PWR081" H 7400 3100 50  0001 C CNN
 F 1 "GND" H 7400 3200 50  0000 C CNN
 F 2 "" H 7400 3350 50  0001 C CNN
@@
 $EndComp
 $Comp
-L +5V #PWR080
+L +5V #PWR082
 U 1 1 595FB931
 P 6900 800
-F 0 "#PWR080" H 6900 650 50  0001 C CNN
+F 0 "#PWR082" H 6900 650 50  0001 C CNN
 F 1 "+5V" H 6900 940 50  0000 C CNN
 F 2 "" H 6900 800 50  0001 C CNN
@@
 p68 file:///home/kleinjt/Downloads/BBB_SRM.pdf check pullups against,\nhttp://beagleboard.org/support/bone101
 $Comp
-L +3V3 #PWR081
+L +3V3 #PWR083
 U 1 1 595C92A3
 P 9750 5400
-F 0 "#PWR081" H 9750 5250 50  0001 C CNN
+F 0 "#PWR083" H 9750 5250 50  0001 C CNN
 F 1 "+3V3" H 9750 5540 50  0000 C CNN
 F 2 "" H 9750 5400 50  0001 C CNN
@@
 	10100 6100 10100 6150
 NoConn ~ 7400 3000
+Wire Wire Line
+	9500 1150 9600 1150
+Wire Wire Line
+	9500 1250 9600 1250
+Wire Wire Line
+	10100 1150 10200 1150
+Wire Wire Line
+	10100 1250 10200 1250
 $EndSCHEMATC

Commit message: change all LED current limited resistors from 1k to 10k...
Parts:
- R304, R305: value 1k -> 10k
Changed lines of the file:
@@
 P 9750 5600
 F 0 "R304" H 9780 5620 50  0000 L CNN
-F 1 "1k" H 9780 5560 50  0000 L CNN
+F 1 "10k" H 9780 5560 50  0000 L CNN
 F 2 "Resistors_SMD:R_0402" H 9750 5600 50  0001 C CNN
 F 3 "" H 9750 5600 50  0001 C CNN
@@
 P 10100 5600
 F 0 "R305" H 10130 5620 50  0000 L CNN
-F 1 "1k" H 10130 5560 50  0000 L CNN
+F 1 "10k" H 10130 5560 50  0000 L CNN
 F 2 "Resistors_SMD:R_0402" H 10100 5600 50  0001 C CNN
 F 3 "" H 10100 5600 50  0001 C CNN

Commit message: work on vna r1 schematic..
Other:
- note added: "1.2V"
- note added: "TODO - isolate P8-46 to P8-31 with highz buffer chip to avoid fighting boot config resistors"
- note added: "gnd"
- note added: "high"
- note added: "low"
Changed lines of the file:
@@
 Wire Wire Line
 	10100 1250 10200 1250
+Text Notes 10800 3150 1    60   ~ 0
+gnd
+Text Notes 8900 3250 2    60   ~ 0
+gnd
+Text Notes 9000 2950 3    60   ~ 0
+1.2V
+Text Notes 8900 3300 2    60   ~ 12
+low
+Text Notes 10900 3250 2    60   ~ 12
+low
+Text Notes 11050 3150 2    60   ~ 12
+high
+Text Notes 11050 3050 2    60   ~ 12
+high
+Text Notes 10900 2950 2    60   ~ 12
+low
+Text Notes 8850 3000 2    60   ~ 12
+high
+Text Notes 8850 3100 2    60   ~ 12
+high
+Text Notes 8600 3500 0    60   ~ 12
+TODO - isolate P8-46 to P8-31 with highz buffer chip to avoid fighting boot config resistors
 $EndSCHEMATC
