File: breakouts/amp_macom_vga/amp_macom_vga.sch (KiCad schematic (older format))
At the start: 52 parts, among them J101 RF_Shield_Two_Pieces, J102 CONN_01X02, J103 CONN_01X04, Q101 DMG2305UX, Q102 DMG2305UX, U101 CONN_SMA_2GND, U102 LM2776, U103 LTC2630, U104 MAAM-011100, U105 CONN_SMA_2GND, U106 LTC2054HV, U107 MAX810MTRG

Commit message: finished maam-011100 board
Parts:
- JP101: footprint Pin_Headers:Pin_Header_Straight_1x03 -> vna_footprints:JMP_3
- RV101: footprint Potentiometers:Potentiometer_Bourns_3296W_3-8Zoll_Inline_ScrewUp -> SMD_Packages:POT_SMD
Changed lines of the file:
@@
 F 0 "RV101" V 2775 4550 50  0000 C CNN
 F 1 "POT" V 2850 4550 50  0000 C CNN
-F 2 "Potentiometers:Potentiometer_Bourns_3296W_3-8Zoll_Inline_ScrewUp" H 2950 4550 50  0001 C CNN
+F 2 "SMD_Packages:POT_SMD" H 2950 4550 50  0001 C CNN
 F 3 "" H 2950 4550 50  0001 C CNN
 	1    2950 4550
@@
 F 0 "JP101" H 3650 4450 50  0000 L CNN
 F 1 "Jumper_NC_Dual" H 3600 4650 50  0000 C BNN
-F 2 "Pin_Headers:Pin_Header_Straight_1x03" H 3600 4550 50  0001 C CNN
+F 2 "vna_footprints:JMP_3" H 3600 4550 50  0001 C CNN
 F 3 "" H 3600 4550 50  0001 C CNN
 	1    3600 4550
