File: hardware/vna_r1/power.sch (KiCad schematic (older format))
At the start: 40 parts, among them J901 CONN_01X02, U901 ADP7158, U902 ADP7158, U903 ADP7158, U904 OKR-T/3-W12-C, U905 TPS2041B, U906 LTC1983

Commit message: layout on vna r1 control board
Parts:
- removed C902, C913, C919, C921: 10 uF, Capacitors_SMD:C_0603, symbol C_Small
- removed C904, C907, C910, C923: 1 uF, Capacitors_SMD:C_0402, symbol C_Small
- removed C918, C920, C922, C924, C925: 100 nF, Capacitors_SMD:C_0402, symbol C_Small
- removed C926: 100 pF, Capacitors_SMD:C_0402, symbol C_Small
- removed L901: L_Small, Resistors_SMD:R_0805, symbol L_Small
- removed R905, R906: 10k, Resistors_SMD:R_0402, symbol R_Small
- removed U901: ADP7158, Housings_DFN_QFN:DFN-10-1EP_3x3mm_Pitch0.5mm, symbol ADP7158
- removed U905: TPS2041B, TO_SOT_Packages_SMD:SOT-23-5, symbol TPS2041B
- removed U906: LTC1983, TO_SOT_Packages_SMD:SOT-23-6, symbol LTC1983
Connections:
- net labels removed: -5V, -5V_EN, 3V3_RF_EN, 3V3_RF_SENSE, AMP_5V, RF_AMP_EN, VDD_RF
- wire segments 130 -> 68
- no-connect marks 2 -> 1
Other:
- note removed: "a few mA"
- note removed: "provide switched (interlocked?) 5V supply for amplifier, 70 mA"
- note removed: "switch to lower cost LTC2054CS5?"

Commit message: more work on vna r1..
Parts:
- added L601: L_Small, Resistors_SMD:R_0402, symbol L_Small
Connections:
- net USB_DC: now also L601.2
- net VDD_RTC: now also L601.1
Changed lines of the file:
@@
 	-1   0    0    1
 $EndComp
+$Comp
+L VDD_LO #SUPPLY0227
+U 1 1 5AAB674C
+P 1100 6400
+F 0 "#SUPPLY0227" H 1100 6400 45  0001 L BNN
+F 1 "VDD_LO" H 1100 6550 45  0000 L BNN
+F 2 "" H 1100 6400 60  0001 C CNN
+F 3 "" H 1100 6400 60  0001 C CNN
+	1    1100 6400
+	1    0    0    -1
+$EndComp
+$Comp
+L VDD_CLK #SUPPLY0228
+U 1 1 5AAB6796
+P 1500 6400
+F 0 "#SUPPLY0228" H 1500 6400 45  0001 L BNN
+F 1 "VDD_CLK" H 1500 6560 45  0000 L BNN
+F 2 "" H 1500 6400 60  0001 C CNN
+F 3 "" H 1500 6400 60  0001 C CNN
+	1    1500 6400
+	1    0    0    -1
+$EndComp
+Wire Wire Line
+	1100 6500 1100 6550
+Wire Wire Line
+	1100 6550 1200 6550
+Wire Wire Line
+	1400 6550 1500 6550
+Wire Wire Line
+	1500 6550 1500 6500
+$Comp
+L L_Small L601
+U 1 1 5AAB6A5A
+P 1300 6550
+F 0 "L601" H 1330 6590 50  0000 L CNN
+F 1 "L_Small" H 1330 6510 50  0000 L CNN
+F 2 "Resistors_SMD:R_0402" H 1300 6550 50  0001 C CNN
+F 3 "" H 1300 6550 50  0001 C CNN
+	1    1300 6550
+	0    1    1    0
+$EndComp
 $EndSCHEMATC

Commit message: footprint assignment for vna r1 synth and demod
Parts:
- removed C903, C914: 10 uF, Capacitors_SMD:C_0603, symbol C_Small
- removed C905, C908, C911: 1 uF, Capacitors_SMD:C_0402, symbol C_Small
- removed L601: L_Small, Resistors_SMD:R_0402, symbol L_Small
- removed U902: ADP7158, Housings_DFN_QFN:DFN-10-1EP_3x3mm_Pitch0.5mm, symbol ADP7158
Connections:
- net VDD_RTC renamed +3V3

Commit message: component placement on vna r1 demod
Parts:
- removed C916: 100 uF, Capacitors_SMD:c_elec_10x10, symbol C_Small
- added R602: R_Small, Resistors_SMD:R_0402, symbol R_Small
Connections:
- net +3V3: now also R602.2
- net 3V3_PLL_SENSE: no longer names the net of U903.3 (VOUT_SENSE)
- net 3V3_PLL_SENSE: now also R602.1
Changed lines of the file:
@@
 	2650 8250 2650 8300
 Wire Wire Line
-	2700 7850 3300 7850
+	2400 7850 3300 7850
 $Comp
 L R_Small R901
@@
 Wire Wire Line
 	3150 7750 3150 7650
-Text HLabel 2700 7850 0    60   Input ~ 0
-3V3_PLL_SENSE
-Wire Wire Line
-	7100 7100 7100 7450
-Wire Wire Line
-	7100 7650 7100 8000
 $Comp
-L GND #PWR0216
-U 1 1 595F6EEE
-P 7100 8000
-F 0 "#PWR0216" H 7100 7750 50  0001 C CNN
-F 1 "GND" H 7100 7850 50  0000 C CNN
-F 2 "" H 7100 8000 50  0001 C CNN
-F 3 "" H 7100 8000 50  0001 C CNN
-	1    7100 8000
-	1    0    0    -1
-$EndComp
-$Comp
-L +5V #PWR0217
-U 1 1 595F6D3F
-P 7100 7100
-F 0 "#PWR0217" H 7100 6950 50  0001 C CNN
-F 1 "+5V" H 7100 7240 50  0000 C CNN
-F 2 "" H 7100 7100 50  0001 C CNN
-F 3 "" H 7100 7100 50  0001 C CNN
-	1    7100 7100
-	1    0    0    -1
-$EndComp
-$Comp
-L C_Small C916
-U 1 1 595F6B79
-P 7100 7550
-F 0 "C916" H 7110 7620 50  0000 L CNN
-F 1 "100 uF" H 7110 7470 50  0000 L CNN
-F 2 "Capacitors_SMD:c_elec_10x10" H 7100 7550 50  0001 C CNN
-F 3 "" H 7100 7550 50  0001 C CNN
-	1    7100 7550
-	-1   0    0    1
-$EndComp
-$Comp
-L +3V3 #PWR0218
+L +3V3 #PWR0216
 U 1 1 5ACC44BC
 P 1600 7650
-F 0 "#PWR0218" H 1600 7500 50  0001 C CNN
+F 0 "#PWR0216" H 1600 7500 50  0001 C CNN
 F 1 "+3V3" H 1600 7790 50  0000 C CNN
 F 2 "" H 1600 7650 50  0001 C CNN
@@
 	0    -1   -1   0
 $EndComp
+$Comp
+L R_Small R602
+U 1 1 5AD576A9
+P 2300 7850
+F 0 "R602" H 2330 7870 50  0000 L CNN
+F 1 "R_Small" H 2330 7810 50  0000 L CNN
+F 2 "Resistors_SMD:R_0402" H 2300 7850 50  0001 C CNN
+F 3 "" H 2300 7850 50  0001 C CNN
+	1    2300 7850
+	0    1    1    0
+$EndComp
+Wire Wire Line
+	2200 7850 2000 7850
+Wire Wire Line
+	2000 7850 2000 7650
+Connection ~ 2000 7650
 $EndSCHEMATC

Commit message: finished vna r1 control board?
Parts:
- added D901, D902: LED_Small, LEDs:LED_0603, symbol LED_Small
- added R905, R907: 10k, Resistors_SMD:R_0402, symbol R_Small
- R901: value R_Small -> DNP
- R902: value R_Small -> 10k
- R906: renamed from R602; value R_Small -> JMP
Connections:
- net +5V: now also D902.2 (A)
- net GND: now also J901.1 (P1), R905.2, R907.2; no longer J901.2 (P2)
- net VPP: now also J901.2 (P2), D901.2 (A); no longer J901.1 (P1)
- new net: D901.1 (K), R905.1
- new net: D902.1 (K), R907.1
Other:
- note removed: "3.3V,\n500 mA for RF\n1200 mA for demod\n500 mA for PLL"
Changed lines of the file:
@@
 Comment4 ""
 $EndDescr
-Text Notes 3400 3200 0    60   ~ 0
-3.3V,\n500 mA for RF\n1200 mA for demod\n500 mA for PLL
 $Comp
 L OKR-T/3-W12-C U904
@@
 $EndComp
 $Comp
-L VPP #PWR614
+L VPP #PWR0201
 U 1 1 595CA82E
 P 9550 7050
-F 0 "#PWR614" H 9550 6900 50  0001 C CNN
+F 0 "#PWR0201" H 9550 6900 50  0001 C CNN
 F 1 "VPP" H 9550 7200 50  0000 C CNN
 F 2 "" H 9550 7050 50  0001 C CNN
@@
 	9550 7150 9550 7050
 $Comp
-L GND #PWR613
+L GND #PWR0202
 U 1 1 595CA9A5
 P 8700 8000
-F 0 "#PWR613" H 8700 7750 50  0001 C CNN
+F 0 "#PWR0202" H 8700 7750 50  0001 C CNN
 F 1 "GND" H 8700 7850 50  0000 C CNN
 F 2 "" H 8700 8000 50  0001 C CNN
@@
 $EndComp
 $Comp
-L GND #PWR616
+L GND #PWR0203
 U 1 1 595CAE17
+P 15300 7900
+F 0 "#PWR0203" H 15300 7650 50  0001 C CNN
+F 1 "GND" H 15300 7750 50  0000 C CNN
+F 2 "" H 15300 7900 50  0001 C CNN
+F 3 "" H 15300 7900 50  0001 C CNN
+	1    15300 7900
+	1    0    0    -1
+$EndComp
+$Comp
+L VPP #PWR0204
+U 1 1 595CAF0A
 P 15400 7900
-F 0 "#PWR616" H 15400 7650 50  0001 C CNN
-F 1 "GND" H 15400 7750 50  0000 C CNN
+F 0 "#PWR0204" H 15400 7750 50  0001 C CNN
+F 1 "VPP" H 15400 8050 50  0000 C CNN
 F 2 "" H 15400 7900 50  0001 C CNN
 F 3 "" H 15400 7900 50  0001 C CNN
 	1    15400 7900
-	1    0    0    -1
-$EndComp
-$Comp
-L VPP #PWR615
-U 1 1 595CAF0A
-P 15300 7900
-F 0 "#PWR615" H 15300 7750 50  0001 C CNN
-F 1 "VPP" H 15300 8050 50  0000 C CNN
-F 2 "" H 15300 7900 50  0001 C CNN
-F 3 "" H 15300 7900 50  0001 C CNN
-	1    15300 7900
-	-1   0    0    1
-$EndComp
-Wire Wire Line
-	15300 7700 15300 7900
-Wire Wire Line
-	15400 7900 15400 7700
-$Comp
-L +5V #PWR611
+	-1   0    0    1
+$EndComp
+Wire Wire Line
+	15400 7700 15400 7900
+Wire Wire Line
+	15300 7900 15300 7700
+$Comp
+L +5V #PWR0205
 U 1 1 595CB86B
 P 7600 7100
-F 0 "#PWR611" H 7600 6950 50  0001 C CNN
+F 0 "#PWR0205" H 7600 6950 50  0001 C CNN
 F 1 "+5V" H 7600 7240 50  0000 C CNN
 F 2 "" H 7600 7100 50  0001 C CNN
@@
 $EndComp
 $Comp
-L GND #PWR612
+L GND #PWR0206
 U 1 1 595CDAB9
 P 7600 8000
-F 0 "#PWR612" H 7600 7750 50  0001 C CNN
+F 0 "#PWR0206" H 7600 7750 50  0001 C CNN
 F 1 "GND" H 7600 7850 50  0000 C CNN
 F 2 "" H 7600 8000 50  0001 C CNN
@@
 $EndComp
 $Comp
-L GND #PWR606
+L GND #PWR0207
 U 1 1 595D24C4
 P 3900 8600
-F 0 "#PWR606" H 3900 8350 50  0001 C CNN
+F 0 "#PWR0207" H 3900 8350 50  0001 C CNN
 F 1 "GND" H 3900 8450 50  0000 C CNN
 F 2 "" H 3900 8600 50  0001 C CNN
@@
 $EndComp
 $Comp
-L GND #PWR607
+L GND #PWR0208
 U 1 1 595D24D0
 P 4750 8600
-F 0 "#PWR607" H 4750 8350 50  0001 C CNN
+F 0 "#PWR0208" H 4750 8350 50  0001 C CNN
 F 1 "GND" H 4750 8450 50  0000 C CNN
 F 2 "" H 4750 8600 50  0001 C CNN
@@
 $EndComp
 $Comp
-L GND #PWR608
+L GND #PWR0209
 U 1 1 595D24DC
 P 5150 8600
-F 0 "#PWR608" H 5150 8350 50  0001 C CNN
+F 0 "#PWR0209" H 5150 8350 50  0001 C CNN
 F 1 "GND" H 5150 8450 50  0000 C CNN
 F 2 "" H 5150 8600 50  0001 C CNN
@@
 $EndComp
 $Comp
-L GND #PWR610
+L GND #PWR0210
 U 1 1 595D24E8
 P 5450 8600
-F 0 "#PWR610" H 5450 8350 50  0001 C CNN
+F 0 "#PWR0210" H 5450 8350 50  0001 C CNN
 F 1 "GND" H 5450 8450 50  0000 C CNN
 F 2 "" H 5450 8600 50  0001 C CNN
@@
 $EndComp
 $Comp
-L VPP #PWR609
+L VPP #PWR0211
 U 1 1 595D24EE
 P 5450 7650
-F 0 "#PWR609" H 5450 7500 50  0001 C CNN
+F 0 "#PWR0211" H 5450 7500 50  0001 C CNN
 F 1 "VPP" H 5450 7800 50  0000 C CNN
 F 2 "" H 5450 7650 50  0001 C CNN
@@
 $EndComp
 $Comp
-L GND #PWR602
+L GND #PWR0212
 U 1 1 595D24FA
 P 1800 8300
-F 0 "#PWR602" H 1800 8050 50  0001 C CNN
+F 0 "#PWR0212" H 1800 8050 50  0001 C CNN
 F 1 "GND" H 1800 8150 50  0000 C CNN
 F 2 "" H 1800 8300 50  0001 C CNN
@@
 	2650 7950 2650 8050
 $Comp
-L GND #PWR603
+L GND #PWR0213
 U 1 1 595D2520
 P 2650 8300
-F 0 "#PWR603" H 2650 8050 50  0001 C CNN
+F 0 "#PWR0213" H 2650 8050 50  0001 C CNN
 F 1 "GND" H 2650 8150 50  0000 C CNN
 F 2 "" H 2650 8300 50  0001 C CNN
@@
 P 2900 8350
 F 0 "R901" H 2930 8370 50  0000 L CNN
-F 1 "R_Small" H 2930 8310 50  0000 L CNN
+F 1 "DNP" H 2930 8310 50  0000 L CNN
 F 2 "Resistors_SMD:R_0402" H 2900 8350 50  0001 C CNN
 F 3 "" H 2900 8350 50  0001 C CNN
@@
 P 2900 8700
 F 0 "R902" H 2930 8720 50  0000 L CNN
-F 1 "R_Small" H 2930 8660 50  0000 L CNN
+F 1 "10k" H 2930 8660 50  0000 L CNN
 F 2 "Resistors_SMD:R_0402" H 2900 8700 50  0001 C CNN
 F 3 "" H 2900 8700 50  0001 C CNN
@@
 $EndComp
 $Comp
-L GND #PWR605
+L GND #PWR0214
 U 1 1 595D28FE
 P 2900 8950
-F 0 "#PWR605" H 2900 8700 50  0001 C CNN
+F 0 "#PWR0214" H 2900 8700 50  0001 C CNN
 F 1 "GND" H 2900 8800 50  0000 C CNN
 F 2 "" H 2900 8950 50  0001 C CNN
@@
 	3150 8050 3150 8550
 $Comp
-L VPP #PWR604
+L VPP #PWR0215
 U 1 1 595D3935
 P 2900 8200
-F 0 "#PWR604" H 2900 8050 50  0001 C CNN
+F 0 "#PWR0215" H 2900 8050 50  0001 C CNN
 F 1 "VPP" H 2900 8350 50  0000 C CNN
 F 2 "" H 2900 8200 50  0001 C CNN
@@
 	3150 7750 3150 7650
 $Comp
-L +3V3 #PWR601
+L +3V3 #PWR0216
 U 1 1 5ACC44BC
 P 1600 7650
-F 0 "#PWR601" H 1600 7500 50  0001 C CNN
+F 0 "#PWR0216" H 1600 7500 50  0001 C CNN
 F 1 "+3V3" H 1600 7790 50  0000 C CNN
 F 2 "" H 1600 7650 50  0001 C CNN
@@
 $EndComp
 $Comp
-L R_Small R602
+L R_Small R906
 U 1 1 5AD576A9
 P 2300 7850
-F 0 "R602" H 2330 7870 50  0000 L CNN
-F 1 "R_Small" H 2330 7810 50  0000 L CNN
+F 0 "R906" H 2330 7870 50  0000 L CNN
+F 1 "JMP" H 2330 7810 50  0000 L CNN
 F 2 "Resistors_SMD:R_0402" H 2300 7850 50  0001 C CNN
 F 3 "" H 2300 7850 50  0001 C CNN
@@
 	2000 7850 2000 7650
 Connection ~ 2000 7650
+$Comp
+L LED_Small D901
+U 1 1 5AF079B4
+P 5450 6100
+F 0 "D901" H 5400 6225 50  0000 L CNN
+F 1 "LED_Small" H 5275 6000 50  0000 L CNN
+F 2 "LEDs:LED_0603" V 5450 6100 50  0001 C CNN
+F 3 "" V 5450 6100 50  0001 C CNN
+	1    5450 6100
+	0    -1   -1   0
+$EndComp
+$Comp
+L VPP #PWR0217
+U 1 1 5AF07A56
+P 5450 5800
+F 0 "#PWR0217" H 5450 5650 50  0001 C CNN
+F 1 "VPP" H 5450 5950 50  0000 C CNN
+F 2 "" H 5450 5800 50  0001 C CNN
+F 3 "" H 5450 5800 50  0001 C CNN
+	1    5450 5800
+	1    0    0    -1
+$EndComp
+$Comp
+L +5V #PWR0218
+U 1 1 5AF07A8E
+P 5750 5800
+F 0 "#PWR0218" H 5750 5650 50  0001 C CNN
+F 1 "+5V" H 5750 5940 50  0000 C CNN
+F 2 "" H 5750 5800 50  0001 C CNN
+F 3 "" H 5750 5800 50  0001 C CNN
+	1    5750 5800
+	1    0    0    -1
+$EndComp
+$Comp
+L GND #PWR0219
+U 1 1 5AF07AC6
+P 5450 6650
+F 0 "#PWR0219" H 5450 6400 50  0001 C CNN
+F 1 "GND" H 5450 6500 50  0000 C CNN
+F 2 "" H 5450 6650 50  0001 C CNN
+F 3 "" H 5450 6650 50  0001 C CNN
+	1    5450 6650
+	1    0    0    -1
+$EndComp
+$Comp
+L R_Small R905
+U 1 1 5AF07B90
+P 5450 6450
+F 0 "R905" H 5480 6470 50  0000 L CNN
+F 1 "10k" H 5480 6410 50  0000 L CNN
+F 2 "Resistors_SMD:R_0402" H 5450 6450 50  0001 C CNN
+F 3 "" H 5450 6450 50  0001 C CNN
+	1    5450 6450
+	1    0    0    -1
+$EndComp
+Wire Wire Line
+	5450 5800 5450 6000
+Wire Wire Line
+	5450 6200 5450 6350
+Wire Wire Line
+	5450 6550 5450 6650
+$Comp
+L LED_Small D902
+U 1 1 5AF07E72
+P 5750 6100
+F 0 "D902" H 5700 6225 50  0000 L CNN
+F 1 "LED_Small" H 5575 6000 50  0000 L CNN
+F 2 "LEDs:LED_0603" V 5750 6100 50  0001 C CNN
+F 3 "" V 5750 6100 50  0001 C CNN
+	1    5750 6100
+	0    -1   -1   0
+$EndComp
+$Comp
+L GND #PWR0220
+U 1 1 5AF07E78
+P 5750 6650
+F 0 "#PWR0220" H 5750 6400 50  0001 C CNN
+F 1 "GND" H 5750 6500 50  0000 C CNN
+F 2 "" H 5750 6650 50  0001 C CNN
+F 3 "" H 5750 6650 50  0001 C CNN
+	1    5750 6650
+	1    0    0    -1
+$EndComp
+$Comp
+L R_Small R907
+U 1 1 5AF07E7E
+P 5750 6450
+F 0 "R907" H 5780 6470 50  0000 L CNN
+F 1 "10k" H 5780 6410 50  0000 L CNN
+F 2 "Resistors_SMD:R_0402" H 5750 6450 50  0001 C CNN
+F 3 "" H 5750 6450 50  0001 C CNN
+	1    5750 6450
+	1    0    0    -1
+$EndComp
+Wire Wire Line
+	5750 5800 5750 6000
+Wire Wire Line
+	5750 6200 5750 6350
+Wire Wire Line
+	5750 6550 5750 6650
 $EndSCHEMATC
