File: hardware/vna_r1_synth/vna_r1_synth.kicad_pcb (KiCad board)
At the start: 4 copper layers, 78 x 56 mm, 147 parts, among them J301 Conn_02x10_Odd_Even, U201 LMX2594, U301 CONN_SMA_2GND, U302 CONN_SMA_2GND, U303 LM27762, U304 74HC244, U305 74LVC1G32, U306 LD39100, U401 LTC2630-LZ8, U402 MAAM-011100, U403 ADRF5020, U404 LTC2054CS5, U501 CONN_SMA_2GND, U502 CONN_SMA_2GND, U503 CONN_SMA_2GND, U504 CONN_SMA_2GND, U505 CONN_SMA_2GND, U902 ADP7158

Commit message: finished vna r1 synth?
Parts:
- added G***: LOGO, vna_footprints:snail, B.Cu at (91.8, 129.2)
- added REF**: VIA_OSH4LAYER_MIN, vna_footprints:VIA_p35mm_p55mm, F.Cu at (111.0, 107.0)
- added REF**: VIA_OSH4LAYER_MIN, vna_footprints:VIA_OSH4LAYER_MIN, F.Cu at (103.4, 106.2)
- added REF**: VIA_OSH4LAYER_MIN, vna_footprints:VIA_p35mm_p55mm, F.Cu at (109.0, 145.0)
- added REF**: VIA_OSH4LAYER_MIN, vna_footprints:VIA_p35mm_p55mm, F.Cu at (107.0, 145.0)
- added REF**: VIA_OSH4LAYER_MIN, vna_footprints:VIA_p35mm_p55mm, F.Cu at (107.0, 149.0)
- added REF**: VIA_OSH4LAYER_MIN, vna_footprints:VIA_p35mm_p55mm, F.Cu at (105.0, 149.0)
- added REF**: VIA_OSH4LAYER_MIN, vna_footprints:VIA_p35mm_p55mm, F.Cu at (105.0, 145.0)
- added REF**: VIA_OSH4LAYER_MIN, vna_footprints:VIA_p35mm_p55mm, F.Cu at (103.0, 145.0)
- added REF**: VIA_OSH4LAYER_MIN, vna_footprints:VIA_p35mm_p55mm, F.Cu at (103.0, 149.0)
- added REF**: VIA_OSH4LAYER_MIN, vna_footprints:VIA_p35mm_p55mm, F.Cu at (101.0, 149.0)
- added REF**: VIA_OSH4LAYER_MIN, vna_footprints:VIA_p35mm_p55mm, F.Cu at (101.0, 145.0)
- added REF**: VIA_OSH4LAYER_MIN, vna_footprints:VIA_p35mm_p55mm, F.Cu at (99.0, 145.0)
- added REF**: VIA_OSH4LAYER_MIN, vna_footprints:VIA_OSH4LAYER_MIN, F.Cu at (105.2, 104.4)
- added REF**: VIA_OSH4LAYER_MIN, vna_footprints:VIA_p35mm_p55mm, F.Cu at (99.0, 149.0)
- added REF**: VIA_OSH4LAYER_MIN, vna_footprints:VIA_p35mm_p55mm, F.Cu at (97.0, 149.0)
- added REF**: VIA_OSH4LAYER_MIN, vna_footprints:VIA_p35mm_p55mm, F.Cu at (97.0, 145.0)
- added REF**: VIA_OSH4LAYER_MIN, vna_footprints:VIA_p35mm_p55mm, F.Cu at (95.0, 145.0)
- added REF**: VIA_OSH4LAYER_MIN, vna_footprints:VIA_p35mm_p55mm, F.Cu at (95.0, 149.0)
- added REF**: VIA_OSH4LAYER_MIN, vna_footprints:VIA_p35mm_p55mm, F.Cu at (93.0, 149.0)
- added REF**: VIA_OSH4LAYER_MIN, vna_footprints:VIA_p35mm_p55mm, F.Cu at (93.0, 145.0)
- added REF**: VIA_OSH4LAYER_MIN, vna_footprints:VIA_p35mm_p55mm, F.Cu at (91.0, 145.0)
- added REF**: VIA_OSH4LAYER_MIN, vna_footprints:VIA_p35mm_p55mm, F.Cu at (91.0, 149.0)
- added REF**: VIA_OSH4LAYER_MIN, vna_footprints:VIA_p35mm_p55mm, F.Cu at (89.0, 149.0)
- added REF**: VIA_OSH4LAYER_MIN, vna_footprints:VIA_OSH4LAYER_MIN, F.Cu at (107.2, 104.6)
- added REF**: VIA_OSH4LAYER_MIN, vna_footprints:VIA_p35mm_p55mm, F.Cu at (89.0, 145.0)
- added REF**: VIA_OSH4LAYER_MIN, vna_footprints:VIA_p35mm_p55mm, F.Cu at (87.0, 145.0)
- added REF**: VIA_OSH4LAYER_MIN, vna_footprints:VIA_p35mm_p55mm, F.Cu at (87.0, 149.0)
- added REF**: VIA_OSH4LAYER_MIN, vna_footprints:VIA_p35mm_p55mm, F.Cu at (85.0, 149.0)
- added REF**: VIA_OSH4LAYER_MIN, vna_footprints:VIA_p35mm_p55mm, F.Cu at (85.0, 145.0)
- added REF**: VIA_OSH4LAYER_MIN, vna_footprints:VIA_p35mm_p55mm, F.Cu at (81.0, 145.0)
- added REF**: VIA_OSH4LAYER_MIN, vna_footprints:VIA_p35mm_p55mm, F.Cu at (82.0, 149.0)
- added REF**: VIA_OSH4LAYER_MIN, vna_footprints:VIA_p35mm_p55mm, F.Cu at (80.0, 149.0)
- added REF**: VIA_OSH4LAYER_MIN, vna_footprints:VIA_p35mm_p55mm, F.Cu at (80.0, 145.0)
- added REF**: VIA_OSH4LAYER_MIN, vna_footprints:VIA_p35mm_p55mm, F.Cu at (78.0, 145.0)
- added REF**: VIA_OSH4LAYER_MIN, vna_footprints:VIA_OSH4LAYER_MIN, F.Cu at (105.4, 106.4)
- added REF**: VIA_OSH4LAYER_MIN, vna_footprints:VIA_p35mm_p55mm, F.Cu at (78.0, 149.0)
- added REF**: VIA_OSH4LAYER_MIN, vna_footprints:VIA_p35mm_p55mm, F.Cu at (76.0, 149.0)
- added REF**: VIA_OSH4LAYER_MIN, vna_footprints:VIA_p35mm_p55mm, F.Cu at (76.0, 145.0)
- added REF**: VIA_OSH4LAYER_MIN, vna_footprints:VIA_p35mm_p55mm, F.Cu at (74.0, 145.0)
- added REF**: VIA_OSH4LAYER_MIN, vna_footprints:VIA_p35mm_p55mm, F.Cu at (74.0, 149.0)
- added REF**: VIA_OSH4LAYER_MIN, vna_footprints:VIA_p35mm_p55mm, F.Cu at (72.0, 149.0)
- added REF**: VIA_OSH4LAYER_MIN, vna_footprints:VIA_p35mm_p55mm, F.Cu at (72.0, 145.0)
- added REF**: VIA_OSH4LAYER_MIN, vna_footprints:VIA_p35mm_p55mm, F.Cu at (69.0, 145.0)
- added REF**: VIA_OSH4LAYER_MIN, vna_footprints:VIA_p35mm_p55mm, F.Cu at (69.0, 149.0)
- added REF**: VIA_OSH4LAYER_MIN, vna_footprints:VIA_p35mm_p55mm, F.Cu at (66.0, 149.0)
- added REF**: VIA_OSH4LAYER_MIN, vna_footprints:VIA_OSH4LAYER_MIN, F.Cu at (106.0, 106.4)
- added REF**: VIA_OSH4LAYER_MIN, vna_footprints:VIA_p35mm_p55mm, F.Cu at (66.0, 145.0)
- added REF**: VIA_OSH4LAYER_MIN, vna_footprints:VIA_p35mm_p55mm, F.Cu at (63.0, 145.0)
- added REF**: VIA_OSH4LAYER_MIN, vna_footprints:VIA_p35mm_p55mm, F.Cu at (63.0, 149.0)
- added REF**: VIA_OSH4LAYER_MIN, vna_footprints:VIA_p35mm_p55mm, F.Cu at (60.0, 149.0)
- added REF**: VIA_OSH4LAYER_MIN, vna_footprints:VIA_p35mm_p55mm, F.Cu at (60.0, 145.0)
- added REF**: VIA_OSH4LAYER_MIN, vna_footprints:VIA_p35mm_p55mm, F.Cu at (57.0, 145.0)
- added REF**: VIA_OSH4LAYER_MIN, vna_footprints:VIA_p35mm_p55mm, F.Cu at (57.0, 149.0)
- added REF**: VIA_OSH4LAYER_MIN, vna_footprints:VIA_p35mm_p55mm, F.Cu at (54.0, 149.0)
- added REF**: VIA_OSH4LAYER_MIN, vna_footprints:VIA_p35mm_p55mm, F.Cu at (54.0, 145.0)
- added REF**: VIA_OSH4LAYER_MIN, vna_footprints:VIA_p35mm_p55mm, F.Cu at (50.0, 148.0)
- added REF**: VIA_OSH4LAYER_MIN, vna_footprints:VIA_OSH4LAYER_MIN, F.Cu at (106.6, 106.4)
- added REF**: VIA_OSH4LAYER_MIN, vna_footprints:VIA_p35mm_p55mm, F.Cu at (51.0, 145.0)
- added REF**: VIA_OSH4LAYER_MIN, vna_footprints:VIA_p35mm_p55mm, F.Cu at (50.0, 141.5)
- added REF**: VIA_OSH4LAYER_MIN, vna_footprints:VIA_p35mm_p55mm, F.Cu at (50.0, 139.0)
- added REF**: VIA_OSH4LAYER_MIN, vna_footprints:VIA_p35mm_p55mm, F.Cu at (50.0, 135.2)
- added REF**: VIA_OSH4LAYER_MIN, vna_footprints:VIA_p35mm_p55mm, F.Cu at (50.0, 131.0)
- added REF**: VIA_OSH4LAYER_MIN, vna_footprints:VIA_p35mm_p55mm, F.Cu at (50.0, 128.0)
- added REF**: VIA_OSH4LAYER_MIN, vna_footprints:VIA_p35mm_p55mm, F.Cu at (50.0, 124.5)
- added REF**: VIA_OSH4LAYER_MIN, vna_footprints:VIA_p35mm_p55mm, F.Cu at (50.0, 123.0)
- added REF**: VIA_OSH4LAYER_MIN, vna_footprints:VIA_p35mm_p55mm, F.Cu at (50.0, 121.0)
- added REF**: VIA_OSH4LAYER_MIN, vna_footprints:VIA_p35mm_p55mm, F.Cu at (50.0, 119.0)
- added REF**: VIA_OSH4LAYER_MIN, vna_footprints:VIA_OSH4LAYER_MIN, F.Cu at (106.6, 107.0)
- added REF**: VIA_OSH4LAYER_MIN, vna_footprints:VIA_p35mm_p55mm, F.Cu at (50.0, 117.0)
- added REF**: VIA_OSH4LAYER_MIN, vna_footprints:VIA_p35mm_p55mm, F.Cu at (50.0, 113.8)
- added REF**: VIA_OSH4LAYER_MIN, vna_footprints:VIA_p35mm_p55mm, F.Cu at (50.0, 112.0)
- added REF**: VIA_OSH4LAYER_MIN, vna_footprints:VIA_p35mm_p55mm, F.Cu at (50.0, 110.0)
- added REF**: VIA_OSH4LAYER_MIN, vna_footprints:VIA_p35mm_p55mm, F.Cu at (50.0, 107.0)
- added REF**: VIA_OSH4LAYER_MIN, vna_footprints:VIA_p35mm_p55mm, F.Cu at (50.0, 105.0)
- added REF**: VIA_OSH4LAYER_MIN, vna_footprints:VIA_p35mm_p55mm, F.Cu at (50.0, 103.0)
- added REF**: VIA_OSH4LAYER_MIN, vna_footprints:VIA_p35mm_p55mm, F.Cu at (50.0, 98.0)
- added REF**: VIA_OSH4LAYER_MIN, vna_footprints:VIA_p35mm_p55mm, F.Cu at (50.0, 95.0)
- added REF**: VIA_OSH4LAYER_MIN, vna_footprints:VIA_p35mm_p55mm, F.Cu at (66.0, 95.0)
- added REF**: VIA_OSH4LAYER_MIN, vna_footprints:VIA_OSH4LAYER_MIN, F.Cu at (106.0, 107.0)
- added REF**: VIA_OSH4LAYER_MIN, vna_footprints:VIA_p35mm_p55mm, F.Cu at (63.0, 95.0)
- added REF**: VIA_OSH4LAYER_MIN, vna_footprints:VIA_p35mm_p55mm, F.Cu at (60.0, 95.0)
- added REF**: VIA_OSH4LAYER_MIN, vna_footprints:VIA_p35mm_p55mm, F.Cu at (57.0, 95.0)
- added REF**: VIA_OSH4LAYER_MIN, vna_footprints:VIA_p35mm_p55mm, F.Cu at (54.0, 95.0)
- added REF**: VIA_OSH4LAYER_MIN, vna_footprints:VIA_p35mm_p55mm, F.Cu at (54.0, 98.0)
- added REF**: VIA_OSH4LAYER_MIN, vna_footprints:VIA_p35mm_p55mm, F.Cu at (57.0, 98.0)
- added REF**: VIA_OSH4LAYER_MIN, vna_footprints:VIA_p35mm_p55mm, F.Cu at (60.0, 98.0)
- added REF**: VIA_OSH4LAYER_MIN, vna_footprints:VIA_p35mm_p55mm, F.Cu at (63.0, 98.0)
- added REF**: VIA_OSH4LAYER_MIN, vna_footprints:VIA_p35mm_p55mm, F.Cu at (66.0, 98.0)
- added REF**: VIA_OSH4LAYER_MIN, vna_footprints:VIA_p35mm_p55mm, F.Cu at (74.0, 98.0)
- added REF**: VIA_OSH4LAYER_MIN, vna_footprints:VIA_OSH4LAYER_MIN, F.Cu at (105.4, 107.0)
- added REF**: VIA_OSH4LAYER_MIN, vna_footprints:VIA_p35mm_p55mm, F.Cu at (74.0, 95.0)
- added REF**: VIA_OSH4LAYER_MIN, vna_footprints:VIA_p35mm_p55mm, F.Cu at (76.0, 95.0)
- added REF**: VIA_OSH4LAYER_MIN, vna_footprints:VIA_p35mm_p55mm, F.Cu at (76.0, 98.0)
- added REF**: VIA_OSH4LAYER_MIN, vna_footprints:VIA_p35mm_p55mm, F.Cu at (78.0, 95.0)
- added REF**: VIA_OSH4LAYER_MIN, vna_footprints:VIA_p35mm_p55mm, F.Cu at (78.0, 98.0)
- added REF**: VIA_OSH4LAYER_MIN, vna_footprints:VIA_p35mm_p55mm, F.Cu at (72.0, 95.0)
- added REF**: VIA_OSH4LAYER_MIN, vna_footprints:VIA_p35mm_p55mm, F.Cu at (69.0, 95.0)
- added REF**: VIA_OSH4LAYER_MIN, vna_footprints:VIA_p35mm_p55mm, F.Cu at (72.0, 97.0)
- added REF**: VIA_OSH4LAYER_MIN, vna_footprints:VIA_p35mm_p55mm, F.Cu at (72.0, 99.0)
- added REF**: VIA_OSH4LAYER_MIN, vna_footprints:VIA_p35mm_p55mm, F.Cu at (69.0, 99.0)
- added REF**: VIA_OSH4LAYER_MIN, vna_footprints:VIA_OSH4LAYER_MIN, F.Cu at (105.4, 107.6)
- added REF**: VIA_OSH4LAYER_MIN, vna_footprints:VIA_p35mm_p55mm, F.Cu at (69.0, 100.8)
- added REF**: VIA_OSH4LAYER_MIN, vna_footprints:VIA_p35mm_p55mm, F.Cu at (72.6, 102.9)
- added REF**: VIA_OSH4LAYER_MIN, vna_footprints:VIA_p35mm_p55mm, F.Cu at (72.4, 105.0)
- added REF**: VIA_OSH4LAYER_MIN, vna_footprints:VIA_p35mm_p55mm, F.Cu at (69.0, 105.0)
- added REF**: VIA_OSH4LAYER_MIN, vna_footprints:VIA_p35mm_p55mm, F.Cu at (69.0, 107.0)
- added REF**: VIA_OSH4LAYER_MIN, vna_footprints:VIA_p35mm_p55mm, F.Cu at (72.4, 107.0)
- added REF**: VIA_OSH4LAYER_MIN, vna_footprints:VIA_p35mm_p55mm, F.Cu at (72.4, 109.0)
- added REF**: VIA_OSH4LAYER_MIN, vna_footprints:VIA_p35mm_p55mm, F.Cu at (69.0, 109.0)
- added REF**: VIA_OSH4LAYER_MIN, vna_footprints:VIA_p35mm_p55mm, F.Cu at (69.0, 111.0)
- added REF**: VIA_OSH4LAYER_MIN, vna_footprints:VIA_p35mm_p55mm, F.Cu at (72.4, 111.0)
- added REF**: VIA_OSH4LAYER_MIN, vna_footprints:VIA_p35mm_p55mm, F.Cu at (111.5, 109.0)
- added REF**: VIA_OSH4LAYER_MIN, vna_footprints:VIA_OSH4LAYER_MIN, F.Cu at (106.0, 107.6)
- added REF**: VIA_OSH4LAYER_MIN, vna_footprints:VIA_p35mm_p55mm, F.Cu at (72.4, 113.0)
- added REF**: VIA_OSH4LAYER_MIN, vna_footprints:VIA_p35mm_p55mm, F.Cu at (69.0, 113.0)
- added REF**: VIA_OSH4LAYER_MIN, vna_footprints:VIA_p35mm_p55mm, F.Cu at (69.0, 115.0)
- added REF**: VIA_OSH4LAYER_MIN, vna_footprints:VIA_p35mm_p55mm, F.Cu at (72.4, 115.0)
- added REF**: VIA_OSH4LAYER_MIN, vna_footprints:VIA_p35mm_p55mm, F.Cu at (72.4, 117.0)
- added REF**: VIA_OSH4LAYER_MIN, vna_footprints:VIA_p35mm_p55mm, F.Cu at (69.0, 117.0)
- added REF**: VIA_OSH4LAYER_MIN, vna_footprints:VIA_p35mm_p55mm, F.Cu at (69.0, 119.0)
- added REF**: VIA_OSH4LAYER_MIN, vna_footprints:VIA_p35mm_p55mm, F.Cu at (72.4, 119.0)
- added REF**: VIA_OSH4LAYER_MIN, vna_footprints:VIA_p35mm_p55mm, F.Cu at (69.0, 121.0)
- added REF**: VIA_OSH4LAYER_MIN, vna_footprints:VIA_p35mm_p55mm, F.Cu at (69.0, 123.0)
- added REF**: VIA_OSH4LAYER_MIN, vna_footprints:VIA_OSH4LAYER_MIN, F.Cu at (106.6, 107.6)
- added REF**: VIA_OSH4LAYER_MIN, vna_footprints:VIA_p35mm_p55mm, F.Cu at (69.0, 126.0)
- added REF**: VIA_OSH4LAYER_MIN, vna_footprints:VIA_p35mm_p55mm, F.Cu at (72.4, 126.0)
- added REF**: VIA_OSH4LAYER_MIN, vna_footprints:VIA_p35mm_p55mm, F.Cu at (72.0, 130.0)
- added REF**: VIA_OSH4LAYER_MIN, vna_footprints:VIA_p35mm_p55mm, F.Cu at (69.0, 130.0)
- added REF**: VIA_OSH4LAYER_MIN, vna_footprints:VIA_p35mm_p55mm, F.Cu at (69.0, 132.0)
- added REF**: VIA_OSH4LAYER_MIN, vna_footprints:VIA_p35mm_p55mm, F.Cu at (72.0, 132.0)
- added REF**: VIA_OSH4LAYER_MIN, vna_footprints:VIA_p35mm_p55mm, F.Cu at (72.0, 134.0)
- added REF**: VIA_OSH4LAYER_MIN, vna_footprints:VIA_p35mm_p55mm, F.Cu at (69.0, 134.0)
- added REF**: VIA_OSH4LAYER_MIN, vna_footprints:VIA_p35mm_p55mm, F.Cu at (69.0, 142.4)
- added REF**: VIA_OSH4LAYER_MIN, vna_footprints:VIA_p35mm_p55mm, F.Cu at (72.0, 142.4)
- added REF**: VIA_OSH4LAYER_MIN, vna_footprints:VIA_OSH4LAYER_MIN, F.Cu at (106.8, 108.8)
- added REF**: VIA_OSH4LAYER_MIN, vna_footprints:VIA_p35mm_p55mm, F.Cu at (72.0, 144.0)
- added REF**: VIA_OSH4LAYER_MIN, vna_footprints:VIA_p35mm_p55mm, F.Cu at (69.0, 144.0)
- added REF**: VIA_OSH4LAYER_MIN, vna_footprints:VIA_p35mm_p55mm, F.Cu at (94.0, 105.0)
- added REF**: VIA_OSH4LAYER_MIN, vna_footprints:VIA_p35mm_p55mm, F.Cu at (91.0, 107.0)
- added REF**: VIA_OSH4LAYER_MIN, vna_footprints:VIA_p35mm_p55mm, F.Cu at (89.0, 107.0)
- added REF**: VIA_OSH4LAYER_MIN, vna_footprints:VIA_p35mm_p55mm, F.Cu at (87.0, 107.0)
- added REF**: VIA_OSH4LAYER_MIN, vna_footprints:VIA_p35mm_p55mm, F.Cu at (85.0, 107.0)
- added REF**: VIA_OSH4LAYER_MIN, vna_footprints:VIA_p35mm_p55mm, F.Cu at (81.0, 107.0)
- added REF**: VIA_OSH4LAYER_MIN, vna_footprints:VIA_p35mm_p55mm, F.Cu at (77.0, 107.0)
- added REF**: VIA_OSH4LAYER_MIN, vna_footprints:VIA_p35mm_p55mm, F.Cu at (75.0, 107.0)
- added REF**: VIA_OSH4LAYER_MIN, vna_footprints:VIA_OSH4LAYER_MIN, F.Cu at (106.8, 105.2)
- added REF**: VIA_OSH4LAYER_MIN, vna_footprints:VIA_p35mm_p55mm, F.Cu at (75.0, 110.0)
- added REF**: VIA_OSH4LAYER_MIN, vna_footprints:VIA_p35mm_p55mm, F.Cu at (77.0, 110.0)
- added REF**: VIA_OSH4LAYER_MIN, vna_footprints:VIA_p35mm_p55mm, F.Cu at (78.0, 110.0)
- added REF**: VIA_OSH4LAYER_MIN, vna_footprints:VIA_p35mm_p55mm, F.Cu at (81.0, 110.0)
- added REF**: VIA_OSH4LAYER_MIN, vna_footprints:VIA_p35mm_p55mm, F.Cu at (85.0, 110.0)
- added REF**: VIA_OSH4LAYER_MIN, vna_footprints:VIA_p35mm_p55mm, F.Cu at (87.0, 110.0)
- added REF**: VIA_OSH4LAYER_MIN, vna_footprints:VIA_p35mm_p55mm, F.Cu at (89.0, 110.0)
- added REF**: VIA_OSH4LAYER_MIN, vna_footprints:VIA_p35mm_p55mm, F.Cu at (91.0, 110.0)
- added REF**: VIA_OSH4LAYER_MIN, vna_footprints:VIA_p35mm_p55mm, F.Cu at (93.0, 108.0)
- added REF**: VIA_OSH4LAYER_MIN, vna_footprints:VIA_p35mm_p55mm, F.Cu at (95.0, 106.0)
- added REF**: VIA_OSH4LAYER_MIN, vna_footprints:VIA_OSH4LAYER_MIN, F.Cu at (105.2, 105.2)
- added REF**: VIA_OSH4LAYER_MIN, vna_footprints:VIA_p35mm_p55mm, F.Cu at (97.0, 104.0)
- added REF**: VIA_OSH4LAYER_MIN, vna_footprints:VIA_p35mm_p55mm, F.Cu at (97.0, 102.0)
- added REF**: VIA_OSH4LAYER_MIN, vna_footprints:VIA_p35mm_p55mm, F.Cu at (96.0, 102.0)
- added REF**: VIA_OSH4LAYER_MIN, vna_footprints:VIA_p35mm_p55mm, F.Cu at (81.0, 98.0)
- added REF**: VIA_OSH4LAYER_MIN, vna_footprints:VIA_p35mm_p55mm, F.Cu at (84.0, 98.0)
- added REF**: VIA_OSH4LAYER_MIN, vna_footprints:VIA_p35mm_p55mm, F.Cu at (86.0, 98.0)
- added REF**: VIA_OSH4LAYER_MIN, vna_footprints:VIA_p35mm_p55mm, F.Cu at (89.0, 98.0)
- added REF**: VIA_OSH4LAYER_MIN, vna_footprints:VIA_p35mm_p55mm, F.Cu at (92.0, 98.0)
- added REF**: VIA_OSH4LAYER_MIN, vna_footprints:VIA_p35mm_p55mm, F.Cu at (95.0, 98.0)
- added REF**: VIA_OSH4LAYER_MIN, vna_footprints:VIA_p35mm_p55mm, F.Cu at (98.0, 98.0)
- added REF**: VIA_OSH4LAYER_MIN, vna_footprints:VIA_OSH4LAYER_MIN, F.Cu at (104.2, 106.2)
- added REF**: VIA_OSH4LAYER_MIN, vna_footprints:VIA_p35mm_p55mm, F.Cu at (101.0, 98.0)
- added REF**: VIA_OSH4LAYER_MIN, vna_footprints:VIA_p35mm_p55mm, F.Cu at (81.0, 95.0)
- added REF**: VIA_OSH4LAYER_MIN, vna_footprints:VIA_p35mm_p55mm, F.Cu at (84.0, 95.0)
- added REF**: VIA_OSH4LAYER_MIN, vna_footprints:VIA_p35mm_p55mm, F.Cu at (86.0, 95.0)
- added REF**: VIA_OSH4LAYER_MIN, vna_footprints:VIA_p35mm_p55mm, F.Cu at (89.0, 95.0)
- added REF**: VIA_OSH4LAYER_MIN, vna_footprints:VIA_p35mm_p55mm, F.Cu at (92.0, 95.0)
- added REF**: VIA_OSH4LAYER_MIN, vna_footprints:VIA_p35mm_p55mm, F.Cu at (95.0, 95.0)
- added REF**: VIA_OSH4LAYER_MIN, vna_footprints:VIA_p35mm_p55mm, F.Cu at (98.0, 95.0)
- added REF**: VIA_OSH4LAYER_MIN, vna_footprints:VIA_p35mm_p55mm, F.Cu at (101.0, 95.0)
- added REF**: VIA_OSH4LAYER_MIN, vna_footprints:VIA_p35mm_p55mm, F.Cu at (104.0, 95.0)
- added REF**: VIA_OSH4LAYER_MIN, vna_footprints:VIA_OSH4LAYER_MIN, F.Cu at (105.2, 108.8)
- added REF**: VIA_OSH4LAYER_MIN, vna_footprints:VIA_p35mm_p55mm, F.Cu at (107.0, 95.0)
- added REF**: VIA_OSH4LAYER_MIN, vna_footprints:VIA_p35mm_p55mm, F.Cu at (110.0, 95.0)
- added REF**: VIA_OSH4LAYER_MIN, vna_footprints:VIA_p35mm_p55mm, F.Cu at (115.0, 96.0)
- added REF**: VIA_OSH4LAYER_MIN, vna_footprints:VIA_p35mm_p55mm, F.Cu at (115.0, 98.0)
- added REF**: VIA_OSH4LAYER_MIN, vna_footprints:VIA_p35mm_p55mm, F.Cu at (110.0, 98.0)
- added REF**: VIA_OSH4LAYER_MIN, vna_footprints:VIA_p35mm_p55mm, F.Cu at (103.0, 99.0)
- added REF**: VIA_OSH4LAYER_MIN, vna_footprints:VIA_p35mm_p55mm, F.Cu at (107.0, 100.0)
- added REF**: VIA_OSH4LAYER_MIN, vna_footprints:VIA_p35mm_p55mm, F.Cu at (103.0, 102.0)
- added REF**: VIA_OSH4LAYER_MIN, vna_footprints:VIA_p35mm_p55mm, F.Cu at (105.0, 102.0)
- added REF**: VIA_OSH4LAYER_MIN, vna_footprints:VIA_p35mm_p55mm, F.Cu at (103.0, 104.0)
- added REF**: VIA_OSH4LAYER_MIN, vna_footprints:VIA_OSH4LAYER_MIN, F.Cu at (104.2, 107.8)
- added REF**: VIA_OSH4LAYER_MIN, vna_footprints:VIA_p35mm_p55mm, F.Cu at (104.0, 116.0)
- added REF**: VIA_OSH4LAYER_MIN, vna_footprints:VIA_p35mm_p55mm, F.Cu at (100.0, 116.0)
- added REF**: VIA_OSH4LAYER_MIN, vna_footprints:VIA_p35mm_p55mm, F.Cu at (100.0, 114.0)
- added REF**: VIA_OSH4LAYER_MIN, vna_footprints:VIA_p35mm_p55mm, F.Cu at (104.0, 114.0)
- added REF**: VIA_OSH4LAYER_MIN, vna_footprints:VIA_p35mm_p55mm, F.Cu at (115.0, 115.0)
- added REF**: VIA_OSH4LAYER_MIN, vna_footprints:VIA_p35mm_p55mm, F.Cu at (113.0, 115.0)
- added REF**: VIA_OSH4LAYER_MIN, vna_footprints:VIA_p35mm_p55mm, F.Cu at (111.0, 115.0)
- added REF**: VIA_OSH4LAYER_MIN, vna_footprints:VIA_p35mm_p55mm, F.Cu at (109.0, 115.0)
- added REF**: VIA_OSH4LAYER_MIN, vna_footprints:VIA_p35mm_p55mm, F.Cu at (106.0, 114.0)
- added REF**: VIA_OSH4LAYER_MIN, vna_footprints:VIA_p35mm_p55mm, F.Cu at (105.0, 112.0)
- added REF**: VIA_OSH4LAYER_MIN, vna_footprints:VIA_OSH4LAYER_MIN, F.Cu at (98.8, 107.8)
- added REF**: VIA_OSH4LAYER_MIN, vna_footprints:VIA_p35mm_p55mm, F.Cu at (103.0, 111.0)
- added REF**: VIA_OSH4LAYER_MIN, vna_footprints:VIA_p35mm_p55mm, F.Cu at (101.0, 111.0)
- added REF**: VIA_OSH4LAYER_MIN, vna_footprints:VIA_p35mm_p55mm, F.Cu at (99.0, 112.0)
- added REF**: VIA_OSH4LAYER_MIN, vna_footprints:VIA_p35mm_p55mm, F.Cu at (97.0, 114.0)
- added REF**: VIA_OSH4LAYER_MIN, vna_footprints:VIA_p35mm_p55mm, F.Cu at (97.0, 116.0)
- added REF**: VIA_OSH4LAYER_MIN, vna_footprints:VIA_p35mm_p55mm, F.Cu at (98.0, 118.0)
- added REF**: VIA_OSH4LAYER_MIN, vna_footprints:VIA_p35mm_p55mm, F.Cu at (100.0, 118.0)
- added REF**: VIA_OSH4LAYER_MIN, vna_footprints:VIA_p35mm_p55mm, F.Cu at (102.0, 118.0)
- added REF**: VIA_OSH4LAYER_MIN, vna_footprints:VIA_p35mm_p55mm, F.Cu at (104.0, 118.0)
- added REF**: VIA_OSH4LAYER_MIN, vna_footprints:VIA_p35mm_p55mm, F.Cu at (106.0, 118.0)
- added REF**: VIA_OSH4LAYER_MIN, vna_footprints:VIA_OSH4LAYER_MIN, F.Cu at (100.4, 107.8)
- added REF**: VIA_OSH4LAYER_MIN, vna_footprints:VIA_p35mm_p55mm, F.Cu at (109.0, 118.0)
- added REF**: VIA_OSH4LAYER_MIN, vna_footprints:VIA_p35mm_p55mm, F.Cu at (111.0, 118.0)
- added REF**: VIA_OSH4LAYER_MIN, vna_footprints:VIA_p35mm_p55mm, F.Cu at (115.0, 118.0)
- added REF**: VIA_OSH4LAYER_MIN, vna_footprints:VIA_p35mm_p55mm, F.Cu at (115.0, 125.0)
- added REF**: VIA_OSH4LAYER_MIN, vna_footprints:VIA_p35mm_p55mm, F.Cu at (112.0, 125.0)
- added REF**: VIA_OSH4LAYER_MIN, vna_footprints:VIA_p35mm_p55mm, F.Cu at (110.0, 125.0)
- added REF**: VIA_OSH4LAYER_MIN, vna_footprints:VIA_p35mm_p55mm, F.Cu at (108.0, 125.0)
- added REF**: VIA_OSH4LAYER_MIN, vna_footprints:VIA_p35mm_p55mm, F.Cu at (106.0, 125.0)
- added REF**: VIA_OSH4LAYER_MIN, vna_footprints:VIA_p35mm_p55mm, F.Cu at (104.0, 125.0)
- added REF**: VIA_OSH4LAYER_MIN, vna_footprints:VIA_p35mm_p55mm, F.Cu at (102.0, 125.0)
- added REF**: VIA_OSH4LAYER_MIN, vna_footprints:VIA_p35mm_p55mm, F.Cu at (72.0, 100.0)
- added REF**: VIA_OSH4LAYER_MIN, vna_footprints:VIA_OSH4LAYER_MIN, F.Cu at (99.2, 107.8)
- added REF**: VIA_OSH4LAYER_MIN, vna_footprints:VIA_p35mm_p55mm, F.Cu at (100.0, 125.0)
- added REF**: VIA_OSH4LAYER_MIN, vna_footprints:VIA_p35mm_p55mm, F.Cu at (97.0, 129.0)
- added REF**: VIA_OSH4LAYER_MIN, vna_footprints:VIA_p35mm_p55mm, F.Cu at (98.0, 125.0)
- added REF**: VIA_OSH4LAYER_MIN, vna_footprints:VIA_p35mm_p55mm, F.Cu at (97.0, 125.0)
- added REF**: VIA_OSH4LAYER_MIN, vna_footprints:VIA_p35mm_p55mm, F.Cu at (98.0, 129.0)
- added REF**: VIA_OSH4LAYER_MIN, vna_footprints:VIA_p35mm_p55mm, F.Cu at (100.0, 129.0)
- added REF**: VIA_OSH4LAYER_MIN, vna_footprints:VIA_p35mm_p55mm, F.Cu at (102.0, 129.0)
- added REF**: VIA_OSH4LAYER_MIN, vna_footprints:VIA_p35mm_p55mm, F.Cu at (104.0, 129.0)
- added REF**: VIA_OSH4LAYER_MIN, vna_footprints:VIA_p35mm_p55mm, F.Cu at (106.0, 129.0)
- added REF**: VIA_OSH4LAYER_MIN, vna_footprints:VIA_p35mm_p55mm, F.Cu at (108.0, 129.0)
- added REF**: VIA_OSH4LAYER_MIN, vna_footprints:VIA_OSH4LAYER_MIN, F.Cu at (99.6, 107.8)
- added REF**: VIA_OSH4LAYER_MIN, vna_footprints:VIA_p35mm_p55mm, F.Cu at (112.0, 129.0)
- added REF**: VIA_OSH4LAYER_MIN, vna_footprints:VIA_p35mm_p55mm, F.Cu at (115.0, 129.0)
- added REF**: VIA_OSH4LAYER_MIN, vna_footprints:VIA_p35mm_p55mm, F.Cu at (110.0, 129.0)
- added REF**: VIA_OSH4LAYER_MIN, vna_footprints:VIA_p35mm_p55mm, F.Cu at (110.0, 136.0)
- added REF**: VIA_OSH4LAYER_MIN, vna_footprints:VIA_p35mm_p55mm, F.Cu at (96.0, 136.0)
- added REF**: VIA_OSH4LAYER_MIN, vna_footprints:VIA_p35mm_p55mm, F.Cu at (98.0, 136.0)
- added REF**: VIA_OSH4LAYER_MIN, vna_footprints:VIA_p35mm_p55mm, F.Cu at (100.0, 136.0)
- added REF**: VIA_OSH4LAYER_MIN, vna_footprints:VIA_p35mm_p55mm, F.Cu at (102.0, 136.0)
- added REF**: VIA_OSH4LAYER_MIN, vna_footprints:VIA_p35mm_p55mm, F.Cu at (104.0, 136.0)
- added REF**: VIA_OSH4LAYER_MIN, vna_footprints:VIA_p35mm_p55mm, F.Cu at (106.0, 136.0)
- added REF**: VIA_OSH4LAYER_MIN, vna_footprints:VIA_p35mm_p55mm, F.Cu at (72.0, 139.6)
- added REF**: VIA_OSH4LAYER_MIN, vna_footprints:VIA_p35mm_p55mm, F.Cu at (108.0, 136.0)
- added REF**: VIA_OSH4LAYER_MIN, vna_footprints:VIA_p35mm_p55mm, F.Cu at (111.0, 136.0)
- added REF**: VIA_OSH4LAYER_MIN, vna_footprints:VIA_p35mm_p55mm, F.Cu at (115.0, 136.0)
- added REF**: VIA_OSH4LAYER_MIN, vna_footprints:VIA_p35mm_p55mm, F.Cu at (115.0, 138.0)
- added REF**: VIA_OSH4LAYER_MIN, vna_footprints:VIA_p35mm_p55mm, F.Cu at (111.0, 138.0)
- added REF**: VIA_OSH4LAYER_MIN, vna_footprints:VIA_p35mm_p55mm, F.Cu at (110.0, 138.0)
- added REF**: VIA_OSH4LAYER_MIN, vna_footprints:VIA_p35mm_p55mm, F.Cu at (108.0, 138.0)
- added REF**: VIA_OSH4LAYER_MIN, vna_footprints:VIA_p35mm_p55mm, F.Cu at (106.0, 138.0)
- added REF**: VIA_OSH4LAYER_MIN, vna_footprints:VIA_p35mm_p55mm, F.Cu at (104.0, 138.0)
- added REF**: VIA_OSH4LAYER_MIN, vna_footprints:VIA_p35mm_p55mm, F.Cu at (102.0, 138.0)
- added REF**: VIA_OSH4LAYER_MIN, vna_footprints:VIA_p35mm_p55mm, F.Cu at (69.0, 139.6)
- added REF**: VIA_OSH4LAYER_MIN, vna_footprints:VIA_p35mm_p55mm, F.Cu at (100.0, 138.0)
- added REF**: VIA_OSH4LAYER_MIN, vna_footprints:VIA_p35mm_p55mm, F.Cu at (98.0, 138.0)
- added REF**: VIA_OSH4LAYER_MIN, vna_footprints:VIA_p35mm_p55mm, F.Cu at (78.0, 107.0)
- added REF**: VIA_OSH4LAYER_MIN, vna_footprints:VIA_p35mm_p55mm, F.Cu at (97.0, 118.0)
- added REF**: VIA_OSH4LAYER_MIN, vna_footprints:VIA_p35mm_p55mm, F.Cu at (96.0, 138.0)
- added REF**: VIA_OSH4LAYER_MIN, vna_footprints:VIA_p35mm_p55mm, F.Cu at (76.0, 147.0)
- added REF**: VIA_OSH4LAYER_MIN, vna_footprints:VIA_p35mm_p55mm, F.Cu at (51.5, 101.8)
- added REF**: VIA_OSH4LAYER_MIN, vna_footprints:VIA_OSH4LAYER_MIN, F.Cu at (100.0, 107.8)
- added REF**: VIA_OSH4LAYER_MIN, vna_footprints:VIA_p35mm_p55mm, F.Cu at (75.0, 119.0)
- added REF**: VIA_OSH4LAYER_MIN, vna_footprints:VIA_p35mm_p55mm, F.Cu at (75.0, 121.0)
- added REF**: VIA_OSH4LAYER_MIN, vna_footprints:VIA_p35mm_p55mm, F.Cu at (75.0, 117.0)
- added REF**: VIA_OSH4LAYER_MIN, vna_footprints:VIA_p35mm_p55mm, F.Cu at (111.0, 106.0)
- added REF**: VIA_OSH4LAYER_MIN, vna_footprints:VIA_p35mm_p55mm, F.Cu at (115.0, 107.0)
- added REF**: VIA_OSH4LAYER_MIN, vna_footprints:VIA_p35mm_p55mm, F.Cu at (113.0, 105.0)
- added REF**: VIA_OSH4LAYER_MIN, vna_footprints:VIA_OSH4LAYER_MIN, F.Cu at (100.2, 109.0)
- added REF**: VIA_OSH4LAYER_MIN, vna_footprints:VIA_p35mm_p55mm, F.Cu at (113.0, 109.0)
- added REF**: VIA_OSH4LAYER_MIN, vna_footprints:VIA_p35mm_p55mm, F.Cu at (111.0, 105.0)
- added REF**: VIA_OSH4LAYER_MIN, vna_footprints:VIA_p35mm_p55mm, F.Cu at (114.8, 105.0)
- added REF**: VIA_OSH4LAYER_MIN, vna_footprints:VIA_p35mm_p55mm, F.Cu at (114.8, 109.0)
- added REF**: VIA_OSH4LAYER_MIN, vna_footprints:VIA_p35mm_p55mm, F.Cu at (108.0, 126.8)
- added REF**: VIA_OSH4LAYER_MIN, vna_footprints:VIA_p35mm_p55mm, F.Cu at (104.0, 126.8)
- added REF**: VIA_OSH4LAYER_MIN, vna_footprints:VIA_p35mm_p55mm, F.Cu at (100.0, 126.8)
- added REF**: VIA_OSH4LAYER_MIN, vna_footprints:VIA_p35mm_p55mm, F.Cu at (97.0, 126.8)
- added REF**: VIA_OSH4LAYER_MIN, vna_footprints:VIA_p35mm_p55mm, F.Cu at (60.2, 116.0)
- added REF**: VIA_OSH4LAYER_MIN, vna_footprints:VIA_p35mm_p55mm, F.Cu at (56.8, 119.2)
- added REF**: VIA_OSH4LAYER_MIN, vna_footprints:VIA_OSH4LAYER_MIN, F.Cu at (99.8, 109.0)
- added REF**: VIA_OSH4LAYER_MIN, vna_footprints:VIA_p35mm_p55mm, F.Cu at (57.5, 120.0)
- added REF**: VIA_OSH4LAYER_MIN, vna_footprints:VIA_p35mm_p55mm, F.Cu at (62.0, 116.0)
- added REF**: VIA_OSH4LAYER_MIN, vna_footprints:VIA_p35mm_p55mm, F.Cu at (58.8, 116.0)
- added REF**: VIA_OSH4LAYER_MIN, vna_footprints:VIA_p35mm_p55mm, F.Cu at (60.5, 120.0)
- added REF**: VIA_OSH4LAYER_MIN, vna_footprints:VIA_p35mm_p55mm, F.Cu at (57.2, 106.0)
- added REF**: VIA_OSH4LAYER_MIN, vna_footprints:VIA_p35mm_p55mm, F.Cu at (58.0, 107.8)
- added REF**: VIA_OSH4LAYER_MIN, vna_footprints:VIA_p35mm_p55mm, F.Cu at (61.5, 107.8)
- added REF**: VIA_OSH4LAYER_MIN, vna_footprints:VIA_p35mm_p55mm, F.Cu at (63.0, 107.5)
- added REF**: VIA_OSH4LAYER_MIN, vna_footprints:VIA_p35mm_p55mm, F.Cu at (65.0, 125.5)
- added REF**: VIA_OSH4LAYER_MIN, vna_footprints:VIA_p35mm_p55mm, F.Cu at (65.0, 124.0)
- added REF**: VIA_OSH4LAYER_MIN, vna_footprints:VIA_OSH4LAYER_MIN, F.Cu at (109.0, 108.0)
- added REF**: VIA_OSH4LAYER_MIN, vna_footprints:VIA_p35mm_p55mm, F.Cu at (63.5, 124.0)
- added REF**: VIA_OSH4LAYER_MIN, vna_footprints:VIA_p35mm_p55mm, F.Cu at (61.5, 124.0)
- added REF**: VIA_OSH4LAYER_MIN, vna_footprints:VIA_p35mm_p55mm, F.Cu at (60.5, 124.0)
- added REF**: VIA_OSH4LAYER_MIN, vna_footprints:VIA_p35mm_p55mm, F.Cu at (56.0, 124.0)
- added REF**: VIA_OSH4LAYER_MIN, vna_footprints:VIA_p35mm_p55mm, F.Cu at (57.5, 124.0)
- added REF**: VIA_OSH4LAYER_MIN, vna_footprints:VIA_p35mm_p55mm, F.Cu at (59.0, 124.0)
- added REF**: VIA_OSH4LAYER_MIN, vna_footprints:VIA_p35mm_p55mm, F.Cu at (59.0, 125.5)
- added REF**: VIA_OSH4LAYER_MIN, vna_footprints:VIA_p35mm_p55mm, F.Cu at (60.5, 130.0)
- added REF**: VIA_OSH4LAYER_MIN, vna_footprints:VIA_p35mm_p55mm, F.Cu at (62.0, 130.0)
- added REF**: VIA_OSH4LAYER_MIN, vna_footprints:VIA_p35mm_p55mm, F.Cu at (59.0, 130.0)
- added REF**: VIA_OSH4LAYER_MIN, vna_footprints:VIA_OSH4LAYER_MIN, F.Cu at (107.2, 109.6)
- added REF**: VIA_OSH4LAYER_MIN, vna_footprints:VIA_p35mm_p55mm, F.Cu at (65.0, 130.0)
- added REF**: VIA_OSH4LAYER_MIN, vna_footprints:VIA_p35mm_p55mm, F.Cu at (65.0, 131.5)
- added REF**: VIA_OSH4LAYER_MIN, vna_footprints:VIA_p35mm_p55mm, F.Cu at (63.5, 131.5)
- added REF**: VIA_OSH4LAYER_MIN, vna_footprints:VIA_p35mm_p55mm, F.Cu at (62.0, 131.5)
- added REF**: VIA_OSH4LAYER_MIN, vna_footprints:VIA_p35mm_p55mm, F.Cu at (60.5, 131.5)
- added REF**: VIA_OSH4LAYER_MIN, vna_footprints:VIA_p35mm_p55mm, F.Cu at (59.0, 131.5)
- added REF**: VIA_OSH4LAYER_MIN, vna_footprints:VIA_p35mm_p55mm, F.Cu at (57.5, 131.5)
- added REF**: VIA_OSH4LAYER_MIN, vna_footprints:VIA_p35mm_p55mm, F.Cu at (56.0, 131.5)
- added REF**: VIA_OSH4LAYER_MIN, vna_footprints:VIA_p35mm_p55mm, F.Cu at (56.0, 130.0)
- added REF**: VIA_OSH4LAYER_MIN, vna_footprints:VIA_p35mm_p55mm, F.Cu at (107.0, 98.0)
- added REF**: VIA_OSH4LAYER_MIN, vna_footprints:VIA_OSH4LAYER_MIN, F.Cu at (105.2, 109.8)
- added REF**: VIA_OSH4LAYER_MIN, vna_footprints:VIA_p35mm_p55mm, F.Cu at (104.0, 98.0)
- added REF**: VIA_OSH4LAYER_MIN, vna_footprints:VIA_p35mm_p55mm, F.Cu at (111.0, 147.0)
- added REF**: VIA_OSH4LAYER_MIN, vna_footprints:VIA_p35mm_p55mm, F.Cu at (107.0, 147.0)
- added REF**: VIA_OSH4LAYER_MIN, vna_footprints:VIA_p35mm_p55mm, F.Cu at (103.0, 147.0)
- added REF**: VIA_OSH4LAYER_MIN, vna_footprints:VIA_p35mm_p55mm, F.Cu at (99.0, 147.0)
- added REF**: VIA_OSH4LAYER_MIN, vna_footprints:VIA_p35mm_p55mm, F.Cu at (95.0, 147.0)
- added REF**: VIA_OSH4LAYER_MIN, vna_footprints:VIA_p35mm_p55mm, F.Cu at (91.0, 147.0)
- added REF**: VIA_OSH4LAYER_MIN, vna_footprints:VIA_p35mm_p55mm, F.Cu at (87.0, 147.0)
- added REF**: VIA_OSH4LAYER_MIN, vna_footprints:VIA_p35mm_p55mm, F.Cu at (80.0, 147.0)
- added REF**: VIA_OSH4LAYER_MIN, vna_footprints:VIA_p35mm_p55mm, F.Cu at (54.0, 147.0)
- added REF**: VIA_OSH4LAYER_MIN, vna_footprints:VIA_OSH4LAYER_MIN, F.Cu at (103.4, 107.8)
- added REF**: VIA_OSH4LAYER_MIN, vna_footprints:VIA_p35mm_p55mm, F.Cu at (60.0, 147.0)
- added REF**: VIA_OSH4LAYER_MIN, vna_footprints:VIA_p35mm_p55mm, F.Cu at (66.0, 147.0)
- added REF**: VIA_OSH4LAYER_MIN, vna_footprints:VIA_p35mm_p55mm, F.Cu at (72.0, 147.0)
- added REF**: VIA_OSH4LAYER_MIN, vna_footprints:VIA_p35mm_p55mm, F.Cu at (113.0, 145.0)
- added REF**: VIA_OSH4LAYER_MIN, vna_footprints:VIA_p35mm_p55mm, F.Cu at (113.0, 149.0)
- added REF**: VIA_OSH4LAYER_MIN, vna_footprints:VIA_p35mm_p55mm, F.Cu at (115.0, 149.0)
- added REF**: VIA_OSH4LAYER_MIN, vna_footprints:VIA_p35mm_p55mm, F.Cu at (115.0, 145.0)
- added REF**: VIA_OSH4LAYER_MIN, vna_footprints:VIA_p35mm_p55mm, F.Cu at (111.0, 145.0)
- added REF**: VIA_OSH4LAYER_MIN, vna_footprints:VIA_p35mm_p55mm, F.Cu at (111.0, 149.0)
- added REF**: VIA_OSH4LAYER_MIN, vna_footprints:VIA_p35mm_p55mm, F.Cu at (109.0, 149.0)
- moved C415 1.63 mm to (110.2, 109.2)
- moved C226 0.45 mm to (93.2, 121.2)
- moved L202 0.45 mm to (93.2, 122.2)
- moved L201 0.25 mm to (84.8, 129.9)
- moved C225 0.15 mm to (85.8, 130.0)
Routing:
- net GND: track 117.1 -> 128.9 mm, vias 100 -> 95
- net Net-(C225-Pad2): track 4.51 -> 8.39 mm
- net /conn_power/SYNTH_REF_N: track 59.4 -> 63.1 mm
- net /conn_power/SYNTH_REF_P: track 56.2 -> 59.0 mm
- net +3V3: track 163.9 -> 166.6 mm
- net /AMP_VD: track 56.9 -> 59.6 mm
- net Net-(C226-Pad2): track 6.02 -> 8.14 mm
- net +5V: track 32.8 -> 34.1 mm
- net -2V5: track 68.3 -> 67.6 mm
- net /PORT_SEL: track 74.2 -> 73.6 mm
Other:
- net class Default: clearance 0.1254 -> 0.135
- rule pad_to_mask_clearance: 0.05 -> 0.04
- rule trace_clearance: 0.1254 -> 0.135
- board text added: "1"
- board text added: "2"
- board text added: "AUX OUT"
- board text added: "LO 1"
- board text added: "LO 2"
- board text added: "REF P"
- board text added: "vna demod 2018.05"
