File: breakouts/maam_011109/maam_011109/maam_011109.kicad_pcb (KiCad board)
At the start: 2 copper layers, 16 parts, among them J101 Conn_Coaxial, J102 GND, J103 Vc, J104 Vdet, J105 Vd, J106 Conn_Coaxial, J107 GND, U101 MAAM-011109

Commit message: finished maam-011109 breakout layout
Parts:
- added G***: LOGO, vna_footprints:snail, B.Cu at (110.8, 79.6)
- moved J102 37.2 mm to (105.0, 77.5)
- moved J103 34.4 mm to (110.0, 77.5)
- moved J105 33.7 mm to (120.0, 77.5)
- moved J104 30.3 mm to (115.0, 77.5)
- moved J107 29.8 mm to (124.0, 77.5)
- moved C102 26.9 mm to (114.2, 82.0), turned to 180 degrees
- moved C104 24.2 mm to (117.4, 81.5)
- moved C103 24.0 mm to (117.4, 82.9)
- moved L101 22.9 mm to (114.7, 83.9), turned to 270 degrees
- moved TP101 18.1 mm to (113.9, 94.0)
- moved C101 0.42 mm to (111.7, 84.3)
Routing:
- net Net-(C102-Pad1): track 0.00 -> 11.4 mm
- net Net-(J104-Pad1): track 0.00 -> 11.1 mm
- net Net-(C101-Pad1): track 0.00 -> 9.46 mm
- net Net-(J101-Pad1): track 0.00 -> 6.44 mm
- net Net-(J106-Pad1): track 0.00 -> 6.38 mm
- net GND: track 0.00 -> 5.91 mm, vias 0 -> 47
- net Net-(TP103-Pad1): track 0.00 -> 4.46 mm
- net Net-(TP102-Pad1): track 0.00 -> 4.46 mm
- net Net-(L101-Pad2): track 0.00 -> 1.47 mm
- added copper zone on B.Cu, net GND
- added copper zone on In1.Cu, net GND
Other:
- board outline added: 23.1 x 19.7 mm
- copper layers 2 -> 4
- net class Default: trace_width 0.25 -> 0.41
- net class RF added: clearance 0.2, trace_width 0.41, via_dia 0.8, via_drill 0.4
- rule via_min_drill: 0.3 -> 0.254
- board text added: "0V"
- board text added: "MAAM-011109"
- board text added: "Vc"
- board text added: "Vd"
- board text added: "Vt"
