File: breakouts/pe42543_breakout/pe42543_breakout.kicad_pcb (KiCad board)
At the start: 4 copper layers, 25.1 x 34 mm, 28 parts, among them J101 Conn_Coaxial, J102 Vdd, J103 Vss, J104 V2, J105 V1, J106 Conn_Coaxial, J107 Conn_Coaxial, J108 Conn_Coaxial, J109 Conn_Coaxial, J110 GND, J111 GND, U101 PE42543

Commit message: update pe42543 paste mask
Other:
- rule solder_mask_min_width: 0.135 -> 0.1
