File: hardware/vna_mm_ref/vna_mm_ref.kicad_pcb (KiCad board)
At the start: 4 copper layers, 115.5 x 66 mm, 229 parts, among them J201 Conn_Coaxial, J202 Conn_Coaxial, J401 Conn_Coaxial, J402 Conn_Coaxial, J501 Conn_02x10_Odd_Even, J502 Conn_01x07, K401 1-1462051-1, Q501 FDS6890A, SW501 SW_DIP_x02, SW502 SW_DIP_x02, U201 LTC6957xDD-3, U301 HMC1031, U401 DOCAT050F-010.0M, U402 74AHC1G04, U403 DRV8837C, U404 LTC6957xDD-3, U501 LTC4365DDB, U502 ADP7156, U503 ADP7156, U504 74AHC244, U505 LMT84DCK, X301 ABLNO-V-100.000MHZ

Commit message: cleanup and update vna mm synth schematic for modern kicad libraries
Other:
- board text removed: "JLCJLCJLCJLC"
Changed lines of the file:
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@@
   (general
     (thickness 1.6)
-    (drawings 27)
+    (drawings 30)
     (tracks 1561)
     (zones 0)
@@
   (layers
     (0 F.Cu signal)
-    (1 In1.Cu signal)
-    (2 In2.Cu signal)
-    (31 B.Cu signal)
+    (1 In1.Cu signal hide)
+    (2 In2.Cu signal hide)
+    (31 B.Cu signal hide)
     (32 B.Adhes user)
-    (33 F.Adhes user)
+    (33 F.Adhes user hide)
     (34 B.Paste user)
     (35 F.Paste user)
@@
     (38 B.Mask user)
     (39 F.Mask user)
-    (40 Dwgs.User user)
+    (40 Dwgs.User user hide)
     (41 Cmts.User user hide)
     (42 Eco1.User user)
@@
     (visible_elements FFFDFF7F)
     (pcbplotparams
-      (layerselection 0x010f8_ffffffff)
+      (layerselection 0x00000_7ffffff9)
       (usegerberextensions true)
       (usegerberattributes false)
@@
       (padsonsilk false)
       (subtractmaskfromsilk false)
-      (outputformat 1)
+      (outputformat 5)
       (mirror false)
       (drillshape 0)
       (scaleselection 1)
-      (outputdirectory "gerbs/"))
+      (outputdirectory "mech/"))
   )
   (net 0 "")
@@
     )
   )
-  (gr_text JLCJLCJLCJLC (at 150.5 72.75) (layer F.SilkS)
-    (effects (font (size 0.8 0.8) (thickness 0.15)))
-  )
+  (gr_poly (pts (xy 254 64.5) (xy 254 69.5) (xy 144 69.5) (xy 144 87.75) (xy 138.5 87.75) (xy 138.5 64.5)) (layer Dwgs.User) (width 0.1))
+  (gr_poly (pts (xy 254 87.25) (xy 241.75 87.25) (xy 241.75 81.5) (xy 254 81.5)) (layer Dwgs.User) (width 0.1))
+  (gr_poly (pts (xy 193 94.25) (xy 193 105) (xy 254 105) (xy 254 99) (xy 235 99) (xy 235 94.25)) (layer Dwgs.User) (width 0.1))
+  (gr_poly (pts (xy 175.5 86.75) (xy 175.5 99.25) (xy 138.5 99.25) (xy 138.5 105) (xy 181 105) (xy 181 86.75)) (layer Dwgs.User) (width 0.1))
   (gr_line (start 138.5 104.25) (end 138.5 39.75) (layer Edge.Cuts) (width 0.05))
   (gr_line (start 253.25 105) (end 139.25 105) (layer Edge.Cuts) (width 0.05))
