File: hardware/vna_mm_synth/bandselect_att.sch (KiCad schematic (older format))
At the start: 20 parts

Commit message: added power supply sequencing
Parts:
- gave numbers to parts that had none: 20

Commit message: changed synth midband filter bank to admv8416, added rf test points
Parts:
- removed FL902, FL903: low_pass_filter, symbol synth_lib:low_pass_filter
- removed FL904, FL905: band_pass_filter, symbol synth_lib:band_pass_filter
- added C? (x2): 100 nF, Capacitors_SMD:C_0402, symbol device:C_Small
- added C? (x2): 100 pF, Capacitors_SMD:C_0402, symbol device:C_Small
- added J? (x2): Conn_Coaxial, symbol Connector:Conn_Coaxial
- added L? (x2): L_Small, symbol Device:L_Small
- added U?: ADMV8416, Housings_DFN_QFN:QFN-40-1EP_6x6mm_Pitch0.5mm, symbol vna_mm:ADMV8416
Connections:
- net MID2 is gone; now on net MID: U901.2 (RF2)
- net X2_FEED is gone; now on net X2_FEED_RFOUT: U901.17 (RF3)
- net GND: now also C?.2, C?.2, C?.2, C?.2, J?.2 (Ext), J?.2 (Ext), U?.1 (NC), U?.10 (NC), U?.12 (GND), U?.14 (NC), U?.16 (GND), U?.17 (NC), U?.18 (GND), U?.2 (NC), U?.20 (NC), U?.21 (NC), U?.22 (NC), U?.23 (NC), U?.24 (NC), U?.25 (GND), U?.27 (GND), U?.28 (NC), U?.29 (NC), U?.3 (NC), U?.30 (NC), U?.31 (NC), U?.32 (NC), U?.33 (NC), U?.34 (NC), U?.35 (NC), U?.36 (NC), U?.37 (NC), U?.38 (NC), U?.39 (NC), U?.4 (GND), U?.40 (NC), U?.41 (GND), U?.6 (GND), U?.7 (NC), U?.8 (NC), U?.9 (NC)
- net SW_MID_RFIN: now also U?.5 (RFIN); no longer U901.12 (RFC)
- net MID1: no longer names the net of U901.22 (RF1)
- net MID1_FILT renamed MID
- net MID2_FILT renamed BYPASS
- net MID3: no longer names the net of U901.7 (RF4)
- net MID3: now also J?.1 (In)
- net MID3_FILT: no longer names the net of U902.7 (RF4)
- net MID3_FILT: now also J?.1 (In)
- new net: U901.12 (RFC), U?.26 (RFOUT)
- new net: C?.1, C?.1, L?.2, U?.11 (VEE)
- new net: C?.1, C?.1, L?.2, U?.13 (VDD)
- new net +5VP: L?.1
- new net -5V: L?.1
- new net FILT_VCTL: U?.15 (VCTL)
- new net FILT_VTUNE: U?.19 (VTUNE)
- no-connect marks 0 -> 1
Other:
- note removed: "BPF, 15-18 GHz"
- note removed: "BPF, 9-14.5 GHz"
- note removed: "LPF, 11-15 GHz"
- note removed: "LPF, 7.5-11 GHz"
- moved on the sheet: C901, C902, C903, C904, C905, C906, C907, FL901, FL906, L901, L902, R901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

Commit message: added trl cal and set of breakout boards
Parts:
- L901, L902: renamed from L?; value L_Small -> BLM15GG471; footprint (none) -> Resistors_SMD:R_0402
- L903: renamed from L901; value L_Small -> BLM15GG471; footprint (none) -> Resistors_SMD:R_0402
- L904: renamed from L902; value L_Small -> BLM15GG471; footprint (none) -> Resistors_SMD:R_0402
- gave numbers to parts that had none: 7
- renumbered C901 to C905, C902 to C906, C903 to C907, C904 to C908, C905 to C909, C906 to C910, C907 to C911, FL906 to FL902, U901 to U902, U902 to U903, U903 to U904

Commit message: fixed mirrored 3.3V regulator on sequencer board, created and assigned footprints for synth
Parts:
- added R903, R904: TBD, Resistors_SMD:R_0402, symbol device:R_Small
- FL901: footprint (none) -> vna_footprints:stepped_lpf_8ghz_fr408
- FL902: footprint (none) -> vna_footprints:stepped_lpf_20ghz_fr408
- U902, U903: footprint (none) -> vna_mm:RFSW__PE42543A-X
Connections:
- net FILT_VCTL: now also R903.2; no longer U901.15 (VCTL)
- net GND: now also R904.2
- new net: R903.1, R904.1, U901.15 (VCTL)
Other:
- note added: "SEQUENCE:\n1 - VDD/VEE\n2 - VCTL\n3 - VTUNE"
- moved on the sheet: FL901
Changed lines of the file:
@@
 Text HLabel 17800 9200 3    60   Input ~ 0
 SW_HIGH_RFIN
-Text HLabel 2700 2950 0    60   Input ~ 0
+Text HLabel 4600 2750 0    60   Input ~ 0
 SW_LOW_RFIN
 Text HLabel 2500 6750 0    60   Input ~ 0
@@
 Text HLabel 6500 6900 2    50   Output ~ 0
 X2_FEED_RFOUT
-Text Notes 2300 2800 0    50   ~ 0
+Text Notes 4200 2600 0    50   ~ 0
 LPF, 8 GHz
 Text Notes 10300 10550 0    50   ~ 0
@@
 F 0 "U903" H 13000 7000 50  0000 C CNN
 F 1 "PE42543" H 12900 7100 50  0000 C CNN
-F 2 "" H 12250 6300 50  0001 C CNN
+F 2 "vna_mm:RFSW__PE42543A-X" H 12250 6300 50  0001 C CNN
 F 3 "https://www.psemi.com/pdf/datasheets/pe42543ds.pdf" H 12250 6300 50  0001 C CNN
 	1    12250 6300
@@
 F 0 "FL902" H 13800 6615 50  0000 C CNN
 F 1 "low_pass_filter" H 13800 6524 50  0000 C CNN
-F 2 "" H 13700 6450 50  0001 C CNN
+F 2 "vna_footprints:stepped_lpf_20ghz_fr408" H 13700 6450 50  0001 C CNN
 F 3 "" H 13700 6450 50  0001 C CNN
 	1    13800 6300
@@
 Text Label 11550 6450 2    50   ~ 0
 LOW_FILT
-Text Label 4200 2950 0    50   ~ 0
+Text Label 6100 2750 0    50   ~ 0
 LOW_FILT
 Wire Wire Line
-	4200 2950 4000 2950
+	6100 2750 5900 2750
 $Comp
 L power:GND #PWR0905
 U 1 1 5D5CD5D0
-P 3400 3450
-F 0 "#PWR0905" H 3400 3200 50  0001 C CNN
-F 1 "GND" H 3400 3300 50  0000 C CNN
-F 2 "" H 3400 3450 50  0001 C CNN
-F 3 "" H 3400 3450 50  0001 C CNN
-	1    3400 3450
-	1    0    0    -1
-$EndComp
-Wire Wire Line
-	3400 3400 3400 3450
+P 5300 3250
+F 0 "#PWR0905" H 5300 3000 50  0001 C CNN
+F 1 "GND" H 5300 3100 50  0000 C CNN
+F 2 "" H 5300 3250 50  0001 C CNN
+F 3 "" H 5300 3250 50  0001 C CNN
+	1    5300 3250
+	1    0    0    -1
+$EndComp
+Wire Wire Line
+	5300 3200 5300 3250
 $Comp
 L vna_mm:PE42543 U902
@@
 F 0 "U902" H 6550 7450 50  0000 C CNN
 F 1 "PE42543" H 6450 7550 50  0000 C CNN
-F 2 "" H 5800 6750 50  0001 C CNN
+F 2 "vna_mm:RFSW__PE42543A-X" H 5800 6750 50  0001 C CNN
 F 3 "https://www.psemi.com/pdf/datasheets/pe42543ds.pdf" H 5800 6750 50  0001 C CNN
 	1    5800 6750
@@
 MID
 Wire Wire Line
-	2700 2950 2800 2950
+	4600 2750 4700 2750
 $Comp
 L power:+3.3VP #PWR0930
@@
 L synth_lib:low_pass_filter FL901
 U 1 1 5D33146F
-P 3400 2950
-F 0 "FL901" H 3400 3265 50  0000 C CNN
-F 1 "low_pass_filter" H 3400 3174 50  0000 C CNN
-F 2 "" H 3300 3100 50  0001 C CNN
-F 3 "" H 3300 3100 50  0001 C CNN
-	1    3400 2950
+P 5300 2750
+F 0 "FL901" H 5300 3065 50  0000 C CNN
+F 1 "low_pass_filter" H 5300 2974 50  0000 C CNN
+F 2 "vna_footprints:stepped_lpf_8ghz_fr408" H 5200 2900 50  0001 C CNN
+F 3 "" H 5200 2900 50  0001 C CNN
+	1    5300 2750
 	1    0    0    -1
 $EndComp
@@
 Wire Wire Line
 	2700 8600 2700 9250
-Text HLabel 2500 7000 0    60   Input ~ 0
+Text HLabel 1050 7000 0    60   Input ~ 0
 FILT_VCTL
 Text HLabel 2500 7100 0    60   Input ~ 0
 FILT_VTUNE
-Wire Wire Line
-	2500 7000 2800 7000
 Wire Wire Line
 	2500 7100 2800 7100
@@
 $EndComp
 NoConn ~ 6500 6800
+$Comp
+L device:R_Small R903
+U 1 1 5E1ED397
+P 1250 7000
+F 0 "R903" V 1054 7000 50  0000 C CNN
+F 1 "TBD" V 1145 7000 50  0000 C CNN
+F 2 "Resistors_SMD:R_0402" H 1250 7000 60  0001 C CNN
+F 3 "" H 1250 7000 60  0000 C CNN
+	1    1250 7000
+	0    1    1    0
+$EndComp
+$Comp
+L device:R_Small R904
+U 1 1 5E1ED777
+P 1500 7250
+F 0 "R904" H 1559 7296 50  0000 L CNN
+F 1 "TBD" H 1559 7205 50  0000 L CNN
+F 2 "Resistors_SMD:R_0402" H 1500 7250 60  0001 C CNN
+F 3 "" H 1500 7250 60  0000 C CNN
+	1    1500 7250
+	1    0    0    -1
+$EndComp
+$Comp
+L power:GND #PWR0101
+U 1 1 5E1EDAA9
+P 1500 7450
+F 0 "#PWR0101" H 1500 7200 50  0001 C CNN
+F 1 "GND" H 1500 7300 50  0000 C CNN
+F 2 "" H 1500 7450 50  0001 C CNN
+F 3 "" H 1500 7450 50  0001 C CNN
+	1    1500 7450
+	-1   0    0    -1
+$EndComp
+Wire Wire Line
+	1350 7000 1500 7000
+Wire Wire Line
+	1500 7150 1500 7000
+Connection ~ 1500 7000
+Wire Wire Line
+	1500 7000 2800 7000
+Wire Wire Line
+	1150 7000 1050 7000
+Wire Wire Line
+	1500 7450 1500 7350
+Text Notes 3250 7700 0    50   ~ 0
+SEQUENCE:\n1 - VDD/VEE\n2 - VCTL\n3 - VTUNE
 $EndSCHEMATC

Commit message: started separate reference clock generation board
Changed lines of the file:
@@
 U 1 1 5D31C51E
 P 17800 8150
-F 0 "U904" H 17106 8097 60  0000 R CNN
-F 1 "ADRF5020" H 17106 8203 60  0000 R CNN
+F 0 "U904" H 17250 7650 60  0000 R CNN
+F 1 "ADRF5020" H 17250 7550 60  0000 R CNN
 F 2 "" H 17800 8150 60  0001 C CNN
 F 3 "" H 17800 8150 60  0001 C CNN

Commit message: component placement on vna ref board
Parts:
- FL901, FL902: symbol synth_lib:low_pass_filter -> vna_mm_synth-rescue:low_pass_filter-synth_lib
Changed lines of the file:
@@
 	12200 5100 12200 5500
 $Comp
-L synth_lib:low_pass_filter FL902
+L vna_mm_synth-rescue:low_pass_filter-synth_lib FL902
 U 1 1 5D55EE36
 P 13800 6300
@@
 $EndComp
 $Comp
-L synth_lib:low_pass_filter FL901
+L vna_mm_synth-rescue:low_pass_filter-synth_lib FL901
 U 1 1 5D33146F
 P 5300 2750

Commit message: cleanup and update vna mm synth schematic for modern kicad libraries
Parts:
- C901, C902, C903, C904, C905, C906, C907, C908, C909, C910, C911: footprint Capacitors_SMD:C_0402 -> Capacitor_SMD:C_0402_1005Metric; symbol device:C_Small -> Device:C_Small
- FL901, FL902: symbol vna_mm_synth-rescue:low_pass_filter-synth_lib -> vna_mm:low_pass_filter
- J901, J902: footprint (none) -> vna_mm:SF2921-61345
- L901, L902, L903, L904: footprint Resistors_SMD:R_0402 -> Inductor_SMD:L_0402_1005Metric
- R901, R902, R903, R904: footprint Resistors_SMD:R_0402 -> Resistor_SMD:R_0402_1005Metric; symbol device:R_Small -> Device:R_Small
Changed lines of the file:
@@
 $Descr A2 23386 16535
 encoding utf-8
-Sheet 9 12
+Sheet 9 11
 Title ""
 Date ""
@@
 $EndComp
 $Comp
-L device:C_Small C909
+L Device:C_Small C909
 U 1 1 5D2A18AE
 P 15750 7850
 F 0 "C909" H 15760 7920 50  0000 L CNN
 F 1 "10 pF" H 15760 7770 50  0000 L CNN
-F 2 "Capacitors_SMD:C_0402" H 15750 7850 50  0001 C CNN
+F 2 "Capacitor_SMD:C_0402_1005Metric" H 15750 7850 50  0001 C CNN
 F 3 "" H 15750 7850 50  0001 C CNN
 	1    15750 7850
@@
 $EndComp
 $Comp
-L device:R_Small R901
+L Device:R_Small R901
 U 1 1 5D2A18AD
 P 16000 8050
 F 0 "R901" H 16030 8070 50  0000 L CNN
 F 1 "1k" H 16030 8010 50  0000 L CNN
-F 2 "Resistors_SMD:R_0402" H 16000 8050 50  0001 C CNN
+F 2 "Resistor_SMD:R_0402_1005Metric" H 16000 8050 50  0001 C CNN
 F 3 "" H 16000 8050 50  0001 C CNN
 	1    16000 8050
@@
 $EndComp
 $Comp
-L device:R_Small R902
+L Device:R_Small R902
 U 1 1 5D2A18AB
 P 16550 8250
 F 0 "R902" H 16580 8270 50  0000 L CNN
 F 1 "1k" H 16580 8210 50  0000 L CNN
-F 2 "Resistors_SMD:R_0402" H 16550 8250 50  0001 C CNN
+F 2 "Resistor_SMD:R_0402_1005Metric" H 16550 8250 50  0001 C CNN
 F 3 "" H 16550 8250 50  0001 C CNN
 	1    16550 8250
@@
 $EndComp
 $Comp
-L device:C_Small C910
+L Device:C_Small C910
 U 1 1 5D2A18A9
 P 16850 7700
 F 0 "C910" H 16860 7770 50  0000 L CNN
 F 1 "10 pF" H 16860 7620 50  0000 L CNN
-F 2 "Capacitors_SMD:C_0402" H 16850 7700 50  0001 C CNN
+F 2 "Capacitor_SMD:C_0402_1005Metric" H 16850 7700 50  0001 C CNN
 F 3 "" H 16850 7700 50  0001 C CNN
 	1    16850 7700
@@
 $EndComp
 $Comp
-L device:C_Small C911
+L Device:C_Small C911
 U 1 1 5D2A18A6
 P 16850 8650
 F 0 "C911" H 16860 8720 50  0000 L CNN
 F 1 "10 pF" H 16860 8570 50  0000 L CNN
-F 2 "Capacitors_SMD:C_0402" H 16850 8650 50  0001 C CNN
+F 2 "Capacitor_SMD:C_0402_1005Metric" H 16850 8650 50  0001 C CNN
 F 3 "" H 16850 8650 50  0001 C CNN
 	1    16850 8650
@@
 $EndComp
 $Comp
-L device:C_Small C907
+L Device:C_Small C907
 U 1 1 5D515E00
 P 12650 5150
 F 0 "C907" H 12660 5220 50  0000 L CNN
 F 1 "100 pF" H 12660 5070 50  0000 L CNN
-F 2 "Capacitors_SMD:C_0402" H 12650 5150 50  0001 C CNN
+F 2 "Capacitor_SMD:C_0402_1005Metric" H 12650 5150 50  0001 C CNN
 F 3 "" H 12650 5150 50  0001 C CNN
 	1    12650 5150
@@
 $EndComp
 $Comp
-L device:C_Small C908
+L Device:C_Small C908
 U 1 1 5D5164E4
 P 13000 5150
 F 0 "C908" H 13010 5220 50  0000 L CNN
 F 1 "100 nF" H 13010 5070 50  0000 L CNN
-F 2 "Capacitors_SMD:C_0402" H 13000 5150 50  0001 C CNN
+F 2 "Capacitor_SMD:C_0402_1005Metric" H 13000 5150 50  0001 C CNN
 F 3 "" H 13000 5150 50  0001 C CNN
 	1    13000 5150
@@
 F 0 "L904" H 12448 4796 50  0000 L CNN
 F 1 "BLM15GG471" H 12448 4705 50  0000 L CNN
-F 2 "Resistors_SMD:R_0402" H 12400 4750 50  0001 C CNN
+F 2 "Inductor_SMD:L_0402_1005Metric" H 12400 4750 50  0001 C CNN
 F 3 "~" H 12400 4750 50  0001 C CNN
 	1    12400 4750
@@
 	12200 5100 12200 5500
 $Comp
-L vna_mm_synth-rescue:low_pass_filter-synth_lib FL902
+L vna_mm:low_pass_filter FL902
 U 1 1 5D55EE36
 P 13800 6300
@@
 $EndComp
 $Comp
-L device:C_Small C906
+L Device:C_Small C906
 U 1 1 5D5FFF9B
 P 5400 5600
 F 0 "C906" H 5410 5670 50  0000 L CNN
 F 1 "100 pF" H 5410 5520 50  0000 L CNN
-F 2 "Capacitors_SMD:C_0402" H 5400 5600 50  0001 C CNN
+F 2 "Capacitor_SMD:C_0402_1005Metric" H 5400 5600 50  0001 C CNN
 F 3 "" H 5400 5600 50  0001 C CNN
 	1    5400 5600
@@
 $EndComp
 $Comp
-L device:C_Small C905
+L Device:C_Small C905
 U 1 1 5D5FFFA1
 P 5050 5600
 F 0 "C905" H 5060 5670 50  0000 L CNN
 F 1 "100 nF" H 5060 5520 50  0000 L CNN
-F 2 "Capacitors_SMD:C_0402" H 5050 5600 50  0001 C CNN
+F 2 "Capacitor_SMD:C_0402_1005Metric" H 5050 5600 50  0001 C CNN
 F 3 "" H 5050 5600 50  0001 C CNN
 	1    5050 5600
@@
 F 0 "L903" H 5698 5246 50  0000 L CNN
 F 1 "BLM15GG471" H 5698 5155 50  0000 L CNN
-F 2 "Resistors_SMD:R_0402" H 5650 5200 50  0001 C CNN
+F 2 "Inductor_SMD:L_0402_1005Metric" H 5650 5200 50  0001 C CNN
 F 3 "~" H 5650 5200 50  0001 C CNN
 	1    5650 5200
@@
 $EndComp
 $Comp
-L vna_mm_synth-rescue:low_pass_filter-synth_lib FL901
+L vna_mm:low_pass_filter FL901
 U 1 1 5D33146F
 P 5300 2750
@@
 F 0 "J901" H 7850 5375 50  0000 L CNN
 F 1 "Conn_Coaxial" H 7850 5284 50  0000 L CNN
-F 2 "" H 7750 5400 50  0001 C CNN
+F 2 "vna_mm:SF2921-61345" H 7750 5400 50  0001 C CNN
 F 3 " ~" H 7750 5400 50  0001 C CNN
 	1    7750 5400
@@
 F 0 "J902" H 10200 5325 50  0000 L CNN
 F 1 "Conn_Coaxial" H 10200 5234 50  0000 L CNN
-F 2 "" H 10100 5350 50  0001 C CNN
+F 2 "vna_mm:SF2921-61345" H 10100 5350 50  0001 C CNN
 F 3 " ~" H 10100 5350 50  0001 C CNN
 	1    10100 5350
@@
 	3650 5650 4100 5650
 $Comp
-L device:C_Small C903
+L Device:C_Small C903
 U 1 1 5DB27BB7
 P 4100 5800
 F 0 "C903" H 4110 5870 50  0000 L CNN
 F 1 "100 pF" H 4110 5720 50  0000 L CNN
-F 2 "Capacitors_SMD:C_0402" H 4100 5800 50  0001 C CNN
+F 2 "Capacitor_SMD:C_0402_1005Metric" H 4100 5800 50  0001 C CNN
 F 3 "" H 4100 5800 50  0001 C CNN
 	1    4100 5800
@@
 $EndComp
 $Comp
-L device:C_Small C904
+L Device:C_Small C904
 U 1 1 5DB27680
 P 4450 5800
 F 0 "C904" H 4460 5870 50  0000 L CNN
 F 1 "100 nF" H 4460 5720 50  0000 L CNN
-F 2 "Capacitors_SMD:C_0402" H 4450 5800 50  0001 C CNN
+F 2 "Capacitor_SMD:C_0402_1005Metric" H 4450 5800 50  0001 C CNN
 F 3 "" H 4450 5800 50  0001 C CNN
 	1    4450 5800
@@
 	3350 5650 2900 5650
 $Comp
-L device:C_Small C902
+L Device:C_Small C902
 U 1 1 5DBB2C72
 P 2900 5800
 F 0 "C902" H 2910 5870 50  0000 L CNN
 F 1 "100 pF" H 2910 5720 50  0000 L CNN
-F 2 "Capacitors_SMD:C_0402" H 2900 5800 50  0001 C CNN
+F 2 "Capacitor_SMD:C_0402_1005Metric" H 2900 5800 50  0001 C CNN
 F 3 "" H 2900 5800 50  0001 C CNN
 	1    2900 5800
@@
 $EndComp
 $Comp
-L device:C_Small C901
+L Device:C_Small C901
 U 1 1 5DBB2C78
 P 2550 5800
 F 0 "C901" H 2560 5870 50  0000 L CNN
 F 1 "100 nF" H 2560 5720 50  0000 L CNN
-F 2 "Capacitors_SMD:C_0402" H 2550 5800 50  0001 C CNN
+F 2 "Capacitor_SMD:C_0402_1005Metric" H 2550 5800 50  0001 C CNN
 F 3 "" H 2550 5800 50  0001 C CNN
 	1    2550 5800
@@
 F 0 "L901" H 3398 5446 50  0000 L CNN
 F 1 "BLM15GG471" H 3398 5355 50  0000 L CNN
-F 2 "Resistors_SMD:R_0402" H 3350 5400 50  0001 C CNN
+F 2 "Inductor_SMD:L_0402_1005Metric" H 3350 5400 50  0001 C CNN
 F 3 "~" H 3350 5400 50  0001 C CNN
 	1    3350 5400
@@
 F 0 "L902" H 3500 5450 50  0000 L CNN
 F 1 "BLM15GG471" H 3100 5350 50  0000 L CNN
-F 2 "Resistors_SMD:R_0402" H 3650 5400 50  0001 C CNN
+F 2 "Inductor_SMD:L_0402_1005Metric" H 3650 5400 50  0001 C CNN
 F 3 "~" H 3650 5400 50  0001 C CNN
 	1    3650 5400
@@
 NoConn ~ 6500 6800
 $Comp
-L device:R_Small R903
+L Device:R_Small R903
 U 1 1 5E1ED397
 P 1250 7000
 F 0 "R903" V 1054 7000 50  0000 C CNN
 F 1 "TBD" V 1145 7000 50  0000 C CNN
-F 2 "Resistors_SMD:R_0402" H 1250 7000 60  0001 C CNN
+F 2 "Resistor_SMD:R_0402_1005Metric" H 1250 7000 60  0001 C CNN
 F 3 "" H 1250 7000 60  0000 C CNN
 	1    1250 7000
@@
 $EndComp
 $Comp
-L device:R_Small R904
+L Device:R_Small R904
 U 1 1 5E1ED777
 P 1500 7250
 F 0 "R904" H 1559 7296 50  0000 L CNN
 F 1 "TBD" H 1559 7205 50  0000 L CNN
-F 2 "Resistors_SMD:R_0402" H 1500 7250 60  0001 C CNN
+F 2 "Resistor_SMD:R_0402_1005Metric" H 1500 7250 60  0001 C CNN
 F 3 "" H 1500 7250 60  0000 C CNN
 	1    1500 7250
