File: hardware/vna_mm_synth/level_control.sch (KiCad schematic (older format))
At the start: 21 parts

Commit message: added power supply sequencing
Parts:
- gave numbers to parts that had none: 21

Commit message: added trl cal and set of breakout boards
Parts:
- C801, C802, C803, C804, C805, C806, C807, C808, C809, C811, C812, C813: footprint (none) -> Capacitors_SMD:C_0402
- C810, C814: footprint (none) -> Capacitors_SMD:C_0603
- L801, L802, L803, L804: value L_Small -> BLM15GG471; footprint (none) -> Resistors_SMD:R_0402

Commit message: fixed mirrored 3.3V regulator on sequencer board, created and assigned footprints for synth
Parts:
- U802, U803: footprint (none) -> vna_mm:MACOM_LGA9
Changed lines of the file:
@@
 F 0 "U802" H 5000 4500 50  0000 L CNN
 F 1 "MAAM-011109" H 5000 4600 50  0000 L CNN
-F 2 "" H 5800 4000 50  0001 C CNN
+F 2 "vna_mm:MACOM_LGA9" H 5800 4000 50  0001 C CNN
 F 3 "" H 5800 4000 50  0001 C CNN
 	1    5800 4000
@@
 F 0 "U803" H 7200 4500 50  0000 L CNN
 F 1 "MAAM-011109" H 7200 4600 50  0000 L CNN
-F 2 "" H 8000 4000 50  0001 C CNN
+F 2 "vna_mm:MACOM_LGA9" H 8000 4000 50  0001 C CNN
 F 3 "" H 8000 4000 50  0001 C CNN
 	1    8000 4000

Commit message: cleanup and update vna mm synth schematic for modern kicad libraries
Parts:
- C801, C802, C803, C804, C805, C806, C807, C808, C809, C811, C812, C813: footprint Capacitors_SMD:C_0402 -> Capacitor_SMD:C_0402_1005Metric
- C810, C814: footprint Capacitors_SMD:C_0603 -> Capacitor_SMD:C_0603_1608Metric
- L801, L802, L803, L804: footprint Resistors_SMD:R_0402 -> Inductor_SMD:L_0402_1005Metric
Changed lines of the file:
@@
 $Descr A4 11693 8268
 encoding utf-8
-Sheet 8 12
+Sheet 8 11
 Title ""
 Date ""
@@
 F 0 "C813" H 9242 2946 50  0000 L CNN
 F 1 "100 nF" H 9242 2855 50  0000 L CNN
-F 2 "Capacitors_SMD:C_0402" H 9150 2900 50  0001 C CNN
+F 2 "Capacitor_SMD:C_0402_1005Metric" H 9150 2900 50  0001 C CNN
 F 3 "~" H 9150 2900 50  0001 C CNN
 	1    9150 2900
@@
 F 0 "C812" H 8742 2946 50  0000 L CNN
 F 1 "100 pF" H 8742 2855 50  0000 L CNN
-F 2 "Capacitors_SMD:C_0402" H 8650 2900 50  0001 C CNN
+F 2 "Capacitor_SMD:C_0402_1005Metric" H 8650 2900 50  0001 C CNN
 F 3 "~" H 8650 2900 50  0001 C CNN
 	1    8650 2900
@@
 F 0 "C808" H 7042 2946 50  0000 L CNN
 F 1 "100 nF" H 7042 2855 50  0000 L CNN
-F 2 "Capacitors_SMD:C_0402" H 6950 2900 50  0001 C CNN
+F 2 "Capacitor_SMD:C_0402_1005Metric" H 6950 2900 50  0001 C CNN
 F 3 "~" H 6950 2900 50  0001 C CNN
 	1    6950 2900
@@
 F 0 "C807" H 6542 2946 50  0000 L CNN
 F 1 "100 pF" H 6542 2855 50  0000 L CNN
-F 2 "Capacitors_SMD:C_0402" H 6450 2900 50  0001 C CNN
+F 2 "Capacitor_SMD:C_0402_1005Metric" H 6450 2900 50  0001 C CNN
 F 3 "~" H 6450 2900 50  0001 C CNN
 	1    6450 2900
@@
 F 0 "C810" H 7542 2946 50  0000 L CNN
 F 1 "2.2 uF" H 7542 2855 50  0000 L CNN
-F 2 "Capacitors_SMD:C_0603" H 7450 2900 50  0001 C CNN
+F 2 "Capacitor_SMD:C_0603_1608Metric" H 7450 2900 50  0001 C CNN
 F 3 "~" H 7450 2900 50  0001 C CNN
 	1    7450 2900
@@
 F 0 "C814" H 9742 2946 50  0000 L CNN
 F 1 "2.2 uF" H 9742 2855 50  0000 L CNN
-F 2 "Capacitors_SMD:C_0603" H 9650 2900 50  0001 C CNN
+F 2 "Capacitor_SMD:C_0603_1608Metric" H 9650 2900 50  0001 C CNN
 F 3 "~" H 9650 2900 50  0001 C CNN
 	1    9650 2900
@@
 F 0 "C806" H 5392 5396 50  0000 L CNN
 F 1 "100 nF" H 5392 5305 50  0000 L CNN
-F 2 "Capacitors_SMD:C_0402" H 5300 5350 50  0001 C CNN
+F 2 "Capacitor_SMD:C_0402_1005Metric" H 5300 5350 50  0001 C CNN
 F 3 "~" H 5300 5350 50  0001 C CNN
 	1    5300 5350
@@
 F 0 "C805" H 4892 5396 50  0000 L CNN
 F 1 "100 pF" H 4892 5305 50  0000 L CNN
-F 2 "Capacitors_SMD:C_0402" H 4800 5350 50  0001 C CNN
+F 2 "Capacitor_SMD:C_0402_1005Metric" H 4800 5350 50  0001 C CNN
 F 3 "~" H 4800 5350 50  0001 C CNN
 	1    4800 5350
@@
 F 0 "C811" H 7592 5396 50  0000 L CNN
 F 1 "100 nF" H 7592 5305 50  0000 L CNN
-F 2 "Capacitors_SMD:C_0402" H 7500 5350 50  0001 C CNN
+F 2 "Capacitor_SMD:C_0402_1005Metric" H 7500 5350 50  0001 C CNN
 F 3 "~" H 7500 5350 50  0001 C CNN
 	1    7500 5350
@@
 F 0 "C809" H 7092 5396 50  0000 L CNN
 F 1 "100 pF" H 7092 5305 50  0000 L CNN
-F 2 "Capacitors_SMD:C_0402" H 7000 5350 50  0001 C CNN
+F 2 "Capacitor_SMD:C_0402_1005Metric" H 7000 5350 50  0001 C CNN
 F 3 "~" H 7000 5350 50  0001 C CNN
 	1    7000 5350
@@
 F 0 "C803" H 4242 2096 50  0000 L CNN
 F 1 "100 pF" H 4242 2005 50  0000 L CNN
-F 2 "Capacitors_SMD:C_0402" H 4150 2050 50  0001 C CNN
+F 2 "Capacitor_SMD:C_0402_1005Metric" H 4150 2050 50  0001 C CNN
 F 3 "~" H 4150 2050 50  0001 C CNN
 	1    4150 2050
@@
 F 0 "L803" H 6248 2496 50  0000 L CNN
 F 1 "BLM15GG471" H 6248 2405 50  0000 L CNN
-F 2 "Resistors_SMD:R_0402" H 6200 2450 50  0001 C CNN
+F 2 "Inductor_SMD:L_0402_1005Metric" H 6200 2450 50  0001 C CNN
 F 3 "~" H 6200 2450 50  0001 C CNN
 	1    6200 2450
@@
 F 0 "L804" H 8448 2446 50  0000 L CNN
 F 1 "BLM15GG471" H 8448 2355 50  0000 L CNN
-F 2 "Resistors_SMD:R_0402" H 8400 2400 50  0001 C CNN
+F 2 "Inductor_SMD:L_0402_1005Metric" H 8400 2400 50  0001 C CNN
 F 3 "~" H 8400 2400 50  0001 C CNN
 	1    8400 2400
@@
 F 0 "L802" H 3998 1546 50  0000 L CNN
 F 1 "BLM15GG471" H 3998 1455 50  0000 L CNN
-F 2 "Resistors_SMD:R_0402" H 3950 1500 50  0001 C CNN
+F 2 "Inductor_SMD:L_0402_1005Metric" H 3950 1500 50  0001 C CNN
 F 3 "~" H 3950 1500 50  0001 C CNN
 	1    3950 1500
@@
 F 0 "C804" H 4742 2096 50  0000 L CNN
 F 1 "100 nF" H 4742 2005 50  0000 L CNN
-F 2 "Capacitors_SMD:C_0402" H 4650 2050 50  0001 C CNN
+F 2 "Capacitor_SMD:C_0402_1005Metric" H 4650 2050 50  0001 C CNN
 F 3 "~" H 4650 2050 50  0001 C CNN
 	1    4650 2050
@@
 F 0 "C802" H 3492 2096 50  0000 L CNN
 F 1 "100 pF" H 3492 2005 50  0000 L CNN
-F 2 "Capacitors_SMD:C_0402" H 3400 2050 50  0001 C CNN
+F 2 "Capacitor_SMD:C_0402_1005Metric" H 3400 2050 50  0001 C CNN
 F 3 "~" H 3400 2050 50  0001 C CNN
 	1    3400 2050
@@
 F 0 "L801" H 3648 1546 50  0000 L CNN
 F 1 "BLM15GG471" H 3648 1455 50  0000 L CNN
-F 2 "Resistors_SMD:R_0402" H 3600 1500 50  0001 C CNN
+F 2 "Inductor_SMD:L_0402_1005Metric" H 3600 1500 50  0001 C CNN
 F 3 "~" H 3600 1500 50  0001 C CNN
 	1    3600 1500
@@
 F 0 "C801" H 2992 2096 50  0000 L CNN
 F 1 "100 nF" H 2992 2005 50  0000 L CNN
-F 2 "Capacitors_SMD:C_0402" H 2900 2050 50  0001 C CNN
+F 2 "Capacitor_SMD:C_0402_1005Metric" H 2900 2050 50  0001 C CNN
 F 3 "~" H 2900 2050 50  0001 C CNN
 	1    2900 2050

Commit message: footprint assignment on vna_mm_synth
Parts:
- U801: footprint (none) -> vna_mm:LGA-24_EP_4x4_Pitch0.5mm
Changed lines of the file:
@@
 EESchema Schematic File Version 4
-LIBS:vna_mm_synth-cache
 EELAYER 30 0
 EELAYER END
@@
 F 0 "U801" H 2150 4750 50  0000 L CNN
 F 1 "ADRF5730" H 2150 4850 50  0000 L CNN
-F 2 "" H 3200 3700 50  0001 C CNN
+F 2 "vna_mm:LGA-24_EP_4x4_Pitch0.5mm" H 3200 3700 50  0001 C CNN
 F 3 "https://www.analog.com/media/en/technical-documentation/data-sheets/ADRF5730.pdf" H 3200 3700 50  0001 C CNN
 	1    3250 4000

Commit message: synth schematic cleanup
Parts:
- renumbered C801 to C1101, C802 to C1102, C803 to C1103, C804 to C1104, C805 to C1105, C806 to C1106, C807 to C1107, C808 to C1108, C809 to C1109, C810 to C1110, C811 to C1111, C812 to C1112, C813 to C1113, C814 to C1114, L801 to L1101, L802 to L1102, L803 to L1103, L804 to L1104, U801 to U1101, U802 to U1102, U803 to U1103
