File: hardware/vna_mm_synth/conn_front.sch (KiCad schematic (older format))
At the start: 4 parts, among them U501 CONN_SMA_2GND, U502 CONN_SMA_2GND

Commit message: added power supply sequencing
Parts:
- removed U501, U502: CONN_SMA_2GND, vna_footprints:SMA_901-10512_6p7MIL_FR408_CPW_LAUNCH, symbol conn_sma_2gnd:CONN_SMA_2GND
- added J301, J302: Conn_Coaxial, symbol Connector:Conn_Coaxial
Connections:
- wire segments 14 -> 6
Changed lines of the file:
@@
 SYNC
-$Comp
-L conn_sma_2gnd:CONN_SMA_2GND U501
-U 1 1 5AB94261
-P 6050 1600
-F 0 "U501" H 5750 1800 60  0000 C CNN
-F 1 "CONN_SMA_2GND" H 6100 1900 60  0000 C CNN
-F 2 "vna_footprints:SMA_901-10512_6p7MIL_FR408_CPW_LAUNCH" H 6050 1600 60  0001 C CNN
-F 3 "" H 6050 1600 60  0000 C CNN
-	1    6050 1600
-	-1   0    0    -1
-$EndComp
 $Comp
 L power:GND #PWR077
 U 1 1 5AB94285
-P 6050 2150
-F 0 "#PWR077" H 6050 1900 50  0001 C CNN
-F 1 "GND" H 6050 2000 50  0000 C CNN
-F 2 "" H 6050 2150 50  0001 C CNN
-F 3 "" H 6050 2150 50  0001 C CNN
-	1    6050 2150
+P 5850 1900
+F 0 "#PWR077" H 5850 1650 50  0001 C CNN
+F 1 "GND" H 5850 1750 50  0000 C CNN
+F 2 "" H 5850 1900 50  0001 C CNN
+F 3 "" H 5850 1900 50  0001 C CNN
+	1    5850 1900
 	1    0    0    -1
-$EndComp
-$Comp
-L conn_sma_2gnd:CONN_SMA_2GND U502
-U 1 1 5ABBB801
-P 6050 2700
-F 0 "U502" H 5750 2900 60  0000 C CNN
-F 1 "CONN_SMA_2GND" H 6100 3000 60  0000 C CNN
-F 2 "vna_footprints:SMA_901-10512_6p7MIL_FR408_CPW_LAUNCH" H 6050 2700 60  0001 C CNN
-F 3 "" H 6050 2700 60  0000 C CNN
-	1    6050 2700
-	-1   0    0    -1
 $EndComp
 $Comp
 L power:GND #PWR078
 U 1 1 5ABBB807
-P 6050 3250
-F 0 "#PWR078" H 6050 3000 50  0001 C CNN
-F 1 "GND" H 6050 3100 50  0000 C CNN
-F 2 "" H 6050 3250 50  0001 C CNN
-F 3 "" H 6050 3250 50  0001 C CNN
-	1    6050 3250
+P 5850 3000
+F 0 "#PWR078" H 5850 2750 50  0001 C CNN
+F 1 "GND" H 5850 2850 50  0000 C CNN
+F 2 "" H 5850 3000 50  0001 C CNN
+F 3 "" H 5850 3000 50  0001 C CNN
+	1    5850 3000
 	1    0    0    -1
 $EndComp
 Wire Wire Line
-	6000 2050 6000 2100
-Wire Wire Line
-	6000 2100 6050 2100
-Wire Wire Line
-	6100 2100 6100 2050
-Wire Wire Line
-	6050 2100 6050 2150
-Connection ~ 6050 2100
-Wire Wire Line
 	5300 1600 5650 1600
-Wire Wire Line
-	6000 3150 6000 3200
-Wire Wire Line
-	6000 3200 6050 3200
-Wire Wire Line
-	6100 3200 6100 3150
-Wire Wire Line
-	6050 3200 6050 3250
-Connection ~ 6050 3200
 Wire Wire Line
 	5300 2700 5650 2700
@@
 	0    1    1    0
 $EndComp
+$Comp
+L Connector:Conn_Coaxial J301
+U 1 1 5D641233
+P 5850 1600
+F 0 "J301" H 5950 1575 50  0000 L CNN
+F 1 "Conn_Coaxial" H 5950 1484 50  0000 L CNN
+F 2 "" H 5850 1600 50  0001 C CNN
+F 3 " ~" H 5850 1600 50  0001 C CNN
+	1    5850 1600
+	1    0    0    -1
+$EndComp
+$Comp
+L Connector:Conn_Coaxial J302
+U 1 1 5D64149F
+P 5850 2700
+F 0 "J302" H 5950 2675 50  0000 L CNN
+F 1 "Conn_Coaxial" H 5950 2584 50  0000 L CNN
+F 2 "" H 5850 2700 50  0001 C CNN
+F 3 " ~" H 5850 2700 50  0001 C CNN
+	1    5850 2700
+	1    0    0    -1
+$EndComp
 Wire Wire Line
-	6050 2100 6100 2100
+	5850 1800 5850 1900
 Wire Wire Line
-	6050 3200 6100 3200
+	5850 3000 5850 2900
 $EndSCHEMATC

Commit message: added trl cal and set of breakout boards
Parts:
- C301: renamed from C501; footprint Capacitors_SMD:C_0201 -> Capacitors_SMD:C_0402
- C302: renamed from C502; footprint Capacitors_SMD:C_0201 -> Capacitors_SMD:C_0402
Changed lines of the file:
@@
 SYNC
 $Comp
-L power:GND #PWR077
+L power:GND #PWR0301
 U 1 1 5AB94285
 P 5850 1900
-F 0 "#PWR077" H 5850 1650 50  0001 C CNN
+F 0 "#PWR0301" H 5850 1650 50  0001 C CNN
 F 1 "GND" H 5850 1750 50  0000 C CNN
 F 2 "" H 5850 1900 50  0001 C CNN
@@
 $EndComp
 $Comp
-L power:GND #PWR078
+L power:GND #PWR0302
 U 1 1 5ABBB807
 P 5850 3000
-F 0 "#PWR078" H 5850 2750 50  0001 C CNN
+F 0 "#PWR0302" H 5850 2750 50  0001 C CNN
 F 1 "GND" H 5850 2850 50  0000 C CNN
 F 2 "" H 5850 3000 50  0001 C CNN
@@
 	5100 2700 4900 2700
 $Comp
-L device:C_Small C502
+L device:C_Small C302
 U 1 1 5AC31626
 P 5200 2700
-F 0 "C502" H 5210 2770 50  0000 L CNN
+F 0 "C302" H 5210 2770 50  0000 L CNN
 F 1 "10 pF" H 5210 2620 50  0000 L CNN
-F 2 "Capacitors_SMD:C_0201" H 5200 2700 50  0001 C CNN
+F 2 "Capacitors_SMD:C_0402" H 5200 2700 50  0001 C CNN
 F 3 "" H 5200 2700 50  0001 C CNN
 	1    5200 2700
@@
 $EndComp
 $Comp
-L device:C_Small C501
+L device:C_Small C301
 U 1 1 5AC31536
 P 5200 1600
-F 0 "C501" H 5210 1670 50  0000 L CNN
+F 0 "C301" H 5210 1670 50  0000 L CNN
 F 1 "10 pF" H 5210 1520 50  0000 L CNN
-F 2 "Capacitors_SMD:C_0201" H 5200 1600 50  0001 C CNN
+F 2 "Capacitors_SMD:C_0402" H 5200 1600 50  0001 C CNN
 F 3 "" H 5200 1600 50  0001 C CNN
 	1    5200 1600

Commit message: cleanup and update vna mm synth schematic for modern kicad libraries
Parts:
- C301, C302: footprint Capacitors_SMD:C_0402 -> Capacitor_SMD:C_0402_1005Metric; symbol device:C_Small -> Device:C_Small
Changed lines of the file:
@@
 $Descr A4 11693 8268
 encoding utf-8
-Sheet 3 12
+Sheet 3 11
 Title ""
 Date ""
@@
 	5100 2700 4900 2700
 $Comp
-L device:C_Small C302
+L Device:C_Small C302
 U 1 1 5AC31626
 P 5200 2700
 F 0 "C302" H 5210 2770 50  0000 L CNN
 F 1 "10 pF" H 5210 2620 50  0000 L CNN
-F 2 "Capacitors_SMD:C_0402" H 5200 2700 50  0001 C CNN
+F 2 "Capacitor_SMD:C_0402_1005Metric" H 5200 2700 50  0001 C CNN
 F 3 "" H 5200 2700 50  0001 C CNN
 	1    5200 2700
@@
 $EndComp
 $Comp
-L device:C_Small C301
+L Device:C_Small C301
 U 1 1 5AC31536
 P 5200 1600
 F 0 "C301" H 5210 1670 50  0000 L CNN
 F 1 "10 pF" H 5210 1520 50  0000 L CNN
-F 2 "Capacitors_SMD:C_0402" H 5200 1600 50  0001 C CNN
+F 2 "Capacitor_SMD:C_0402_1005Metric" H 5200 1600 50  0001 C CNN
 F 3 "" H 5200 1600 50  0001 C CNN
 	1    5200 1600

Commit message: footprint assignment
Parts:
- J301: footprint (none) -> vna_mm:sw_edge_ro4350b_10mil
- J302: footprint (none) -> Connector_Coaxial:SMA_Amphenol_132203-12_Horizontal
Changed lines of the file:
@@
 F 0 "J301" H 5950 1575 50  0000 L CNN
 F 1 "Conn_Coaxial" H 5950 1484 50  0000 L CNN
-F 2 "" H 5850 1600 50  0001 C CNN
+F 2 "vna_mm:sw_edge_ro4350b_10mil" H 5850 1600 50  0001 C CNN
 F 3 " ~" H 5850 1600 50  0001 C CNN
 	1    5850 1600
@@
 F 0 "J302" H 5950 2675 50  0000 L CNN
 F 1 "Conn_Coaxial" H 5950 2584 50  0000 L CNN
-F 2 "" H 5850 2700 50  0001 C CNN
+F 2 "Connector_Coaxial:SMA_Amphenol_132203-12_Horizontal" H 5850 2700 50  0001 C CNN
 F 3 " ~" H 5850 2700 50  0001 C CNN
 	1    5850 2700
