File: breakouts/adc_32xx/ram_adc/adc_frontend_A.sch (KiCad schematic (older format))
At the start: 26 parts, among them T201 MABAES0060, T202 MABAES0060

Commit message: finished first pass adc32xx schematic
Parts:
- added J301: Conn_Coaxial, vna_footprints:732512200_SMA, symbol Connector:Conn_Coaxial
- renumbered C201 to C301, C202 to C302, C203 to C303, C204 to C304, C205 to C305, C206 to C306, C207 to C307, L201 to L301, L202 to L302, L203 to L303, R201 to R301, R202 to R302, R4 to R303, R5 to R304, R203 to R305, R204 to R306, R205 to R307, R206 to R308, R207 to R309, R208 to R310, R209 to R311, R210 to R312, R211 to R313, R212 to R314, T201 to T301, T202 to T302
Connections:
- net GND: now also J301.1 (In)
- net IN_P: no longer names the net of R301.1
- net IN_P: now also J301.2 (Ext)

Commit message: component placement for adc322x breakout
Connections:
- net GND: now also J301.2 (Ext); no longer J301.1 (In)
- net at R301.1: now also J301.1 (In); no longer J301.2 (Ext)
- net OUT_M renamed OUT_N
Changed lines of the file:
@@
 $Descr A4 11693 8268
 encoding utf-8
-Sheet 3 5
+Sheet 2 5
 Title ""
 Date ""
@@
 OUT_P
 Text HLabel 8850 3900 2    50   Output ~ 0
-OUT_M
+OUT_N
 Wire Wire Line
 	1150 3200 1350 3200
@@
 F 3 " ~" H 950 3200 50  0001 C CNN
 	1    950  3200
-	0    -1   -1   0
-$EndComp
-Wire Wire Line
+	-1   0    0    -1
+$EndComp
+Wire Wire Line

Commit message: finished layout of adc32xx ecp5 board
Changed lines of the file:
@@
 AR Path="/5E9D71BC/5D14AF40" Ref="#PWR?"  Part="1"
 AR Path="/5E9E6BF0/5D14AF40" Ref="#PWR0401"  Part="1"
-F 0 "#PWR0301" H 1750 3700 50  0001 C CNN
+F 0 "#PWR0401" H 1750 3700 50  0001 C CNN
 F 1 "GND" H 1755 3777 50  0000 C CNN
 F 2 "" H 1750 3950 50  0001 C CNN
@@
 AR Path="/5E9D71BC/5D14B53A" Ref="C?"  Part="1"
 AR Path="/5E9E6BF0/5D14B53A" Ref="C401"  Part="1"
-F 0 "C301" H 2892 3996 50  0000 L CNN
+F 0 "C401" H 2892 3996 50  0000 L CNN
 F 1 "100 nF" H 2892 3905 50  0000 L CNN
 F 2 "Capacitor_SMD:C_0402_1005Metric" H 2800 3950 50  0001 C CNN
@@
 AR Path="/5E9D71BC/5D14E9F5" Ref="C?"  Part="1"
 AR Path="/5E9E6BF0/5D14E9F5" Ref="C402"  Part="1"
-F 0 "C302" H 3942 3996 50  0000 L CNN
+F 0 "C402" H 3942 3996 50  0000 L CNN
 F 1 "100 nF" H 3942 3905 50  0000 L CNN
 F 2 "Capacitor_SMD:C_0402_1005Metric" H 3850 3950 50  0001 C CNN
@@
 AR Path="/5E9D71BC/5D152365" Ref="#PWR?"  Part="1"
 AR Path="/5E9E6BF0/5D152365" Ref="#PWR0402"  Part="1"
-F 0 "#PWR0302" H 2800 3850 50  0001 C CNN
+F 0 "#PWR0402" H 2800 3850 50  0001 C CNN
 F 1 "GND" H 2805 3927 50  0000 C CNN
 F 2 "" H 2800 4100 50  0001 C CNN
@@
 AR Path="/5E9D71BC/5D152B62" Ref="#PWR?"  Part="1"
 AR Path="/5E9E6BF0/5D152B62" Ref="#PWR0405"  Part="1"
-F 0 "#PWR0305" H 3850 3850 50  0001 C CNN
+F 0 "#PWR0405" H 3850 3850 50  0001 C CNN
 F 1 "GND" H 3855 3927 50  0000 C CNN
 F 2 "" H 3850 4100 50  0001 C CNN
@@
 AR Path="/5E9D71BC/5D1549DC" Ref="C?"  Part="1"
 AR Path="/5E9E6BF0/5D1549DC" Ref="C403"  Part="1"
-F 0 "C303" V 4871 3200 50  0000 C CNN
+F 0 "C403" V 4871 3200 50  0000 C CNN
 F 1 "100 nF" V 4962 3200 50  0000 C CNN
 F 2 "Capacitor_SMD:C_0402_1005Metric" H 5100 3200 50  0001 C CNN
@@
 AR Path="/5E9D71BC/5D154D50" Ref="C?"  Part="1"
 AR Path="/5E9E6BF0/5D154D50" Ref="C404"  Part="1"
-F 0 "C304" V 4871 3600 50  0000 C CNN
+F 0 "C404" V 4871 3600 50  0000 C CNN
 F 1 "100 nF" V 4962 3600 50  0000 C CNN
 F 2 "Capacitor_SMD:C_0402_1005Metric" H 5100 3600 50  0001 C CNN
@@
 AR Path="/5E9D71BC/5D155666" Ref="R?"  Part="1"
 AR Path="/5E9E6BF0/5D155666" Ref="R405"  Part="1"
-F 0 "R305" V 5354 3200 50  0000 C CNN
+F 0 "R405" V 5354 3200 50  0000 C CNN
 F 1 "50" V 5445 3200 50  0000 C CNN
 F 2 "Resistor_SMD:R_0402_1005Metric" H 5550 3200 50  0001 C CNN
@@
 AR Path="/5E9D71BC/5D155DBC" Ref="R?"  Part="1"
 AR Path="/5E9E6BF0/5D155DBC" Ref="R406"  Part="1"
-F 0 "R306" V 5354 3600 50  0000 C CNN
+F 0 "R406" V 5354 3600 50  0000 C CNN
 F 1 "50" V 5445 3600 50  0000 C CNN
 F 2 "Resistor_SMD:R_0402_1005Metric" H 5550 3600 50  0001 C CNN
@@
 AR Path="/5E9D71BC/5D156324" Ref="R?"  Part="1"
 AR Path="/5E9E6BF0/5D156324" Ref="R407"  Part="1"
-F 0 "R307" H 6141 3104 50  0000 R CNN
+F 0 "R407" H 6141 3104 50  0000 R CNN
 F 1 "25" H 6141 3195 50  0000 R CNN
 F 2 "Resistor_SMD:R_0402_1005Metric" H 6200 3150 50  0001 C CNN
@@
 AR Path="/5E9D71BC/5D156A75" Ref="R?"  Part="1"
 AR Path="/5E9E6BF0/5D156A75" Ref="R408"  Part="1"
-F 0 "R308" H 6141 3604 50  0000 R CNN
+F 0 "R408" H 6141 3604 50  0000 R CNN
 F 1 "25" H 6141 3695 50  0000 R CNN
 F 2 "Resistor_SMD:R_0402_1005Metric" H 6200 3650 50  0001 C CNN
@@
 AR Path="/5E9D71BC/5D1570AC" Ref="L?"  Part="1"
 AR Path="/5E9E6BF0/5D1570AC" Ref="L401"  Part="1"
-F 0 "L301" V 5735 2900 50  0000 C CNN
+F 0 "L401" V 5735 2900 50  0000 C CNN
 F 1 "39 nH" V 5644 2900 50  0000 C CNN
 F 2 "Resistor_SMD:R_0402_1005Metric" H 5550 2900 50  0001 C CNN
@@
 AR Path="/5E9D71BC/5D1580B6" Ref="L?"  Part="1"
 AR Path="/5E9E6BF0/5D1580B6" Ref="L402"  Part="1"
-F 0 "L302" V 5735 3900 50  0000 C CNN
+F 0 "L402" V 5735 3900 50  0000 C CNN
 F 1 "39 nH" V 5644 3900 50  0000 C CNN
 F 2 "Resistor_SMD:R_0402_1005Metric" H 5550 3900 50  0001 C CNN
@@
 AR Path="/5E9D71BC/5D15A649" Ref="C?"  Part="1"
 AR Path="/5E9E6BF0/5D15A649" Ref="C405"  Part="1"
-F 0 "C305" H 6458 3454 50  0000 R CNN
+F 0 "C405" H 6458 3454 50  0000 R CNN
 F 1 "100 nF" H 6458 3545 50  0000 R CNN
 F 2 "Capacitor_SMD:C_0402_1005Metric" H 6550 3500 50  0001 C CNN
@@
 AR Path="/5E9D71BC/5D15ABBB" Ref="#PWR?"  Part="1"
 AR Path="/5E9E6BF0/5D15ABBB" Ref="#PWR0406"  Part="1"
-F 0 "#PWR0306" H 6550 3400 50  0001 C CNN
+F 0 "#PWR0406" H 6550 3400 50  0001 C CNN
 F 1 "GND" H 6555 3477 50  0000 C CNN
 F 2 "" H 6550 3650 50  0001 C CNN
@@
 AR Path="/5E9D71BC/5D15B56D" Ref="C?"  Part="1"
 AR Path="/5E9E6BF0/5D15B56D" Ref="C406"  Part="1"
-F 0 "C306" H 6908 3454 50  0000 R CNN
+F 0 "C406" H 6908 3454 50  0000 R CNN
 F 1 "100 nF" H 6908 3545 50  0000 R CNN
 F 2 "Capacitor_SMD:C_0402_1005Metric" H 7000 3500 50  0001 C CNN
@@
 AR Path="/5E9D71BC/5D15B9B2" Ref="#PWR?"  Part="1"
 AR Path="/5E9E6BF0/5D15B9B2" Ref="#PWR0407"  Part="1"
-F 0 "#PWR0307" H 7000 3400 50  0001 C CNN
+F 0 "#PWR0407" H 7000 3400 50  0001 C CNN
 F 1 "GND" H 7005 3477 50  0000 C CNN
 F 2 "" H 7000 3650 50  0001 C CNN
@@
 AR Path="/5E9D71BC/5D16026F" Ref="R?"  Part="1"
 AR Path="/5E9E6BF0/5D16026F" Ref="R409"  Part="1"
-F 0 "R309" V 7596 2900 50  0000 C CNN
+F 0 "R409" V 7596 2900 50  0000 C CNN
 F 1 "0" V 7505 2900 50  0000 C CNN
 F 2 "Resistor_SMD:R_0402_1005Metric" H 7400 2900 50  0001 C CNN
@@
 AR Path="/5E9D71BC/5D16056A" Ref="R?"  Part="1"
 AR Path="/5E9E6BF0/5D16056A" Ref="R410"  Part="1"
-F 0 "R310" V 7596 3900 50  0000 C CNN
+F 0 "R410" V 7596 3900 50  0000 C CNN
 F 1 "0" V 7505 3900 50  0000 C CNN
 F 2 "Resistor_SMD:R_0402_1005Metric" H 7400 3900 50  0001 C CNN
@@
 AR Path="/5E9D71BC/5D166300" Ref="R?"  Part="1"
 AR Path="/5E9E6BF0/5D166300" Ref="R411"  Part="1"
-F 0 "R311" H 7641 3054 50  0000 R CNN
+F 0 "R411" H 7641 3054 50  0000 R CNN
 F 1 "25" H 7641 3145 50  0000 R CNN
 F 2 "Resistor_SMD:R_0402_1005Metric" H 7700 3100 50  0001 C CNN
@@
 AR Path="/5E9D71BC/5D1666F8" Ref="R?"  Part="1"
 AR Path="/5E9E6BF0/5D1666F8" Ref="R412"  Part="1"
-F 0 "R312" H 7641 3654 50  0000 R CNN
+F 0 "R412" H 7641 3654 50  0000 R CNN
 F 1 "25" H 7641 3745 50  0000 R CNN
 F 2 "Resistor_SMD:R_0402_1005Metric" H 7700 3700 50  0001 C CNN
@@
 AR Path="/5E9D71BC/5D166DF8" Ref="C?"  Part="1"
 AR Path="/5E9E6BF0/5D166DF8" Ref="C407"  Part="1"
-F 0 "C307" H 7608 3354 50  0000 R CNN
+F 0 "C407" H 7608 3354 50  0000 R CNN
 F 1 "10 pF" H 7608 3445 50  0000 R CNN
 F 2 "Capacitor_SMD:C_0402_1005Metric" H 7700 3400 50  0001 C CNN
@@
 AR Path="/5E9D71BC/5D167101" Ref="L?"  Part="1"
 AR Path="/5E9E6BF0/5D167101" Ref="L403"  Part="1"
-F 0 "L303" H 8148 3446 50  0000 L CNN
+F 0 "L403" H 8148 3446 50  0000 L CNN
 F 1 "10 pF" H 8148 3355 50  0000 L CNN
 F 2 "Resistor_SMD:R_0402_1005Metric" H 8100 3400 50  0001 C CNN
@@
 AR Path="/5E9D71BC/5D16CFF7" Ref="R?"  Part="1"
 AR Path="/5E9E6BF0/5D16CFF7" Ref="R413"  Part="1"
-F 0 "R313" V 8496 2900 50  0000 C CNN
+F 0 "R413" V 8496 2900 50  0000 C CNN
 F 1 "15" V 8405 2900 50  0000 C CNN
 F 2 "Resistor_SMD:R_0402_1005Metric" H 8300 2900 50  0001 C CNN
@@
 AR Path="/5E9D71BC/5D16D51A" Ref="R?"  Part="1"
 AR Path="/5E9E6BF0/5D16D51A" Ref="R414"  Part="1"
-F 0 "R314" V 8496 3900 50  0000 C CNN
+F 0 "R414" V 8496 3900 50  0000 C CNN
 F 1 "15" V 8405 3900 50  0000 C CNN
 F 2 "Resistor_SMD:R_0402_1005Metric" H 8300 3900 50  0001 C CNN
@@
 AR Path="/5E9D71BC/5D1749B4" Ref="R?"  Part="1"
 AR Path="/5E9E6BF0/5D1749B4" Ref="R402"  Part="1"
-F 0 "R302" H 1691 3754 50  0000 R CNN
+F 0 "R402" H 1691 3754 50  0000 R CNN
 F 1 "0" H 1691 3845 50  0000 R CNN
 F 2 "Resistor_SMD:R_0402_1005Metric" H 1750 3800 50  0001 C CNN
@@
 AR Path="/5E9D71BC/5D1770D6" Ref="R?"  Part="1"
 AR Path="/5E9E6BF0/5D1770D6" Ref="R401"  Part="1"
-F 0 "R301" V 1646 3200 50  0000 C CNN
+F 0 "R401" V 1646 3200 50  0000 C CNN
 F 1 "0" V 1555 3200 50  0000 C CNN
 F 2 "Resistor_SMD:R_0402_1005Metric" H 1450 3200 50  0001 C CNN
@@
 AR Path="/5E9D71BC/5DC5B696" Ref="T?"  Part="1"
 AR Path="/5E9E6BF0/5DC5B696" Ref="T401"  Part="1"
-F 0 "T301" H 2250 2975 50  0000 C CNN
+F 0 "T401" H 2250 2975 50  0000 C CNN
 F 1 "MABAES0060" H 2250 3066 50  0000 C CNN
 F 2 "vna_footprints:5LEAD_BALUN_4p83mm_3p3mm" H 2250 3400 50  0001 C CNN
@@
 AR Path="/5E9D71BC/5DC5DB88" Ref="T?"  Part="1"
 AR Path="/5E9E6BF0/5DC5DB88" Ref="T402"  Part="1"
-F 0 "T302" H 4450 2975 50  0000 C CNN
+F 0 "T402" H 4450 2975 50  0000 C CNN
 F 1 "MABAES0060" H 4450 3066 50  0000 C CNN
 F 2 "vna_footprints:5LEAD_BALUN_4p83mm_3p3mm" H 4450 3400 50  0001 C CNN
@@
 AR Path="/5E9D71BC/5E9DA88D" Ref="R?"  Part="1"
 AR Path="/5E9E6BF0/5E9DA88D" Ref="R404"  Part="1"
-F 0 "R304" H 3441 3904 50  0000 R CNN
+F 0 "R404" H 3441 3904 50  0000 R CNN
 F 1 "DNI" H 3441 3995 50  0000 R CNN
 F 2 "Resistor_SMD:R_0402_1005Metric" H 3500 3950 50  0001 C CNN
@@
 AR Path="/5E9D71BC/5E9DAD73" Ref="R?"  Part="1"
 AR Path="/5E9E6BF0/5E9DAD73" Ref="R403"  Part="1"
-F 0 "R303" H 3191 3904 50  0000 R CNN
+F 0 "R403" H 3191 3904 50  0000 R CNN
 F 1 "DNI" H 3191 3995 50  0000 R CNN
 F 2 "Resistor_SMD:R_0402_1005Metric" H 3250 3950 50  0001 C CNN
@@
 AR Path="/5E9D71BC/5E9E0753" Ref="#PWR?"  Part="1"
 AR Path="/5E9E6BF0/5E9E0753" Ref="#PWR0403"  Part="1"
-F 0 "#PWR0303" H 3250 3850 50  0001 C CNN
+F 0 "#PWR0403" H 3250 3850 50  0001 C CNN
 F 1 "GND" H 3255 3927 50  0000 C CNN
 F 2 "" H 3250 4100 50  0001 C CNN
@@
 AR Path="/5E9D71BC/5E9E35D5" Ref="#PWR?"  Part="1"
 AR Path="/5E9E6BF0/5E9E35D5" Ref="#PWR0404"  Part="1"
-F 0 "#PWR0304" H 3500 3850 50  0001 C CNN
+F 0 "#PWR0404" H 3500 3850 50  0001 C CNN
 F 1 "GND" H 3505 3927 50  0000 C CNN
 F 2 "" H 3500 4100 50  0001 C CNN
@@
 AR Path="/5E9D5B60/5EA1A0C8" Ref="J301"  Part="1"
 AR Path="/5E9E6BF0/5EA1A0C8" Ref="J401"  Part="1"
-F 0 "J301" V 924 3300 50  0000 L CNN
+F 0 "J401" V 924 3300 50  0000 L CNN
 F 1 "Conn_Coaxial" V 833 3300 50  0000 L CNN
 F 2 "vna_footprints:732512200_SMA" H 950 3200 50  0001 C CNN
@@
 AR Path="/5E9D71BC/5EA1D4DC" Ref="#PWR?"  Part="1"
 AR Path="/5E9E6BF0/5EA1D4DC" Ref="#PWR0408"  Part="1"
-F 0 "#PWR0308" H 950 3250 50  0001 C CNN
+F 0 "#PWR0408" H 950 3250 50  0001 C CNN
 F 1 "GND" H 955 3327 50  0000 C CNN
 F 2 "" H 950 3500 50  0001 C CNN
