File: breakouts/adc_32xx/ram_adc/adc.sch (KiCad schematic (older format))
At the start: 20 parts, among them J1 Conn_02x06_Odd_Even, J28 Conn_02x20_Odd_Even, U1 VEMI65AB-HCI, U2 ADC322x

Commit message: finished first pass adc32xx schematic
Parts:
- added C210, C211, C213: DNI, Capacitor_SMD:C_0402_1005Metric, symbol Device:C_Small
- added C214, C215: 100 nF, Capacitor_SMD:C_0402_1005Metric, symbol Device:C_Small
- added J201, J202: Conn_Coaxial, vna_footprints:732512200_SMA, symbol Connector:Conn_Coaxial
- added J205: Conn_01x07, Connector_PinSocket_2.54mm:PinSocket_1x07_P2.54mm_Vertical, symbol Connector_Generic:Conn_01x07
- added R201, R202: DNI, Resistor_SMD:R_0402_1005Metric, symbol Device:R_Small
- added R203, R204: 0, Resistor_SMD:R_0402_1005Metric, symbol Device:R_Small
- added R205: 100, Resistor_SMD:R_0402_1005Metric, symbol Device:R_Small
- J203: renamed from J1; footprint (none) -> Connector_PinHeader_2.54mm:PinHeader_2x06_P2.54mm_Vertical
- J204: renamed from J28; footprint (none) -> Connector_PinHeader_2.54mm:PinHeader_2x20_P2.54mm_Vertical
- R206: renamed from R1; value R_Small -> 1k
- U201: renamed from U1; footprint (none) -> vna_mm:LLP2513-13L
- renumbered C1 to C201, C2 to C202, C3 to C203, C4 to C204, C5 to C205, C6 to C206, C7 to C207, C8 to C208, C9 to C209, C10 to C212, C11 to C216, C12 to C217, C13 to C218, C14 to C219, D1 to D201, U2 to U202
Connections:
- net GND: now also C213.2, J201.1 (In), J202.1 (In), J205.7 (Pin_7), R201.1, R202.1
- net PDN: now also J205.5 (Pin_5)
- net RESET: now also J205.6 (Pin_6)
- net SCLK: now also J205.1 (Pin_1)
- net SDATA: now also J205.2 (Pin_2)
- net SDOUT: now also J205.4 (Pin_4)
- net SEN: now also J205.3 (Pin_3)
- net EN: now reaches J203.6 (Pin_6)
- net CLK_N renamed CLK_ADC_N
- net CLK_ADC_N: now also C215.2; no longer J204.30 (Pin_30)
- net CLK_P renamed CLK_ADC_P
- net CLK_ADC_P: now also C214.2; no longer J204.29 (Pin_29)
- new net: C210.2, C213.1, C215.1, R204.1, R205.1
- new net: C211.1, J202.2 (Ext), R202.2
- new net: C211.2, C214.1, R203.1, R205.2
- new net: C210.1, J201.2 (Ext), R201.2
- new net CLK_FPGA_P: R203.2, R204.2
- new net CLK_N_FPGA: J204.30 (Pin_30)
- new net CLK_P_FPGA: J204.29 (Pin_29)
Other:
- note removed: "TODO: add 2.5V to 1.8V switching regulator"
- note removed: "TODO: check LVDS compatibility ADC->ECP5 (2.5V LVDS)"
- note removed: "TODO: check LVDS compatibility ECP5 >ADC\nADD EXT CLOCK"
- moved on the sheet: J203

Commit message: component placement for adc322x breakout
Parts:
- added C220, C221: 100 nF, Capacitor_SMD:C_0402_1005Metric, symbol Device:C_Small
Connections:
- net CLK_P_FPGA is gone; now on net CLK_FPGA_P: J204.29 (Pin_29)
- net +1V8: now also C220.1, C221.1
- net CLK_FPGA_P: no longer R204.2
- net DA0_N: now also J204.6 (Pin_6); no longer J204.26 (Pin_26)
- net DA0_P: now also J204.5 (Pin_5); no longer J204.25 (Pin_25)
- net DA1_N: now also J204.10 (Pin_10); no longer J204.22 (Pin_22)
- net DA1_P: now also J204.9 (Pin_9); no longer J204.21 (Pin_21)
- net DB0_N: now also J204.22 (Pin_22); no longer J204.10 (Pin_10)
- net DB0_P: now also J204.21 (Pin_21); no longer J204.9 (Pin_9)
- net DB1_N: now also J204.26 (Pin_26); no longer J204.6 (Pin_6)
- net DB1_P: now also J204.25 (Pin_25); no longer J204.5 (Pin_5)
- net DCLK_N: now also J204.14 (Pin_14); no longer J204.18 (Pin_18)
- net DCLK_P: now also J204.13 (Pin_13); no longer J204.17 (Pin_17)
- net FCLK_N: now also J204.18 (Pin_18); no longer J204.14 (Pin_14)
- net FCLK_P: now also J204.17 (Pin_17); no longer J204.13 (Pin_13)
- net GND: now also J201.2 (Ext), J202.2 (Ext), C220.2, C221.2; no longer J201.1 (In), J202.1 (In)
- net at C211.1, R202.2: now also J202.1 (In); no longer J202.2 (Ext)
- net at C210.1, R201.2: now also J201.1 (In); no longer J201.2 (Ext)
- net CLK_N_FPGA renamed CLK_FPGA_N
- net CLK_FPGA_N: now also R204.2
- net IN_A_M renamed IN_A_N
- net IN_B_M renamed IN_B_N
Changed lines of the file:
@@
 $Descr A4 11693 8268
 encoding utf-8
-Sheet 2 5
+Sheet 5 5
 Title ""
 Date ""
@@
 IN_A_P
 Text HLabel 2550 2650 0    50   Input ~ 0
-IN_A_M
+IN_A_N
 Text HLabel 2550 3000 0    50   Input ~ 0
-IN_B_M
+IN_B_N
 Text HLabel 2550 2900 0    50   Input ~ 0
 IN_B_P
@@
 Wire Wire Line
 	5600 4100 5500 4100
+Text Label 8500 3250 2    50   ~ 0
+DB1_P
+Text Label 9500 3250 0    50   ~ 0
+DB1_N
+Text Label 8500 3050 2    50   ~ 0
+DB0_P
+Text Label 9500 3050 0    50   ~ 0
+DB0_N
+Text Label 8500 2850 2    50   ~ 0
+FCLK_P
+Text Label 9500 2850 0    50   ~ 0
+FCLK_N
+Text Label 8500 2650 2    50   ~ 0
+DCLK_P
+Text Label 9500 2650 0    50   ~ 0
+DCLK_N
+Text Label 8500 2450 2    50   ~ 0
+DA1_P
+Text Label 9500 2450 0    50   ~ 0
+DA1_N
 Text Label 8500 2250 2    50   ~ 0
-DB1_P
+DA0_P
 Text Label 9500 2250 0    50   ~ 0
-DB1_N
-Text Label 8500 2450 2    50   ~ 0
-DB0_P
-Text Label 9500 2450 0    50   ~ 0
-DB0_N
-Text Label 8500 2650 2    50   ~ 0
-FCLK_P
-Text Label 9500 2650 0    50   ~ 0
-FCLK_N
-Text Label 8500 2850 2    50   ~ 0
-DCLK_P
-Text Label 9500 2850 0    50   ~ 0
-DCLK_N
-Text Label 8500 3050 2    50   ~ 0
-DA1_P
-Text Label 9500 3050 0    50   ~ 0
-DA1_N
-Text Label 8500 3250 2    50   ~ 0
-DA0_P
-Text Label 9500 3250 0    50   ~ 0
 DA0_N
 Wire Wire Line
@@
 	3100 3900 3200 3900
 Text Label 8500 3450 2    50   ~ 0
-CLK_P_FPGA
+CLK_FPGA_P
 Text Label 9500 3450 0    50   ~ 0
-CLK_N_FPGA
+CLK_FPGA_N
 Text Label 8500 3650 2    50   ~ 0
 SYSREF_P
@@
 Wire Wire Line
 	4700 750  4700 800
-Text Label 6300 5600 0    50   ~ 0
-CLK_ADC_P
-Text Label 6300 6700 0    50   ~ 0
-CLK_ADC_N
 Text Label 5400 6700 2    50   ~ 0
-CLK_FPGA_P
-Text Label 5200 5600 2    50   ~ 0
-CLK_FPGA_P
+CLK_FPGA_N
 $Comp
 L Device:R_Small R204
@@
 F 3 " ~" H 5150 5950 50  0001 C CNN
 	1    5150 5950
-	0    -1   -1   0
+	-1   0    0    -1
 $EndComp
 $Comp
@@
 F 3 " ~" H 5100 7050 50  0001 C CNN
 	1    5100 7050
-	0    -1   -1   0
+	-1   0    0    -1
 $EndComp
 $Comp
@@
 Wire Wire Line
 	1450 5800 1350 5800
+$Comp
+L Device:C_Small C220
+U 1 1 5EBA28B5
+P 8000 1600
+F 0 "C220" H 8092 1646 50  0000 L CNN
+F 1 "100 nF" H 8092 1555 50  0000 L CNN
+F 2 "Capacitor_SMD:C_0402_1005Metric" H 8000 1600 50  0001 C CNN
+F 3 "~" H 8000 1600 50  0001 C CNN
+	1    8000 1600
+	1    0    0    -1
+$EndComp
+$Comp
+L power:GND #PWR?
+U 1 1 5EBA28BB
+P 8000 1750
+AR Path="/5EBA28BB" Ref="#PWR?"  Part="1"
+AR Path="/5E9D7371/5EBA28BB" Ref="#PWR0102"  Part="1"
+F 0 "#PWR0102" H 8000 1500 50  0001 C CNN
+F 1 "GND" H 8005 1577 50  0000 C CNN
+F 2 "" H 8000 1750 50  0001 C CNN
+F 3 "" H 8000 1750 50  0001 C CNN
+	1    8000 1750
+	1    0    0    -1
+$EndComp
+Wire Wire Line
+	8000 1700 8000 1750
+Wire Wire Line
+	8000 1450 8000 1500
+Wire Wire Line
+	7550 1450 8000 1450
+$Comp
+L Device:C_Small C221
+U 1 1 5EBB3C4B
+P 8450 1600
+F 0 "C221" H 8542 1646 50  0000 L CNN
+F 1 "100 nF" H 8542 1555 50  0000 L CNN
+F 2 "Capacitor_SMD:C_0402_1005Metric" H 8450 1600 50  0001 C CNN
+F 3 "~" H 8450 1600 50  0001 C CNN
+	1    8450 1600
+	1    0    0    -1
+$EndComp
+$Comp
+L power:GND #PWR?
+U 1 1 5EBB3C51
+P 8450 1750
+AR Path="/5EBB3C51" Ref="#PWR?"  Part="1"
+AR Path="/5E9D7371/5EBB3C51" Ref="#PWR0103"  Part="1"
+F 0 "#PWR0103" H 8450 1500 50  0001 C CNN
+F 1 "GND" H 8455 1577 50  0000 C CNN
+F 2 "" H 8450 1750 50  0001 C CNN
+F 3 "" H 8450 1750 50  0001 C CNN
+	1    8450 1750
+	1    0    0    -1
+$EndComp
+Wire Wire Line
+	8450 1700 8450 1750
+Wire Wire Line
+	8450 1450 8450 1500
+Wire Wire Line
+	8000 1450 8450 1450
+Text Label 5200 5600 2    50   ~ 0
+CLK_FPGA_P
+Text Label 6300 5600 0    50   ~ 0
+CLK_ADC_P
+Text Label 6300 6700 0    50   ~ 0
+CLK_ADC_N
 $EndSCHEMATC

Commit message: writing to wishbone from the fpga works..
Parts:
- U201: symbol vna_mm:VEMI65AB-HCI -> adc_32xx-rescue:VEMI65AB-HCI-vna_mm
- U202: symbol vna_mm:ADC322x -> adc_32xx-rescue:ADC322x-vna_mm
Changed lines of the file:
@@
 $EndComp
 $Comp
-L vna_mm:ADC322x U?
+L adc_32xx-rescue:ADC322x-vna_mm U?
 U 1 1 5E9D7BC3
 P 4350 3550
@@
 SYSREF_N
 $Comp
-L vna_mm:VEMI65AB-HCI U201
+L adc_32xx-rescue:VEMI65AB-HCI-vna_mm U201
 U 1 1 5EB301B2
 P 2200 4300
